Commit message: Added revised script for rope macro creation and modified mmcuav_rope to work with new macro.

File: mmuav_description/urdf/mmcuav_rope.base.urdf.xacro (robot description, xacro)
@@ -32,19 +32,6 @@
   <xacro:property name="cos45" value="0.7071" />
   <xacro:property name="PI" value="3.1415926535897931" />
-  <xacro:property name="width_1" value="0.004"/>
-  <xacro:property name="body_len" value="0.02"/>
-  <xacro:property name="box_param" value="0.0"/>
-  <xacro:property name="radius" value="0.05"/>
-  <xacro:property name="load_mass" value="0.1"/>
-  <xacro:property name="friction" value="0.02"/>
-  <xacro:property name="damping1" value="0.5"/>
-  <xacro:property name="effort_joint" value="1000"/>
-  <xacro:property name="inertia_rope1" value="0.01"/>
-  <xacro:property name="inertia_rope2" value="0.02"/>
-  <xacro:property name="mass_rope" value="0.01"/>
-  <xacro:property name="mass_link" value="0.001"/>
-  <xacro:property name="inertia_link" value="0.01"/>
-  <xacro:property name="velocity_joint" value="300"/>
-  <xacro:property name="load_inertia" value="0.0"/>
+  <xacro:include filename="$(find mmuav_description)/urdf/rope_macro.xacro" />
+  <xacro:robot_macro base_link="base_link"/>
   <!-- Property Blocks -->
   <xacro:property name="body_inertia">
@@ -62,587 +49,4 @@
   <!-- Included URDF Files -->
   <xacro:include filename="$(find mmuav_description)/urdf/multirotor_base.urdf.xacro" />
-  <link name="rope_1">
-    <visual>
-      <geometry>
-        <cylinder length="${body_len}" radius="${width_1}"/>
-      </geometry>
-      <origin rpy="0.0 0.0 0.0" xyz="0 0 ${-body_len/2}"/>
-    </visual>
-    <collision>
-      <geometry>
-        <cylinder length="${body_len}" radius="${width_1}"/>
-      </geometry>
-      <origin rpy="0.0 0.0 0.0" xyz="0 0 ${-body_len/2}"/>
-    </collision>
-    <inertial>
-      <mass value="${mass_rope}"/>
-      <inertia ixx="${inertia_rope1}" ixy="0.0" ixz="0.0" iyy="${inertia_rope1}" iyz="0.0" izz="${inertia_rope2}"/>
-      <origin rpy="0.0 0.0 0.0" xyz="0 0 ${-body_len/2}"/>
-    </inertial>
-  </link>
-  <link name="rope_2">
-    <visual>
-      <geometry>
-        <cylinder length="${body_len}" radius="${width_1}"/>
-      </geometry>
-      <origin rpy="0.0 0.0 0.0" xyz="0 0 ${-body_len/2}"/>
-    </visual>
-    <collision>
-      <geometry>
-        <cylinder length="${body_len}" radius="${width_1}"/>
-      </geometry>
-      <origin rpy="0.0 0.0 0.0" xyz="0 0 ${-body_len/2}"/>
-    </collision>
-    <inertial>
-      <mass value="${mass_rope}"/>
-      <inertia ixx="${inertia_rope1}" ixy="0.0" ixz="0.0" iyy="${inertia_rope1}" iyz="0.0" izz="${inertia_rope2}"/>
-      <origin rpy="0.0 0.0 0.0" xyz="0 0 ${-body_len/2}"/>
-    </inertial>
-  </link>
-  <link name="rope_3">
-    <visual>
-      <geometry>
-        <cylinder length="${body_len}" radius="${width_1}"/>
-      </geometry>
-      <origin rpy="0.0 0.0 0.0" xyz="0 0 ${-body_len/2}"/>
-    </visual>
-    <collision>
-      <geometry>
-        <cylinder length="${body_len}" radius="${width_1}"/>
-      </geometry>
-      <origin rpy="0.0 0.0 0.0" xyz="0 0 ${-body_len/2}"/>
-    </collision>
-    <inertial>
-      <mass value="${mass_rope}"/>
-      <inertia ixx="${inertia_rope1}" ixy="0.0" ixz="0.0" iyy="${inertia_rope1}" iyz="0.0" izz="${inertia_rope2}"/>
-      <origin rpy="0.0 0.0 0.0" xyz="0 0 ${-body_len/2}"/>
-    </inertial>
-  </link>
-  <link name="rope_4">
-    <visual>
-      <geometry>
-        <cylinder length="${body_len}" radius="${width_1}"/>
-      </geometry>
-      <origin rpy="0.0 0.0 0.0" xyz="0 0 ${-body_len/2}"/>
-    </visual>
-    <collision>
-      <geometry>
-        <cylinder length="${body_len}" radius="${width_1}"/>
-      </geometry>
-      <origin rpy="0.0 0.0 0.0" xyz="0 0 ${-body_len/2}"/>
-    </collision>
-    <inertial>
-      <mass value="${mass_rope}"/>
-      <inertia ixx="${inertia_rope1}" ixy="0.0" ixz="0.0" iyy="${inertia_rope1}" iyz="0.0" izz="${inertia_rope2}"/>
-      <origin rpy="0.0 0.0 0.0" xyz="0 0 ${-body_len/2}"/>
-    </inertial>
-  </link>
-  <link name="rope_5">
-    <visual>
-      <geometry>
-        <cylinder length="${body_len}" radius="${width_1}"/>
-      </geometry>
-      <origin rpy="0.0 0.0 0.0" xyz="0 0 ${-body_len/2}"/>
-    </visual>
-    <collision>
-      <geometry>
-        <cylinder length="${body_len}" radius="${width_1}"/>
-      </geometry>
-      <origin rpy="0.0 0.0 0.0" xyz="0 0 ${-body_len/2}"/>
-    </collision>
-    <inertial>
-      <mass value="${mass_rope}"/>
-      <inertia ixx="${inertia_rope1}" ixy="0.0" ixz="0.0" iyy="${inertia_rope1}" iyz="0.0" izz="${inertia_rope2}"/>
-      <origin rpy="0.0 0.0 0.0" xyz="0 0 ${-body_len/2}"/>
-    </inertial>
-  </link>
-  <link name="rope_6">
-    <visual>
-      <geometry>
-        <cylinder length="${body_len}" radius="${width_1}"/>
-      </geometry>
-      <origin rpy="0.0 0.0 0.0" xyz="0 0 ${-body_len/2}"/>
-    </visual>
-    <collision>
-      <geometry>
-        <cylinder length="${body_len}" radius="${width_1}"/>
-      </geometry>
-      <origin rpy="0.0 0.0 0.0" xyz="0 0 ${-body_len/2}"/>
-    </collision>
-    <inertial>
-      <mass value="${mass_rope}"/>
-      <inertia ixx="${inertia_rope1}" ixy="0.0" ixz="0.0" iyy="${inertia_rope1}" iyz="0.0" izz="${inertia_rope2}"/>
-      <origin rpy="0.0 0.0 0.0" xyz="0 0 ${-body_len/2}"/>
-    </inertial>
-  </link>
-  <link name="rope_7">
-    <visual>
-      <geometry>
-        <cylinder length="${body_len}" radius="${width_1}"/>
-      </geometry>
-      <origin rpy="0.0 0.0 0.0" xyz="0 0 ${-body_len/2}"/>
-    </visual>
-    <collision>
-      <geometry>
-        <cylinder length="${body_len}" radius="${width_1}"/>
-      </geometry>
-      <origin rpy="0.0 0.0 0.0" xyz="0 0 ${-body_len/2}"/>
-    </collision>
-    <inertial>
-      <mass value="${mass_rope}"/>
-      <inertia ixx="${inertia_rope1}" ixy="0.0" ixz="0.0" iyy="${inertia_rope1}" iyz="0.0" izz="${inertia_rope2}"/>
-      <origin rpy="0.0 0.0 0.0" xyz="0 0 ${-body_len/2}"/>
-    </inertial>
-  </link>
-  <link name="rope_8">
-    <visual>
-      <geometry>
-        <cylinder length="${body_len}" radius="${width_1}"/>
-      </geometry>
-      <origin rpy="0.0 0.0 0.0" xyz="0 0 ${-body_len/2}"/>
-    </visual>
-    <collision>
-      <geometry>
-        <cylinder length="${body_len}" radius="${width_1}"/>
-      </geometry>
-      <origin rpy="0.0 0.0 0.0" xyz="0 0 ${-body_len/2}"/>
-    </collision>
-    <inertial>
-      <mass value="${mass_rope}"/>
-      <inertia ixx="${inertia_rope1}" ixy="0.0" ixz="0.0" iyy="${inertia_rope1}" iyz="0.0" izz="${inertia_rope2}"/>
-      <origin rpy="0.0 0.0 0.0" xyz="0 0 ${-body_len/2}"/>
-    </inertial>
-  </link>
-  <link name="rope_9">
-    <visual>
-      <geometry>
-        <cylinder length="${body_len}" radius="${width_1}"/>
-      </geometry>
-      <origin rpy="0.0 0.0 0.0" xyz="0 0 ${-body_len/2}"/>
-    </visual>
-    <collision>
-      <geometry>
-        <cylinder length="${body_len}" radius="${width_1}"/>
-      </geometry>
-      <origin rpy="0.0 0.0 0.0" xyz="0 0 ${-body_len/2}"/>
-    </collision>
-    <inertial>
-      <mass value="${mass_rope}"/>
-      <inertia ixx="${inertia_rope1}" ixy="0.0" ixz="0.0" iyy="${inertia_rope1}" iyz="0.0" izz="${inertia_rope2}"/>
-      <origin rpy="0.0 0.0 0.0" xyz="0 0 ${-body_len/2}"/>
-    </inertial>
-  </link>
-  <link name="rope_10">
-    <visual>
-      <geometry>
-        <cylinder length="${body_len}" radius="${width_1}"/>
-      </geometry>
-      <origin rpy="0.0 0.0 0.0" xyz="0 0 ${-body_len/2}"/>
-    </visual>
-    <collision>
-      <geometry>
-        <cylinder length="${body_len}" radius="${width_1}"/>
-      </geometry>
-      <origin rpy="0.0 0.0 0.0" xyz="0 0 ${-body_len/2}"/>
-    </collision>
-    <inertial>
-      <mass value="${mass_rope}"/>
-      <inertia ixx="${inertia_rope1}" ixy="0.0" ixz="0.0" iyy="${inertia_rope1}" iyz="0.0" izz="${inertia_rope2}"/>
-      <origin rpy="0.0 0.0 0.0" xyz="0 0 ${-body_len/2}"/>
-    </inertial>
-  </link>
-  <link name="load">
-    <visual>
-      <geometry>
-        <sphere radius="${radius}"/>
-      </geometry>
-      <origin rpy="0.0 0.0 0.0" xyz="0 0 ${-radius}"/>
-    </visual>
-    <collision>
-      <geometry>
-        <sphere radius="${radius}"/>
-      </geometry>
-      <origin rpy="0.0 0.0 0.0" xyz="0 0 ${-radius}"/>
-    </collision>
-    <inertial>
-      <mass value="${load_mass}"/>
-      <inertia ixx="${load_inertia}" ixy="0.0" ixz="0.0" iyy="${load_inertia}" iyz="0.0" izz="${load_inertia}"/>
-      <origin rpy="0.0 0.0 0.0" xyz="0 0 ${-radius}"/>
-    </inertial>
-  </link>
-  <link name="rope1Theta">
-    <inertial>
-      <mass value="${mass_link}"/>
-      <inertia ixx="${inertia_link}" ixy="0.0" ixz="0.0" iyy="${inertia_link}" iyz="0.0" izz="${inertia_link}"/>
-    </inertial>
-  </link>
-  <link name="rope1Psi">
-    <inertial>
-      <mass value="${mass_link}"/>
-      <inertia ixx="${inertia_link}" ixy="0.0" ixz="0.0" iyy="${inertia_link}" iyz="0.0" izz="${inertia_link}"/>
-    </inertial>
-  </link>
-  <joint name="base_link_to_rope1Psi" type="revolute">
-    <parent link="base_link"/>
-    <child link="rope1Psi"/>
-    <origin rpy="0.0 0.0 0.0" xyz="0 0 ${-box_param/2}"/>
-    <axis xyz="0 0 1"/>
-    <dynamics damping="${damping1}" friction="${friction}"/>
-    <limit effort="${effort_joint}" lower="${-pi/2}" upper="${pi/2}" velocity="${velocity_joint}"/>
-  </joint>
-  <joint name="rope1Psi_to_rope1Theta" type="revolute">
-    <parent link="rope1Psi"/>
-    <child link="rope1Theta"/>
-    <axis xyz="0 1 0"/>
-    <dynamics damping="${damping1}" friction="${friction}"/>
-    <limit effort="${effort_joint}" lower="${-pi/2}" upper="${pi/2}" velocity="${velocity_joint}"/>
-  </joint>
-  <joint name="rope1Theta_to_rope_1" type="revolute">
-    <parent link="rope1Theta"/>
-    <child link="rope_1"/>
-    <axis xyz="1 0 0"/>
-    <dynamics damping="${damping1}" friction="${friction}"/>
-    <limit effort="${effort_joint}" lower="${-pi/16}" upper="${pi/16}" velocity="${velocity_joint}"/>
-  </joint>
-  <link name="rope2Theta">
-    <inertial>
-      <mass value="${mass_link}"/>
-      <inertia ixx="${inertia_link}" ixy="0.0" ixz="0.0" iyy="${inertia_link}" iyz="0.0" izz="${inertia_link}"/>
-    </inertial>
-  </link>
-  <link name="rope2Psi">
-    <inertial>
-      <mass value="${mass_link}"/>
-      <inertia ixx="${inertia_link}" ixy="0.0" ixz="0.0" iyy="${inertia_link}" iyz="0.0" izz="${inertia_link}"/>
-    </inertial>
-  </link>
-  <joint name="rope_1_to_rope2Psi" type="revolute">
-    <parent link="rope_1"/>
-    <child link="rope2Psi"/>
-    <origin rpy="0.0 0.0 0.0" xyz="0 0 ${-body_len}"/>
-    <axis xyz="0 0 1"/>
-    <dynamics damping="${damping1}" friction="${friction}"/>
-    <limit effort="${effort_joint}" lower="${-pi/2}" upper="${pi/2}" velocity="${velocity_joint}"/>
-  </joint>
-  <joint name="rope2Psi_to_rope2Theta" type="revolute">
-    <parent link="rope2Psi"/>
-    <child link="rope2Theta"/>
-    <axis xyz="0 1 0"/>
-    <dynamics damping="${damping1}" friction="${friction}"/>
-    <limit effort="${effort_joint}" lower="${-pi/2}" upper="${pi/2}" velocity="${velocity_joint}"/>
-  </joint>
-  <joint name="rope2Theta_to_rope_2" type="revolute">
-    <parent link="rope2Theta"/>
-    <child link="rope_2"/>
-    <axis xyz="1 0 0"/>
-    <dynamics damping="${damping1}" friction="${friction}"/>
-    <limit effort="${effort_joint}" lower="${-pi/16}" upper="${pi/16}" velocity="${velocity_joint}"/>
-  </joint>
-  <link name="rope3Theta">
-    <inertial>
-      <mass value="${mass_link}"/>
-      <inertia ixx="${inertia_link}" ixy="0.0" ixz="0.0" iyy="${inertia_link}" iyz="0.0" izz="${inertia_link}"/>
-    </inertial>
-  </link>
-  <link name="rope3Psi">
-    <inertial>
-      <mass value="${mass_link}"/>
-      <inertia ixx="${inertia_link}" ixy="0.0" ixz="0.0" iyy="${inertia_link}" iyz="0.0" izz="${inertia_link}"/>
-    </inertial>
-  </link>
-  <joint name="rope_2_to_rope3Psi" type="revolute">
-    <parent link="rope_2"/>
-    <child link="rope3Psi"/>
-    <origin rpy="0.0 0.0 0.0" xyz="0 0 ${-body_len}"/>
-    <axis xyz="0 0 1"/>
-    <dynamics damping="${damping1}" friction="${friction}"/>
-    <limit effort="${effort_joint}" lower="${-pi/2}" upper="${pi/2}" velocity="${velocity_joint}"/>
-  </joint>
-  <joint name="rope3Psi_to_rope3Theta" type="revolute">
-    <parent link="rope3Psi"/>
-    <child link="rope3Theta"/>
-    <axis xyz="0 1 0"/>
-    <dynamics damping="${damping1}" friction="${friction}"/>
-    <limit effort="${effort_joint}" lower="${-pi/2}" upper="${pi/2}" velocity="${velocity_joint}"/>
-  </joint>
-  <joint name="rope3Theta_to_rope_3" type="revolute">
-    <parent link="rope3Theta"/>
-    <child link="rope_3"/>
-    <axis xyz="1 0 0"/>
-    <dynamics damping="${damping1}" friction="${friction}"/>
-    <limit effort="${effort_joint}" lower="${-pi/16}" upper="${pi/16}" velocity="${velocity_joint}"/>
-  </joint>
-  <link name="rope4Theta">
-    <inertial>
-      <mass value="${mass_link}"/>
-      <inertia ixx="${inertia_link}" ixy="0.0" ixz="0.0" iyy="${inertia_link}" iyz="0.0" izz="${inertia_link}"/>
-    </inertial>
-  </link>
-  <link name="rope4Psi">
-    <inertial>
-      <mass value="${mass_link}"/>
-      <inertia ixx="${inertia_link}" ixy="0.0" ixz="0.0" iyy="${inertia_link}" iyz="0.0" izz="${inertia_link}"/>
-    </inertial>
-  </link>
-  <joint name="rope_3_to_rope4Psi" type="revolute">
-    <parent link="rope_3"/>
-    <child link="rope4Psi"/>
-    <origin rpy="0.0 0.0 0.0" xyz="0 0 ${-body_len}"/>
-    <axis xyz="0 0 1"/>
-    <dynamics damping="${damping1}" friction="${friction}"/>
-    <limit effort="${effort_joint}" lower="${-pi/2}" upper="${pi/2}" velocity="${velocity_joint}"/>
-  </joint>
-  <joint name="rope4Psi_to_rope4Theta" type="revolute">
-    <parent link="rope4Psi"/>
-    <child link="rope4Theta"/>
-    <axis xyz="0 1 0"/>
-    <dynamics damping="${damping1}" friction="${friction}"/>
-    <limit effort="${effort_joint}" lower="${-pi/2}" upper="${pi/2}" velocity="${velocity_joint}"/>
-  </joint>
-  <joint name="rope4Theta_to_rope_4" type="revolute">
-    <parent link="rope4Theta"/>
-    <child link="rope_4"/>
-    <axis xyz="1 0 0"/>
-    <dynamics damping="${damping1}" friction="${friction}"/>
-    <limit effort="${effort_joint}" lower="${-pi/16}" upper="${pi/16}" velocity="${velocity_joint}"/>
-  </joint>
-  <link name="rope5Theta">
-    <inertial>
-      <mass value="${mass_link}"/>
-      <inertia ixx="${inertia_link}" ixy="0.0" ixz="0.0" iyy="${inertia_link}" iyz="0.0" izz="${inertia_link}"/>
-    </inertial>
-  </link>
-  <link name="rope5Psi">
-    <inertial>
-      <mass value="${mass_link}"/>
-      <inertia ixx="${inertia_link}" ixy="0.0" ixz="0.0" iyy="${inertia_link}" iyz="0.0" izz="${inertia_link}"/>
-    </inertial>
-  </link>
-  <joint name="rope_4_to_rope5Psi" type="revolute">
-    <parent link="rope_4"/>
-    <child link="rope5Psi"/>
-    <origin rpy="0.0 0.0 0.0" xyz="0 0 ${-body_len}"/>
-    <axis xyz="0 0 1"/>
-    <dynamics damping="${damping1}" friction="${friction}"/>
-    <limit effort="${effort_joint}" lower="${-pi/2}" upper="${pi/2}" velocity="${velocity_joint}"/>
-  </joint>
-  <joint name="rope5Psi_to_rope5Theta" type="revolute">
-    <parent link="rope5Psi"/>
-    <child link="rope5Theta"/>
-    <axis xyz="0 1 0"/>
-    <dynamics damping="${damping1}" friction="${friction}"/>
-    <limit effort="${effort_joint}" lower="${-pi/2}" upper="${pi/2}" velocity="${velocity_joint}"/>
-  </joint>
-  <joint name="rope5Theta_to_rope_5" type="revolute">
-    <parent link="rope5Theta"/>
-    <child link="rope_5"/>
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