Commit message: Added bunch of changes

File: mmuav_description/urdf/mmcuav_rope.gazebo.xacro (robot description, xacro)
@@ -85,3 +85,15 @@
     <origin xyz="-0.0 0.0 0" rpy="0.0 0.0 0.0" />
   </xacro:odometry_plugin_macro>
+  <!-- Add a wind gust starting at 40s and lasting for 2s. -->
+  <xacro:wind_plugin_macro
+    namespace="$(arg name)"
+    xyz_offset="0 0 0"
+    wind_direction="1 0 0"
+    wind_force_mean="0"
+    wind_gust_direction="1 0 0"
+    wind_gust_duration="12"
+    wind_gust_start="10"
+    wind_gust_force_mean="1"
+    affect_link="load">
+  </xacro:wind_plugin_macro>
 </robot>

File: mmuav_description/urdf/rope_macro_dobar.xacro (robot description, xacro)
@@ -1,5 +1,5 @@
 <?xml version='1.0' encoding='utf-8'?>
 <robot xmlns:xacro="http://www.ros.org/wiki/xacro" name="myrobot">
-  <xacro:macro name="robot_macro" params="base_link:='base_link' radius:=0.1001 effort_joint:=1000 small:=0.005 body_len:=0.0333333333333 load_inertia:=3.2e-07 velocity_joint:=300 damping1:=0.5 large:=100 inertia_link:=0.0015 mass_link:=0.005 inertia_rope2:=0.0 friction:=0.02 load_mass:=0.5 inertia_rope1:=1.55478395062e-07 box_param1:=0.25 spawn_point:=365.0 box_param:=0.0 mass_rope:=0.00166666666667 width_1:=0.00166666666667 k1:=10.0 k2:=100.0">
+  <xacro:macro name="robot_macro" params="base_link:='base_link' radius:=0.1001 effort_joint:=1000 small:=0.005 body_len:=0.0333333333333 load_inertia:=3.2e-07 velocity_joint:=300 damping1:=0.5 large:=100 inertia_link:=0.0015 mass_link:=0.01 inertia_rope2:=0.0 friction:=0.02 load_mass:=0.5 inertia_rope1:=1.55478395062e-07 box_param1:=0.25 spawn_point:=365.0 box_param:=0.0 mass_rope:=0.00166666666667 width_1:=0.00166666666667 k1:=1.0 k2:=1.0">
     <link name="rope_1">
       <visual>
@@ -204,10 +204,10 @@
         <origin rpy="0.0 0.0 0.0" xyz="0 0 ${-radius}"/>
       </visual>
-      <!--collision>
+      <collision>
         <geometry>
           <sphere radius="${radius}"/>
         </geometry>
         <origin rpy="0.0 0.0 0.0" xyz="0 0 ${-radius}"/>
-      </collision-->
+      </collision>
       <inertial>
         <mass value="${load_mass}"/>
@@ -234,5 +234,5 @@
       <axis xyz="0 0 1"/>
       <dynamics damping="${damping1}" friction="0"/>
-      <limit effort="${effort_joint}" lower="${-pi/2}" upper="${pi/2}" velocity="${velocity_joint}"/>
+      <limit effort="${effort_joint}" lower="${-k1*pi/2}" upper="${k1*pi/2}" velocity="${velocity_joint}"/>
     </joint>
     <joint name="rope1Psi_to_rope1Theta" type="revolute">
@@ -241,5 +241,5 @@
       <axis xyz="0 1 0"/>
       <dynamics damping="${damping1}" friction="0"/>
-      <limit effort="${effort_joint}" lower="${-pi/2}" upper="${pi/2}" velocity="${velocity_joint}"/>
+      <limit effort="${effort_joint}" lower="${-k1*pi/2}" upper="${k1*pi/2}" velocity="${velocity_joint}"/>
     </joint>
     <joint name="rope1Theta_to_rope_1" type="revolute">
@@ -248,5 +248,5 @@
       <axis xyz="1 0 0"/>
       <dynamics damping="${damping1}" friction="0"/>
-      <limit effort="${effort_joint}" lower="${-pi/16}" upper="${pi/16}" velocity="${velocity_joint}"/>
+      <limit effort="${effort_joint}" lower="${-k2*pi/16}" upper="${k2*pi/16}" velocity="${velocity_joint}"/>
     </joint>
     <link name="rope2Theta">
@@ -744,5 +744,5 @@
       <axis xyz="0 0 1"/>
       <dynamics damping="${damping1}" friction="${friction}"/>
-      <limit effort="${effort_joint}" lower="${-pi/2}" upper="${pi/2}" velocity="${velocity_joint}"/>
+      <limit effort="${effort_joint}" lower="${-k1*pi/2}" upper="${k1*pi/2}" velocity="${velocity_joint}"/>
     </joint>
     <joint name="rope16Psi_to_rope16Theta" type="revolute">
@@ -751,5 +751,5 @@
       <axis xyz="0 1 0"/>
       <dynamics damping="${damping1}" friction="${friction}"/>
-      <limit effort="${effort_joint}" lower="${-pi/2}" upper="${pi/2}" velocity="${velocity_joint}"/>
+      <limit effort="${effort_joint}" lower="${-k1*pi/2}" upper="${k1*pi/2}" velocity="${velocity_joint}"/>
     </joint>
     <joint name="rope16Theta_to_load" type="revolute">
@@ -758,5 +758,5 @@
       <axis xyz="1 0 0"/>
       <dynamics damping="${damping1}" friction="${friction}"/>
-      <limit effort="${effort_joint}" lower="${-pi/16}" upper="${pi/16}" velocity="${velocity_joint}"/>
+      <limit effort="${effort_joint}" lower="${-k2*pi/16}" upper="${k2*pi/16}" velocity="${velocity_joint}"/>
     </joint>
     <gazebo reference="rope_1">

Commit message: A lot of tweaks to code, added camera.

File: mmuav_description/urdf/mmcuav_rope.gazebo.xacro (robot description, xacro)
@@ -85,4 +85,34 @@
     <origin xyz="-0.0 0.0 0" rpy="0.0 0.0 0.0" />
   </xacro:odometry_plugin_macro>
+  <!-- Mount load generic pose sensor-->
+  <xacro:odometry_plugin_macro
+    namespace="$(arg name)"
+    odometry_sensor_suffix="2"
+    child_frame_id="base"
+    parent_link="load"
+    pose_topic="load_pose"
+    pose_with_covariance_topic="load_pose_with_covariance"
+    position_topic="load_position"
+    transform_topic="load_transform"
+    odometry_topic="load_odometry"
+    parent_frame_id="world"
+    mass_odometry_sensor="0.01"
+    measurement_divisor="10"
+    measurement_delay="10"
+    unknown_delay="0.0"
+    noise_normal_position="0.0 0.0 0.0"
+    noise_normal_quaternion="0.0 0.0 0.0"
+    noise_normal_linear_velocity="0 0 0"
+    noise_normal_angular_velocity="0 0 0"
+    noise_uniform_position="0 0 0"
+    noise_uniform_quaternion="0 0 0"
+    noise_uniform_linear_velocity="0 0 0"
+    noise_uniform_angular_velocity="0 0 0"
+    enable_odometry_map="false"
+    odometry_map=""
+    image_scale="0.1">
+    <inertia ixx="1e-8" ixy="0.0" ixz="0.0" iyy="1e-8" iyz="0.0" izz="1e-8" /> <!-- [kg m^2] [kg m^2] [kg m^2] [kg m^2] [kg m^2] [kg m^2] -->
+    <origin xyz="-0.0 0.0 0" rpy="0.0 0.0 0.0" />
+  </xacro:odometry_plugin_macro>
   <!-- Add a wind gust starting at 40s and lasting for 2s. -->
   <xacro:wind_plugin_macro
@@ -91,9 +121,82 @@
     wind_direction="1 0 0"
     wind_force_mean="0"
-    wind_gust_direction="1 0 0"
-    wind_gust_duration="12"
-    wind_gust_start="10"
-    wind_gust_force_mean="1"
-    affect_link="load">
-  </xacro:wind_plugin_macro>
+    wind_gust_direction="0.7926 0 0.6097"
+    wind_gust_duration="0.01"
+    wind_gust_start="20"
+    wind_gust_force_mean="200.0"
+    wind_gust_force_variance="0"
+    affect_link="load">
+  </xacro:wind_plugin_macro>
+  <!--xacro:wind_plugin_macro
+    namespace="$(arg name)"
+    xyz_offset="0 0 0"
+    wind_direction="1 0 0"
+    wind_force_mean="0"
+    wind_gust_direction="0.7926 0 0.6097"
+    wind_gust_duration="0.01"
+    wind_gust_start="70"
+    wind_gust_force_mean="100.0"
+    wind_gust_force_variance="0"
+    affect_link="load">
+  </xacro:wind_plugin_macro>
+  <xacro:wind_plugin_macro
+    namespace="$(arg name)"
+    xyz_offset="0 0 0"
+    wind_direction="1 0 0"
+    wind_force_mean="0"
+    wind_gust_direction="0.7926 0 0.6097"
+    wind_gust_duration="0.01"
+    wind_gust_start="130"
+    wind_gust_force_mean="150.0"
+    wind_gust_force_variance="0"
+    affect_link="load">
+  </xacro:wind_plugin_macro>
+  <xacro:wind_plugin_macro
+    namespace="$(arg name)"
+    xyz_offset="0 0 0"
+    wind_direction="1 0 0"
+    wind_force_mean="0"
+    wind_gust_direction="0.7926 0 0.6097"
+    wind_gust_duration="0.01"
+    wind_gust_start="310"
+    wind_gust_force_mean="175.0"
+    wind_gust_force_variance="0"
+    affect_link="load">
+  </xacro:wind_plugin_macro>
+  <xacro:wind_plugin_macro
+    namespace="$(arg name)"
+    xyz_offset="0 0 0"
+    wind_direction="1 0 0"
+    wind_force_mean="0"
+    wind_gust_direction="0.7926 0 0.6097"
+    wind_gust_duration="0.01"
+    wind_gust_start="170"
+    wind_gust_force_mean="200.0"
+    wind_gust_force_variance="0"
+    affect_link="load">
+  </xacro:wind_plugin_macro>
+  <xacro:wind_plugin_macro
+    namespace="$(arg name)"
+    xyz_offset="0 0 0"
+    wind_direction="1 0 0"
+    wind_force_mean="0"
+    wind_gust_direction="0.7926 0 0.6097"
+    wind_gust_duration="0.01"
+    wind_gust_start="210"
+    wind_gust_force_mean="225.0"
+    wind_gust_force_variance="0"
+    affect_link="load">
+  </xacro:wind_plugin_macro>
+  <xacro:wind_plugin_macro
+    namespace="$(arg name)"
+    xyz_offset="0 0 0"
+    wind_direction="1 0 0"
+    wind_force_mean="0"
+    wind_gust_direction="0.7926 0 0.6097"
+    wind_gust_duration="0.01"
+    wind_gust_start="250"
+    wind_gust_force_mean="300.0"
+    wind_gust_force_variance="0"
+    affect_link="load">
+  </xacro:wind_plugin_macro-->
 </robot>

File: mmuav_description/urdf/multirotor_base.urdf.xacro (robot description, xacro)
@@ -196,6 +196,6 @@
           <horizontal_fov>1.3962634</horizontal_fov>
           <image>
-            <width>800</width>
-            <height>800</height>
+            <width>1920</width>
+            <height>1080</height>
             <format>R8G8B8</format>
           </image>
@@ -213,5 +213,5 @@
           <alwaysOn>true</alwaysOn>
           <updateRate>0.0</updateRate>
-          <cameraName>morus/camera1</cameraName>
+          <cameraName>mmuav/camera1</cameraName>
           <imageTopicName>image_raw</imageTopicName>
           <cameraInfoTopicName>camera_info</cameraInfoTopicName>

File: mmuav_description/urdf/rope_macro.xacro (robot description, xacro)
@@ -1,5 +1,6 @@
 <?xml version='1.0' encoding='utf-8'?>
+<!-- body len = 0.033333333333333 -->
 <robot xmlns:xacro="http://www.ros.org/wiki/xacro" name="myrobot">
-  <xacro:macro name="robot_macro" params="base_link:='base_link' radius:=0.1001 effort_joint:=1000 small:=0.005 body_len:=0.0333333333333 load_inertia:=3.2e-07 velocity_joint:=300 damping1:=0.5 large:=100 inertia_link:=0.0015 mass_link:=0.005 inertia_rope2:=0.0 friction:=0.02 load_mass:=0.5 inertia_rope1:=1.55478395062e-07 box_param1:=0.25 spawn_point:=365.0 box_param:=0.0 mass_rope:=0.00166666666667 width_1:=0.00166666666667 k1:=10.0 k2:=100.0">
+  <xacro:macro name="robot_macro" params="base_link:='base_link' radius:=0.1001 effort_joint:=1 small:=0.005 body_len:=0.0666666666666 load_inertia:=3.2e-7 velocity_joint:=3000 damping1:=0.085 large:=100 inertia_link:=0.0015 mass_link:=0.005 inertia_rope2:=1.55478395062e-6 friction:=0.002 load_mass:=0.5 inertia_rope1:=1.55478395062e-5 box_param1:=0.25 spawn_point:=365.0 box_param:=0.0 mass_rope:=0.00166666666667 width_1:=0.00166666666667 k1:=1.01 k2:=1.01">
     <link name="rope_1">
       <visual>
@@ -197,10 +198,15 @@
       </inertial>
     </link>
+    <!--material name="Orange">
+      <color rgba="${255/255} ${108/255} ${10/255} 1.0"/>
+    </material-->
     <link name="load">
       <visual>
         <geometry>
-          <sphere radius="${radius}"/>
-        </geometry>
-        <origin rpy="0.0 0.0 0.0" xyz="0 0 ${-radius}"/>
+          <!--sphere radius="${radius}"/ -->
+          <mesh filename="package://mmuav_description/meshes/lupis_color.dae"
+            scale="0.0003 0.0003 0.0003" />
+        </geometry>
+        <origin rpy="${3.14159265358/2} ${-3.14159265358*0/2} ${-3.14159265358/2}" xyz="0.225 0 -0.03"/>
       </visual>
       <!--collision>
@@ -806,5 +812,5 @@
     </gazebo>
     <gazebo reference="load">
-      <material>Gazebo/Red</material>
+      <material>Gazebo/Green</material>
     </gazebo>
   </xacro:macro>

File: mmuav_description/urdf/rope_macro_dobar.xacro (robot description, xacro)
@@ -1,5 +1,6 @@
 <?xml version='1.0' encoding='utf-8'?>
+<!-- body len = 0.033333333333333 -->
 <robot xmlns:xacro="http://www.ros.org/wiki/xacro" name="myrobot">
-  <xacro:macro name="robot_macro" params="base_link:='base_link' radius:=0.1001 effort_joint:=1000 small:=0.005 body_len:=0.0333333333333 load_inertia:=3.2e-07 velocity_joint:=300 damping1:=0.5 large:=100 inertia_link:=0.0015 mass_link:=0.01 inertia_rope2:=0.0 friction:=0.02 load_mass:=0.5 inertia_rope1:=1.55478395062e-07 box_param1:=0.25 spawn_point:=365.0 box_param:=0.0 mass_rope:=0.00166666666667 width_1:=0.00166666666667 k1:=1.0 k2:=1.0">
+  <xacro:macro name="robot_macro" params="base_link:='base_link' radius:=0.1001 effort_joint:=1 small:=0.005 body_len:=0.0333333333333 load_inertia:=3.2e-7 velocity_joint:=3000 damping1:=0.085 large:=100 inertia_link:=0.0015 mass_link:=0.005 inertia_rope2:=1.55478395062e-6 friction:=0.002 load_mass:=0.5 inertia_rope1:=1.55478395062e-5 box_param1:=0.25 spawn_point:=365.0 box_param:=0.0 mass_rope:=0.00166666666667 width_1:=0.00166666666667 k1:=1.01 k2:=1.01">
     <link name="rope_1">
       <visual>
@@ -204,10 +205,10 @@
         <origin rpy="0.0 0.0 0.0" xyz="0 0 ${-radius}"/>
       </visual>
-      <collision>
+      <!--collision>
         <geometry>
           <sphere radius="${radius}"/>
         </geometry>
         <origin rpy="0.0 0.0 0.0" xyz="0 0 ${-radius}"/>
-      </collision>
+      </collision-->
       <inertial>
         <mass value="${load_mass}"/>
@@ -234,5 +235,5 @@
       <axis xyz="0 0 1"/>
       <dynamics damping="${damping1}" friction="0"/>
-      <limit effort="${effort_joint}" lower="${-k1*pi/2}" upper="${k1*pi/2}" velocity="${velocity_joint}"/>
+      <limit effort="${effort_joint}" lower="${-pi/2}" upper="${pi/2}" velocity="${velocity_joint}"/>
     </joint>
     <joint name="rope1Psi_to_rope1Theta" type="revolute">
@@ -241,5 +242,5 @@
       <axis xyz="0 1 0"/>
       <dynamics damping="${damping1}" friction="0"/>
-      <limit effort="${effort_joint}" lower="${-k1*pi/2}" upper="${k1*pi/2}" velocity="${velocity_joint}"/>
+      <limit effort="${effort_joint}" lower="${-pi/2}" upper="${pi/2}" velocity="${velocity_joint}"/>
     </joint>
     <joint name="rope1Theta_to_rope_1" type="revolute">
@@ -248,5 +249,5 @@
       <axis xyz="1 0 0"/>
       <dynamics damping="${damping1}" friction="0"/>
-      <limit effort="${effort_joint}" lower="${-k2*pi/16}" upper="${k2*pi/16}" velocity="${velocity_joint}"/>
+      <limit effort="${effort_joint}" lower="${-pi/16}" upper="${pi/16}" velocity="${velocity_joint}"/>
     </joint>
     <link name="rope2Theta">
@@ -744,5 +745,5 @@
       <axis xyz="0 0 1"/>
       <dynamics damping="${damping1}" friction="${friction}"/>
-      <limit effort="${effort_joint}" lower="${-k1*pi/2}" upper="${k1*pi/2}" velocity="${velocity_joint}"/>
+      <limit effort="${effort_joint}" lower="${-pi/2}" upper="${pi/2}" velocity="${velocity_joint}"/>
     </joint>
     <joint name="rope16Psi_to_rope16Theta" type="revolute">
@@ -751,5 +752,5 @@
       <axis xyz="0 1 0"/>
       <dynamics damping="${damping1}" friction="${friction}"/>
-      <limit effort="${effort_joint}" lower="${-k1*pi/2}" upper="${k1*pi/2}" velocity="${velocity_joint}"/>
+      <limit effort="${effort_joint}" lower="${-pi/2}" upper="${pi/2}" velocity="${velocity_joint}"/>
     </joint>
     <joint name="rope16Theta_to_load" type="revolute">
@@ -758,5 +759,5 @@
       <axis xyz="1 0 0"/>
       <dynamics damping="${damping1}" friction="${friction}"/>
-      <limit effort="${effort_joint}" lower="${-k2*pi/16}" upper="${k2*pi/16}" velocity="${velocity_joint}"/>
+      <limit effort="${effort_joint}" lower="${-pi/16}" upper="${pi/16}" velocity="${velocity_joint}"/>
     </joint>
     <gazebo reference="rope_1">
