Commit message: force sensor changes

File: mmuav_description/urdf/force_sensor.gazebo.xacro (robot description, xacro)
@@ -32,4 +32,6 @@
   <gazebo reference="joint_force_sensor_mount_top">
     <provideFeedback>true</provideFeedback>
+    <kp>1.0e+9</kp>
+    <kd>5.0e+5</kd>
   </gazebo>
   <!-- The ft_sensor plugin  -->
@@ -47,4 +49,9 @@
     </plugin>
   </gazebo>
+  <!--gazebo reference="link_force_sensor_top_mount">
+    <provideFeedback>true</provideFeedback>
+    <kp>1.0e+9</kp>
+    <kd>5.0e+5</kd>
+  </gazebo-->
   <gazebo reference="world">
     <dampingFactor>0.0002</dampingFactor>

File: mmuav_description/urdf/mmuav.base.urdf.xacro (robot description, xacro)
@@ -201,4 +201,34 @@
     joint_name="joint_gripper2_left">
   </xacro:transmisija>
+            <!-- delete afteR-->
+    <link name='link_screw'>
+      <inertial>
+        <mass value="0.5" />
+        <origin rpy="0 0 0" xyz="0.02100388 0.01819119 0.05027511"/>
+        <inertia
+          ixx="0.00020051" ixy="0" ixz="-0.00000019"
+          iyx="0" iyy="0.00020054" iyz="0.00000001"
+          izx="-0.00000019" izy="0.00000001" izz="0.00006377"/>
+      </inertial>
+      <visual>
+        <origin xyz="0 0 0" rpy="0 0 0" />
+        <geometry>
+          <mesh filename="package://mmuav_description/meshes/screw.dae"
+            scale="1 1 1" />
+        </geometry>
+      </visual>
+      <collision name='collision'>
+        <origin xyz="0 0 0" rpy="0 0 0"/>
+        <geometry>
+          <mesh filename="package://mmuav_description/meshes/screw.dae"
+            scale="1 1 1" />
+        </geometry>
+      </collision>
+    </link>
+    <joint name="joint_screw" type="fixed">
+        <origin xyz="0.023 0.006 0.0385" rpy="${PI} 0 ${PI/6}" />
+        <parent link="link_gripper2_left"/>
+        <child link="link_screw"/>
+    </joint>
   <!-- Camera properties -->
   <!--xacro:property name="camera_link" value="0.05" />

File: mmuav_description/urdf/mmuav.gazebo.xacro (robot description, xacro)
@@ -113,10 +113,10 @@
     odometry_sensor_suffix="3"
     child_frame_id="base"
-    parent_link="link_gripper2_right"
-    pose_topic="link_gripper2_right/pose"
-    pose_with_covariance_topic="link_gripper2_right/pose_with_covariance"
-    position_topic="link_gripper2_right/position"
-    transform_topic="link_gripper2_right/transform"
-    odometry_topic="link_gripper2_right/odometry"
+    parent_link="link_gripper1_left"
+    pose_topic="link_gripper1_left/pose"
+    pose_with_covariance_topic="link_gripper1_left/pose_with_covariance"
+    position_topic="link_gripper1_left/position"
+    transform_topic="link_gripper1_left/transform"
+    odometry_topic="link_gripper1_left/odometry"
     parent_frame_id="base_link"
     mass_odometry_sensor="0.01"
@@ -136,5 +136,5 @@
     image_scale="0.1">
     <inertia ixx="0.00001" ixy="0.0" ixz="0.0" iyy="0.00001" iyz="0.0" izz="0.00001" /> <!-- [kg m^2] [kg m^2] [kg m^2] [kg m^2] [kg m^2] [kg m^2] -->
-    <origin xyz="0.04903524 0.0 0" rpy="0.0 0.0 0.0" />
+    <origin xyz="0.01265 0.00104 -0.00134" rpy="0.0 0.0 0.0" />
   </xacro:odometry_plugin_macro>
   <gazebo reference="link_manipulator2uav_left">

File: mmuav_description/urdf/multirotor_base.urdf.xacro (robot description, xacro)
@@ -368,4 +368,11 @@
         </geometry>
       </visual>
+      <!--collision>
+        <origin xyz="0.02047 -0.00104 0.00135" rpy="0 0 0" />
+        <geometry>
+          <mesh filename="package://mmuav_description/meshes/gripper_part2.dae"
+            scale="1 1 1" />
+        </geometry>
+      </collision-->
     </link>
     <!--_____________________________________________________________-->
@@ -535,5 +542,5 @@
     <!--JOINT2 FIXED force_sensor_mount_top-->
     <!--_____________________________________________________________-->
-    <joint name="joint_force_sensor_mount_top" type="revolute">
+    <joint name="joint_force_sensor_mount_top" type="prismatic">
         <origin xyz="-0.01903 -0.05153 0.01661" rpy="${-PI/2} 0 0" />
         <parent link="link_force_sensor_bottom_mount"/>

Commit message: working force_sensr

File: mmuav_description/urdf/force_sensor.gazebo.xacro (robot description, xacro)
@@ -36,5 +36,5 @@
   <gazebo>
     <plugin name="ft_sensor" filename="libgazebo_ros_ft_sensor.so">
-      <updateRate>30.0</updateRate>
+      <updateRate>1000.0</updateRate>
       <robotNamespace>$(arg name)</robotNamespace>
       <topicName>ft_sensor_topic</topicName>
@@ -47,4 +47,7 @@
     </plugin>
   </gazebo>
+  <gazebo>
+    <plugin name="contact_sensor" filename="libcontact.so"/>
+  </gazebo>
   <gazebo reference="world">
     <dampingFactor>0.0002</dampingFactor>

File: mmuav_description/urdf/multirotor_base.urdf.xacro (robot description, xacro)
@@ -488,5 +488,5 @@
         </geometry>
       </visual>
-      <collision name='collision'>
+      <!--collision name='collision'>
         <origin xyz="0 0 0" rpy="0 0 0"/>
         <geometry>
@@ -494,5 +494,5 @@
             scale="1 1 1" />
         </geometry>
-      </collision>
+      </collision-->
     </link>
     <!--_____________________________________________________________-->

Commit message: m

File: mmuav_description/urdf/force_sensor.gazebo.xacro (robot description, xacro)
@@ -47,7 +47,4 @@
     </plugin>
   </gazebo>
-  <gazebo>
-    <plugin name="contact_sensor" filename="libcontact.so"/>
-  </gazebo>
   <gazebo reference="world">
     <dampingFactor>0.0002</dampingFactor>

File: mmuav_description/urdf/multirotor_base.urdf.xacro (robot description, xacro)
@@ -461,5 +461,5 @@
         </geometry>
       </visual>
-      <collision name='collision'>
+      <!--collision name='collision'>
         <origin xyz="0 0 0" rpy="0 0 0"/>
         <geometry>
@@ -467,5 +467,5 @@
             scale="1 1 1" />
         </geometry>
-      </collision>
+      </collision-->
     </link>
     <!--_____________________________________________________________-->
