Commit message: a

File: mmuav_description/urdf/force_sensor.base.urdf.xacro (robot description, xacro)
@@ -7,3 +7,8 @@
     <origin xyz="0 0 0.02" rpy="${PI/2} 0 0"/>
   </xacro:force_sensor>
+  <!--xacro:transmisija
+    trans_number="0"
+    mechanical_reduction = "1"
+    joint_name="joint_force_sensor_mount_top">
+  </xacro:transmisija-->
 </robot>

File: mmuav_description/urdf/force_sensor.gazebo.xacro (robot description, xacro)
@@ -32,11 +32,9 @@
   <gazebo reference="joint_force_sensor_mount_top">
     <provideFeedback>true</provideFeedback>
-    <kp>1.0e+9</kp>
-    <kd>5.0e+5</kd>
   </gazebo>
   <!-- The ft_sensor plugin  -->
   <gazebo>
     <plugin name="ft_sensor" filename="libgazebo_ros_ft_sensor.so">
-      <updateRate>100.0</updateRate>
+      <updateRate>30.0</updateRate>
       <robotNamespace>$(arg name)</robotNamespace>
       <topicName>ft_sensor_topic</topicName>
@@ -49,9 +47,4 @@
     </plugin>
   </gazebo>
-  <!--gazebo reference="link_force_sensor_top_mount">
-    <provideFeedback>true</provideFeedback>
-    <kp>1.0e+9</kp>
-    <kd>5.0e+5</kd>
-  </gazebo-->
   <gazebo reference="world">
     <dampingFactor>0.0002</dampingFactor>

File: mmuav_description/urdf/mmuav.base.urdf.xacro (robot description, xacro)
@@ -179,24 +179,30 @@
   <xacro:transmisija
     trans_number="0"
+    mechanical_reduction = "250"
     joint_name="joint_dynamixel1_left">
   </xacro:transmisija>
   <xacro:transmisija
     trans_number="1"
+    mechanical_reduction = "250"
     joint_name="joint_dynamixel2_left">
   </xacro:transmisija>
   <xacro:transmisija
     trans_number="2"
+    mechanical_reduction = "250"
     joint_name="joint_dynamixel1_right">
   </xacro:transmisija>
   <xacro:transmisija
     trans_number="3"
+    mechanical_reduction = "250"
     joint_name="joint_dynamixel2_right">
   </xacro:transmisija>
   <xacro:transmisija
     trans_number="4"
+    mechanical_reduction = "250"
     joint_name="joint_gripper2_right">
   </xacro:transmisija>
   <xacro:transmisija
     trans_number="5"
+    mechanical_reduction = "250"
     joint_name="joint_gripper2_left">
   </xacro:transmisija>

File: mmuav_description/urdf/multirotor_base.urdf.xacro (robot description, xacro)
@@ -114,5 +114,5 @@
   </xacro:macro>
   <!-- We add a <transmission> block for every joint that we wish to actuate. -->
-  <xacro:macro name="transmisija" params="trans_number joint_name">
+  <xacro:macro name="transmisija" params="trans_number mechanical_reduction joint_name">
     <transmission name="transmission_${trans_number}">
       <type>transmission_interface/SimpleTransmission</type>
@@ -122,5 +122,5 @@
       <actuator name="motor_${trans_number}">
         <hardwareInterface>hardware_interface/EffortJointInterface</hardwareInterface>
-        <mechanicalReduction>1</mechanicalReduction>
+        <mechanicalReduction>${mechanical_reduction}</mechanicalReduction>
       </actuator>
     </transmission>
@@ -448,5 +448,5 @@
       <inertial>
         <mass value="2.0" />
-        <origin rpy="0 0 0" xyz="0.38508257 0.46818651 1.04028639"/>
+        <origin rpy="0 0 0" xyz="0 0.46818651 0"/>
         <inertia
           ixx="0.23434322" ixy="0" ixz="0.0"
@@ -502,5 +502,5 @@
       <inertial>
         <mass value="0.080" />
-        <origin rpy="0 0 0" xyz="0.01903151 0.01661061 0.02154592"/>
+        <origin rpy="0 0 0" xyz="0 0 -0.02998408"/>
         <inertia
           ixx="0.00059994" ixy="0" ixz="0.0"
@@ -508,6 +508,7 @@
           izx="0.0" izy="0" izz="0.00119615"/>
       </inertial>
-      <visual>
-        <origin xyz="0 0 0" rpy="0 0 0" />
+      <!--0.01903151 0.01661061 0.02154592-->
+      <visual>
+        <origin xyz="-0.01903 -0.01661 -0.05153" rpy="0 0 0" />
         <geometry>
           <mesh filename="package://mmuav_description/meshes/forcesensor_mount_top.dae"
@@ -516,5 +517,5 @@
       </visual>
       <collision name='collision'>
-        <origin xyz="0 0 0" rpy="0 0 0"/>
+        <origin xyz="-0.01903 -0.01661 -0.05153" rpy="0 0 0"/>
         <geometry>
           <mesh filename="package://mmuav_description/meshes/forcesensor_mount_top.dae"
@@ -543,5 +544,5 @@
     <!--_____________________________________________________________-->
     <joint name="joint_force_sensor_mount_top" type="prismatic">
-        <origin xyz="-0.01903 -0.05153 0.01661" rpy="${-PI/2} 0 0" />
+        <origin xyz="0 0 0" rpy="${-PI/2} 0 0" />
         <parent link="link_force_sensor_bottom_mount"/>
         <child link="link_force_sensor_top_mount"/>

Commit message: added impedance_control

File: mmuav_description/urdf/force_sensor.base.urdf.xacro (robot description, xacro)
@@ -7,8 +7,3 @@
     <origin xyz="0 0 0.02" rpy="${PI/2} 0 0"/>
   </xacro:force_sensor>
-  <!--xacro:transmisija
-    trans_number="0"
-    mechanical_reduction = "1"
-    joint_name="joint_force_sensor_mount_top">
-  </xacro:transmisija-->
 </robot>

File: mmuav_description/urdf/force_sensor.gazebo.xacro (robot description, xacro)
@@ -27,8 +27,14 @@
   <gazebo reference="link_force_sensor_top_mount">
     <gravity>true</gravity>
-    <self_collide>false</self_collide>
+    <self_collide>true</self_collide>
+    <mu1>0</mu1>
+    <mu2>0</mu2>
+    <fdir1 value = "1 0 0"/>
   </gazebo>
   <!-- Enable the Joint Feedback -->
   <gazebo reference="joint_force_sensor_mount_top">
+    <stopCfm>0.08</stopCfm>
+    <stopErp>0.2</stopErp>
+    <implicitSpringDamper>true</implicitSpringDamper>
     <provideFeedback>true</provideFeedback>
   </gazebo>

File: mmuav_description/urdf/mmuav.base.urdf.xacro (robot description, xacro)
@@ -65,5 +65,5 @@
     ixy="0.0" ixz="0.0"  iyz="0.0" /> <!-- [kg*m^2] [kg*m^2] [kg*m^2] [kg*m^2] [kg*m^2] [kg*m^2] -->
   </xacro:property>
-  <xacro:landing_gear
+  <!--xacro:landing_gear
       parent="base_link"
       gear_num = "1"
@@ -84,5 +84,5 @@
       <origin xyz="0 0.325 -0.075" rpy="0 0 0" />
       <xacro:insert_block name="land_gear_inertia"/>
-  </xacro:landing_gear>
+  </xacro:landing_gear-->
   <!-- Instantiate rotors -->
   <xacro:vertical_rotor
@@ -210,5 +210,5 @@
     <link name='link_screw'>
       <inertial>
-        <mass value="0.5" />
+        <mass value="0.05" />
         <origin rpy="0 0 0" xyz="0.02100388 0.01819119 0.05027511"/>
         <inertia
@@ -233,6 +233,6 @@
     </link>
     <joint name="joint_screw" type="fixed">
-        <origin xyz="0.023 0.006 0.0385" rpy="${PI} 0 ${PI/6}" />
-        <parent link="link_gripper2_left"/>
+        <origin xyz="-0.03100388 0.00719119 -0.03527511" rpy="${PI} 0 ${PI/6}" />
+        <parent link="base_link"/>
         <child link="link_screw"/>
     </joint>

File: mmuav_description/urdf/mmuav.gazebo.xacro (robot description, xacro)
@@ -209,3 +209,10 @@
     <dampingFactor>0.0002</dampingFactor>
   </gazebo>
+  <gazebo reference="link_screw">
+    <gravity>true</gravity>
+    <self_collide>true</self_collide>
+    <mu1>0</mu1>
+    <mu2>0</mu2>
+    <fdir1 value = "1 0 0"/>
+  </gazebo>
 </robot>
