Commit message: added actuator on passive joint

File: mmuav_description/urdf/mmuav.base.urdf.xacro (robot description, xacro)
@@ -166,9 +166,17 @@
   <xacro:transmisija
     trans_number="2"
+    joint_name="joint_q3_passive_left">
+  </xacro:transmisija>
+  <xacro:transmisija
+    trans_number="3"
     joint_name="joint_q1_right">
   </xacro:transmisija>
   <xacro:transmisija
-    trans_number="3"
+    trans_number="4"
     joint_name="joint_q2_right">
   </xacro:transmisija>
+    <xacro:transmisija
+    trans_number="5"
+    joint_name="joint_q3_passive_right">
+  </xacro:transmisija>
 </robot>

File: mmuav_description/urdf/multirotor_base.urdf.xacro (robot description, xacro)
@@ -374,5 +374,4 @@
       <limit upper="1.57" lower="-1.57" effort="10" velocity="1"/>
       <axis xyz="0 1 0" />
-      <dynamics damping="0.0" friction="0.04"/>
     </joint>
   </xacro:macro>

Commit message: added mmc arducopter

File: mmuav_description/urdf/mmuav.base.urdf.xacro (robot description, xacro)
@@ -58,4 +58,5 @@
     body_height="${body_height}"
     mesh_file="${body_mesh_file}">
+    <origin xyz="0 0 0" rpy="0 0 0"/>
     <xacro:insert_block name="body_inertia" />
   </xacro:multirotor_base_macro>

File: mmuav_description/urdf/multirotor_base.urdf.xacro (robot description, xacro)
@@ -3,8 +3,8 @@
   <!-- Main multirotor link -->
   <xacro:macro name="multirotor_base_macro"
-    params="robot_namespace mass body_width body_height mesh_file *inertia">
+    params="robot_namespace mass body_width body_height mesh_file *origin *inertia">
     <link name="base_link"></link>
     <joint name="base_joint" type="fixed">
-      <origin xyz="0 0 0" rpy="0 0 0" />
+      <xacro:insert_block name="origin"/>
       <parent link="base_link" />
       <child link="base_link_inertia" />
@@ -24,12 +24,12 @@
         </geometry>
       </visual>
-      <!--collision>
-        <origin xyz="0 0 0" rpy="0 0 0" />
-        <geometry>
-          <mesh filename="package://mmuav_description/meshes/${mesh_file}"
-            scale="1 1 1" />
+      <collision>
+        <origin xyz="0 0 0" rpy="0 0 0" />
+        <geometry>
+          <!--mesh filename="package://mmuav_description/meshes/${mesh_file}"
+            scale="1 1 1" /-->
           <box size="${body_width} ${body_width} ${body_height}" />
         </geometry>
-      </collision-->
+      </collision>
     </link>
     <!-- IMU -->
@@ -376,3 +376,36 @@
     </joint>
   </xacro:macro>
+  <!-- Definition of movable mass macro -->
+  <xacro:macro name="movable_mass" params="mass_number parent mass dimension path_len color x_axis y_axis z_axis orientation *origin *inertia">
+    <joint name="stick_to_movable_mass_${mass_number}" type="prismatic">
+      <xacro:insert_block name="origin"/>
+      <axis xyz="${x_axis} ${y_axis} ${z_axis}"/>
+      <parent link="${parent}"/>
+      <child link="movable_mass_${mass_number}"/>
+      <limit lower="${-path_len/2}" upper="${path_len/2}" effort="10000" velocity="20"/>
+      <dynamics damping="10" />
+    </joint>
+    <link name="movable_mass_${mass_number}">
+      <visual>
+        <origin rpy="0 0 ${orientation}" xyz="0 0 ${0*dimension/2}"/>
+        <geometry>
+          <box size="${1*dimension} ${1*dimension} ${1*dimension}"/>
+        </geometry>
+      </visual>
+      <collision>
+        <origin rpy="0 0 0" xyz="0 0 ${0*dimension/2}"/>
+        <geometry>
+          <box size="${1*dimension} ${1*dimension} ${1*dimension}"/>
+        </geometry>
+      </collision>
+      <inertial>
+        <origin rpy="0 0 0" xyz="0 0 ${0*dimension/2}"/>
+        <mass value="${mass}"/>
+        <xacro:insert_block name="inertia"/>
+      </inertial>
+    </link>
+    <gazebo reference="movable_mass_${mass_number}">
+      <material>Gazebo/${color}</material>
+    </gazebo>
+  </xacro:macro>
 </robot>

Commit message: Changed mmuav to + configuration.

File: mmuav_description/urdf/mmuav.base.urdf.xacro (robot description, xacro)
@@ -58,5 +58,5 @@
     body_height="${body_height}"
     mesh_file="${body_mesh_file}">
-    <origin xyz="0 0 0" rpy="0 0 0"/>
+    <origin xyz="0 0 0" rpy="0 0 ${-PI/4}"/>
     <xacro:insert_block name="body_inertia" />
   </xacro:multirotor_base_macro>
@@ -77,5 +77,5 @@
     rolling_moment_coefficient="${rolling_moment_coefficient}"
     color="Red">
-    <origin xyz="${cos45*arm_length} ${sin45*arm_length} ${rotor_offset_top}" rpy="0 0 0" />
+    <origin xyz="${1*arm_length} ${0*arm_length} ${rotor_offset_top}" rpy="0 0 0" />
     <xacro:insert_block name="rotor_inertia" />
   </xacro:vertical_rotor>
@@ -94,6 +94,6 @@
     rotor_drag_coefficient="${rotor_drag_coefficient}"
     rolling_moment_coefficient="${rolling_moment_coefficient}"
-    color="Red">
-    <origin xyz="${cos45*arm_length} ${-sin45*arm_length} ${rotor_offset_top}" rpy="0 0 0" />
+    color="Blue">
+    <origin xyz="${0*arm_length} ${1*arm_length} ${rotor_offset_top}" rpy="0 0 0" />
     <xacro:insert_block name="rotor_inertia" />
   </xacro:vertical_rotor>
@@ -112,6 +112,6 @@
     rotor_drag_coefficient="${rotor_drag_coefficient}"
     rolling_moment_coefficient="${rolling_moment_coefficient}"
-    color="Blue">
-    <origin xyz="${-cos45*arm_length} ${sin45*arm_length} ${rotor_offset_top}" rpy="0 0 0" />
+    color="Red">
+    <origin xyz="${-1*arm_length} ${0*arm_length} ${rotor_offset_top}" rpy="0 0 0" />
     <xacro:insert_block name="rotor_inertia" />
   </xacro:vertical_rotor>
@@ -131,5 +131,5 @@
     rolling_moment_coefficient="${rolling_moment_coefficient}"
     color="Blue">
-    <origin xyz="${-cos45*arm_length} ${-sin45*arm_length} ${rotor_offset_top}" rpy="0 0 0" />
+    <origin xyz="${0*arm_length} ${-1*arm_length} ${rotor_offset_top}" rpy="0 0 0" />
     <xacro:insert_block name="rotor_inertia" />
   </xacro:vertical_rotor>
@@ -143,5 +143,6 @@
     suffix="left">
     <axis xyz="0 1 0" />
-    <origin xyz="-0.11188 0.11206 -0.07349" rpy="-1.57079632679 0 0"/>
+    <!-- origin xyz="${-0.11188*sin45} ${0.11206*cos45} -0.07349" rpy="-1.57079632679 0 0"/ -->
+    <origin xyz="0 0.158342 -0.07349" rpy="-1.57079632679 0 0"/>
   </xacro:manipulator>
      <!-- Adding right manipulator -->
@@ -154,5 +155,6 @@
     suffix="right">
     <axis xyz="0 1 0" />
-    <origin xyz="0.11205 -0.11188 -0.07349" rpy="-1.57079632679 0 0"/>
+    <!--origin xyz="${0.11205**sin45} ${-0.11188*cos45} -0.07349" rpy="-1.57079632679 0 0"/ -->
+    <origin xyz="0 -0.158342 -0.07349" rpy="-1.57079632679 0 0"/>
   </xacro:manipulator>
   <!-- Add transmission for joints-->
@@ -177,5 +179,5 @@
     joint_name="joint_q2_right">
   </xacro:transmisija>
-    <xacro:transmisija
+  <xacro:transmisija
     trans_number="5"
     joint_name="joint_q3_passive_right">

Commit message: Added working version for mmuav simulator, Dynamixel pid tuning needed!

File: mmuav_description/urdf/mmuav.base.urdf.xacro (robot description, xacro)
@@ -167,8 +167,8 @@
     joint_name="joint_q2_left">
   </xacro:transmisija>
-  <xacro:transmisija
+  <!--xacro:transmisija
     trans_number="2"
     joint_name="joint_q3_passive_left">
-  </xacro:transmisija>
+  </xacro:transmisija -->
   <xacro:transmisija
     trans_number="3"
@@ -179,7 +179,7 @@
     joint_name="joint_q2_right">
   </xacro:transmisija>
-  <xacro:transmisija
+  <!--xacro:transmisija
     trans_number="5"
     joint_name="joint_q3_passive_right">
-  </xacro:transmisija>
+  </xacro:transmisija-->
 </robot>

File: mmuav_description/urdf/mmuav.gazebo.xacro (robot description, xacro)
@@ -68,3 +68,25 @@
     <origin xyz="-0.0 0.0 0" rpy="0.0 0.0 0.0" />
   </xacro:odometry_plugin_macro>
+  <gazebo>
+    <plugin name="dipole_magnet" filename="libstorm_gazebo_dipole_magnet.so">
+        <bodyName>link_gripper2_left</bodyName>
+        <dipole_moment>1 0 1</dipole_moment>
+        <gain>1</gain> <!-- Magnet gain, additional param that controls the overal magnet moment. Gain can be changed online through ros topic-->
+        <!-- Set to 0 if not using ROS -->
+        <shouldPublish>1</shouldPublish>
+        <topicNs>magnet_left</topicNs>
+        <updateRate>100</updateRate>
+    </plugin>
+  </gazebo>
+  <gazebo>
+    <plugin name="dipole_magnet" filename="libstorm_gazebo_dipole_magnet.so">
+        <bodyName>link_gripper2_right</bodyName>
+        <dipole_moment>1 0 1</dipole_moment>
+        <gain>1</gain> <!-- Magnet gain, additional param that controls the overal magnet moment. Gain can be changed online through ros topic-->
+        <!-- Set to 0 if not using ROS -->
+        <shouldPublish>1</shouldPublish>
+        <topicNs>magnet_right</topicNs>
+        <updateRate>100</updateRate>
+    </plugin>
+  </gazebo>
 </robot>

File: mmuav_description/urdf/multirotor_base.urdf.xacro (robot description, xacro)
@@ -213,12 +213,12 @@
         </geometry>
       </visual>
-      <collision name='collision'>
+      <!--collision name='collision'>
         <origin xyz="0.01261097 0 0.00120978" rpy="0 0 0"/>
         <geometry>
-          <!--mesh filename="package://mmuav_description/meshes/AX12.dae"
-            scale="1 1 1" /-->
-           <box size="0.05 0.041 0.032"/>
-        </geometry>
-      </collision>
+          <mesh filename="package://mmuav_description/meshes/AX12.dae"
+            scale="1 1 1" />
+           <box size="0.05 0.041 0.032" scale="0.01 0.01 0.01"/>
+        </geometry>
+      </collision-->
     </link>
     <!--_____________________________________________________________-->
@@ -281,12 +281,12 @@
         </geometry>
       </visual>
-      <collision name='collision'>
+      <!-- collision name='collision'>
         <origin xyz="0.01261097 0 0.00120978" rpy="0 0 0"/>
         <geometry>
-          <!--mesh filename="package://mmuav_description/meshes/AX12.dae"
-            scale="1 1 1" /-->
-           <box size="0.05 0.041 0.032"/>
-        </geometry>
-      </collision>
+          <mesh filename="package://mmuav_description/meshes/AX12.dae"
+            scale="1 1 1" />
+           <box size="0.05 0.041 0.032" scale="0.01 0.01 0.01"/>
+        </geometry>
+      </collision-->
     </link>
     <!--_____________________________________________________________-->
@@ -315,27 +315,35 @@
     <link name='link_gripper2_${suffix}'>
       <inertial>
-        <mass value="0.01" />
-        <origin xyz="0.02116183 0 0" rpy="1.57079632679 0 0"/>
-        <inertia
+        <mass value="0.5" />
+        <!-- origin xyz="0.02116183 0 0" rpy="1.57079632679 0 0"/ -->
+        <origin xyz="0.08 0 0" rpy="0 0 0"/>
+        <!--inertia
           ixx="0.00000124"
           iyy="0.00000161"
           izz="0.00000270"
+          ixy="0.0" ixz="0.0" iyz="0.0" / -->
+        <inertia
+          ixx="0.00015"
+          iyy="0.00015"
+          izz="0.00015"
           ixy="0.0" ixz="0.0" iyz="0.0" />
       </inertial>
       <visual>
-        <origin xyz="0.02047 -0.00104 -0.00134" rpy="0 0 0" />
+        <!-- origin xyz="0.02047 -0.00104 -0.00134" rpy="0 0 0" / -->
+        <origin xyz="0.08 0.0 0.0" rpy="0 0 0" />
+        <geometry>
+          <!--mesh filename="package://mmuav_description/meshes/gripper_part2.dae"
+            scale="0.1 0.1 0.1" / -->
+           <sphere radius="0.015"/>
+        </geometry>
+      </visual>
+      <!--collision name='collision'>
+        <origin xyz="0.02047 -0.00104 -0.00134" rpy="0 0 0"/>
         <geometry>
           <mesh filename="package://mmuav_description/meshes/gripper_part2.dae"
-            scale="1 1 1" />
-        </geometry>
-      </visual>
-      <collision name='collision'>
-        <origin xyz="0.02047 -0.00104 -0.00134" rpy="0 0 0"/>
-        <geometry>
-          <mesh filename="package://mmuav_description/meshes/gripper_part2.dae"
-            scale="1 1 1" />
-           <!--box size="0.05 0.041 0.032"/-->
-        </geometry>
-      </collision>
+            scale="0.1 0.1 0.1" />
+           <box size="0.05 0.041 0.032"/>
+        </geometry>
+      </collision-->
     </link>
     <joint name="joint_q1_${suffix}" type="revolute">
@@ -343,5 +351,5 @@
       <child link="dynamixel_1_${suffix}" />
       <xacro:insert_block name="origin"/>
-      <limit upper="3.14" lower="-3.14" effort="10" velocity="1"/>
+      <limit upper="3.14" lower="-3.14" effort="200" velocity="5"/>
       <xacro:insert_block name="axis"/>
     </joint>
@@ -360,5 +368,5 @@
       <child link="dynamixel_2_${suffix}" />
       <origin xyz="0 0 0" rpy="0 0 0"/>
-      <limit upper="3.14" lower="-3.14" effort="10" velocity="1"/>
+      <limit upper="3.14" lower="-3.14" effort="200" velocity="5"/>
       <axis xyz="0 1 0" />
     </joint>
@@ -372,5 +380,5 @@
       <child link="link_gripper2_${suffix}" />
       <origin xyz="0.01265148 0.00103883 0.00134042" rpy="0 0 0"/>
-      <limit upper="1.57" lower="-1.57" effort="10" velocity="1"/>
+      <limit upper="1.57" lower="-1.57" effort="2" velocity="1.47"/>
       <axis xyz="0 1 0" />
     </joint>

Commit message: Mmuav stabilizes for small arms gains.

File: mmuav_description/urdf/mmuav.base.urdf.xacro (robot description, xacro)
@@ -15,5 +15,6 @@
   <xacro:property name="time_constant" value="0.0125" /> <!-- [s] -->
   <xacro:property name="max_rot_velocity" value="1475" /> <!-- [rad/s] -->
-  <xacro:property name="rotor_drag_coefficient" value="8.06428e-05" />
+  <!--xacro:property name="rotor_drag_coefficient" value="8.06428e-05" /-->
+  <xacro:property name="rotor_drag_coefficient" value="8.06428e-06" />
   <xacro:property name="rolling_moment_coefficient" value="0.000001" />
   <xacro:property name="imu_mass" value="0.02"/>
@@ -61,4 +62,31 @@
     <xacro:insert_block name="body_inertia" />
   </xacro:multirotor_base_macro>
+  <xacro:property name="land_gear_inertia">
+    <inertia
+    ixx="1e-6"
+    iyy="1e-6"
+    izz="1e-6"
+    ixy="0.0" ixz="0.0"  iyz="0.0" /> <!-- [kg*m^2] [kg*m^2] [kg*m^2] [kg*m^2] [kg*m^2] [kg*m^2] -->
+  </xacro:property>
+  <xacro:landing_gear
+      parent="base_link"
+      gear_num = "1"
+      mass = "1e-6"
+      dim_x = "0.8"
+      dim_y = "0.1"
+      dim_z = "0.05">
+      <origin xyz="0 -0.325 -0.1" rpy="0 0 0" />
+      <xacro:insert_block name="land_gear_inertia"/>
+  </xacro:landing_gear>
+  <xacro:landing_gear
+      parent="base_link"
+      gear_num = "2"
+      mass = "1e-6"
+      dim_x = "0.8"
+      dim_y = "0.1"
+      dim_z = "0.05">
+      <origin xyz="0 0.325 -0.1" rpy="0 0 0" />
+      <xacro:insert_block name="land_gear_inertia"/>
+  </xacro:landing_gear>
   <!-- Instantiate rotors -->
   <xacro:vertical_rotor
@@ -164,22 +192,22 @@
   </xacro:transmisija>
   <xacro:transmisija
+    trans_number="3"
+    joint_name="joint_q1_right">
+  </xacro:transmisija>
+  <xacro:transmisija
     trans_number="1"
     joint_name="joint_q2_left">
   </xacro:transmisija>
-  <!--xacro:transmisija
-    trans_number="2"
-    joint_name="joint_q3_passive_left">
-  </xacro:transmisija -->
-  <xacro:transmisija
-    trans_number="3"
-    joint_name="joint_q1_right">
-  </xacro:transmisija>
   <xacro:transmisija
     trans_number="4"
     joint_name="joint_q2_right">
   </xacro:transmisija>
-  <!--xacro:transmisija
+  <xacro:transmisija
     trans_number="5"
+    joint_name="joint_q3_passive_left">
+  </xacro:transmisija >
+  <xacro:transmisija
+    trans_number="6"
     joint_name="joint_q3_passive_right">
-  </xacro:transmisija-->
+  </xacro:transmisija>
 </robot>

File: mmuav_description/urdf/mmuav.gazebo.xacro (robot description, xacro)
@@ -68,25 +68,14 @@
     <origin xyz="-0.0 0.0 0" rpy="0.0 0.0 0.0" />
   </xacro:odometry_plugin_macro>
-  <gazebo>
+  <!--gazebo>
     <plugin name="dipole_magnet" filename="libstorm_gazebo_dipole_magnet.so">
         <bodyName>link_gripper2_left</bodyName>
         <dipole_moment>1 0 1</dipole_moment>
-        <gain>1</gain> <!-- Magnet gain, additional param that controls the overal magnet moment. Gain can be changed online through ros topic-->
+        <gain>1</gain--> <!-- Magnet gain, additional param that controls the overal magnet moment. Gain can be changed online through ros topic-->
         <!-- Set to 0 if not using ROS -->
-        <shouldPublish>1</shouldPublish>
+        <!--houldPublish>1</shouldPublish>
         <topicNs>magnet_left</topicNs>
         <updateRate>100</updateRate>
     </plugin>
-  </gazebo>
-  <gazebo>
-    <plugin name="dipole_magnet" filename="libstorm_gazebo_dipole_magnet.so">
-        <bodyName>link_gripper2_right</bodyName>
-        <dipole_moment>1 0 1</dipole_moment>
-        <gain>1</gain> <!-- Magnet gain, additional param that controls the overal magnet moment. Gain can be changed online through ros topic-->
-        <!-- Set to 0 if not using ROS -->
-        <shouldPublish>1</shouldPublish>
-        <topicNs>magnet_right</topicNs>
-        <updateRate>100</updateRate>
-    </plugin>
-  </gazebo>
+  </gazebo-->
 </robot>

File: mmuav_description/urdf/multirotor_base.urdf.xacro (robot description, xacro)
@@ -24,12 +24,12 @@
         </geometry>
       </visual>
-      <collision>
-        <origin xyz="0 0 0" rpy="0 0 0" />
-        <geometry>
-          <!--mesh filename="package://mmuav_description/meshes/${mesh_file}"
-            scale="1 1 1" /-->
+      <!--collision>
+        <origin xyz="0 0 0" rpy="0 0 0" />
+        <geometry>
+          <mesh filename="package://mmuav_description/meshes/${mesh_file}"
+            scale="1 1 1" />
           <box size="${body_width} ${body_width} ${body_height}" />
         </geometry>
-      </collision>
+      </collision-->
     </link>
     <!-- IMU -->
@@ -121,7 +121,34 @@
       <actuator name="motor_${trans_number}">
         <hardwareInterface>hardware_interface/EffortActuatorInterface</hardwareInterface>
-        <mechanicalReduction>100</mechanicalReduction>
+        <mechanicalReduction>1</mechanicalReduction>
       </actuator>
     </transmission>
+  </xacro:macro>
+  <xacro:macro name="landing_gear" params="gear_num parent mass dim_x dim_y dim_z *origin *inertia">
+    <joint name="land_gear_${gear_num}" type="fixed">
+      <xacro:insert_block name="origin"/>
+      <axis xyz="0 0 1"/>
+      <parent link="${parent}"/>
+      <child link="land_gear_${gear_num}"/>
+    </joint>
+    <link name="land_gear_${gear_num}">
+      <visual>
+        <origin rpy="0 0 0" xyz="0 0 0"/>
+        <geometry>
+          <box size="0.01 0.01 0.0001"/>
+        </geometry>
+      </visual>
+      <collision>
+        <origin rpy="0 0 0" xyz="0 0 0"/>
+        <geometry>
+          <box size="${dim_x} ${dim_y} ${dim_z}"/>
+        </geometry>
+      </collision>
+      <inertial>
+         <origin rpy="0 0 0" xyz="0 0 0"/>
+        <mass value="${mass}"/>
+        <xacro:insert_block name="inertia"/>
+      </inertial>
+    </link>
   </xacro:macro>
    <!-- camera -->
@@ -315,7 +342,7 @@
     <link name='link_gripper2_${suffix}'>
       <inertial>
-        <mass value="0.5" />
+        <mass value="0.25" />
         <!-- origin xyz="0.02116183 0 0" rpy="1.57079632679 0 0"/ -->
-        <origin xyz="0.08 0 0" rpy="0 0 0"/>
+        <origin xyz="0.04 0 0" rpy="0 0 0"/>
         <!--inertia
           ixx="0.00000124"
@@ -347,10 +374,11 @@
       </collision-->
     </link>
-    <joint name="joint_q1_${suffix}" type="revolute">
+    <joint name="joint_q1_${suffix}" type="continuous">
       <parent link="${parent}"/>
       <child link="dynamixel_1_${suffix}" />
       <xacro:insert_block name="origin"/>
-      <limit upper="3.14" lower="-3.14" effort="200" velocity="5"/>
+      <limit upper="3.14" lower="-3.14" effort="400" velocity="1"/>
       <xacro:insert_block name="axis"/>
+      <dynamics damping="0.07" friction="0.0"/>
     </joint>
     <joint name="Dynamixel1ToF3_${suffix}" type="fixed">
@@ -364,10 +392,11 @@
         <child link="link_F4_fixed_${suffix}"/>
     </joint>
-    <joint name="joint_q2_${suffix}" type="revolute">
+    <joint name="joint_q2_${suffix}" type="continuous">
       <parent link="link_F4_fixed_${suffix}"/>
       <child link="dynamixel_2_${suffix}" />
       <origin xyz="0 0 0" rpy="0 0 0"/>
-      <limit upper="3.14" lower="-3.14" effort="200" velocity="5"/>
+      <limit upper="3.14" lower="-3.14" effort="200" velocity="1"/>
       <axis xyz="0 1 0" />
+      <dynamics damping="0.07" friction="0.0"/>
     </joint>
     <joint name="Dynamixel2ToGripper_${suffix}" type="fixed">
@@ -376,10 +405,12 @@
         <child link="link_gripper1_${suffix}"/>
     </joint>
-    <joint name="joint_q3_passive_${suffix}" type="revolute">
+    <joint name="joint_q3_passive_${suffix}" type="continuous">
       <parent link="link_gripper1_${suffix}"/>
       <child link="link_gripper2_${suffix}" />
       <origin xyz="0.01265148 0.00103883 0.00134042" rpy="0 0 0"/>
-      <limit upper="1.57" lower="-1.57" effort="2" velocity="1.47"/>
+      <limit upper="3.14" lower="-3.14" effort="20" velocity="1"/>
       <axis xyz="0 1 0" />
+      <dynamics damping="0.07" friction="0.0"/>
+      <!--dynamics damping="0.4" friction="0.04"/-->
     </joint>
   </xacro:macro>
