Commit message: Simulation working, inverse still needs tweaking.

File: mmuav_description/urdf/mmuav.base.urdf.xacro (robot description, xacro)
@@ -13,8 +13,9 @@
   <xacro:property name="motor_constant" value="8.54858e-06" /> <!-- [kg*m/s^2] -->
   <xacro:property name="moment_constant" value="0.016" /> <!-- [m] -->
-  <xacro:property name="time_constant" value="0.0125" /> <!-- [s] -->
+  <xacro:property name="time_constant_up" value="0.0125" /> <!-- [s] -->
+  <xacro:property name="time_constant_down" value="0.025" /> <!-- [s] -->
   <xacro:property name="max_rot_velocity" value="1475" /> <!-- [rad/s] -->
   <!--xacro:property name="rotor_drag_coefficient" value="8.06428e-05" /-->
-  <xacro:property name="rotor_drag_coefficient" value="8.06428e-06" />
+  <xacro:property name="rotor_drag_coefficient" value="8.06428e-05" />
   <xacro:property name="rolling_moment_coefficient" value="0.000001" />
   <xacro:property name="imu_mass" value="0.02"/>
@@ -99,5 +100,6 @@
     mass_rotor="${mass_rotor}"
     radius_rotor="${radius_rotor}"
-    time_constant="${time_constant}"
+    time_constant_up="${time_constant_up}"
+    time_constant_down="${time_constant_down}"
     max_rot_velocity="${max_rot_velocity}"
     motor_number="0"
@@ -117,5 +119,6 @@
     mass_rotor="${mass_rotor}"
     radius_rotor="${radius_rotor}"
-    time_constant="${time_constant}"
+    time_constant_up="${time_constant_up}"
+    time_constant_down="${time_constant_down}"
     max_rot_velocity="${max_rot_velocity}"
     motor_number="1"
@@ -129,11 +132,12 @@
     robot_namespace="$(arg name)"
     suffix="back_left"
-    direction="ccw"
-    motor_constant="${motor_constant}"
-    moment_constant="${moment_constant}"
-    parent="base_link"
-    mass_rotor="${mass_rotor}"
-    radius_rotor="${radius_rotor}"
-    time_constant="${time_constant}"
+    direction="cw"
+    motor_constant="${motor_constant}"
+    moment_constant="${moment_constant}"
+    parent="base_link"
+    mass_rotor="${mass_rotor}"
+    radius_rotor="${radius_rotor}"
+    time_constant_up="${time_constant_up}"
+    time_constant_down="${time_constant_down}"
     max_rot_velocity="${max_rot_velocity}"
     motor_number="2"
@@ -147,11 +151,12 @@
     robot_namespace="$(arg name)"
     suffix="back_right"
-    direction="cw"
-    motor_constant="${motor_constant}"
-    moment_constant="${moment_constant}"
-    parent="base_link"
-    mass_rotor="${mass_rotor}"
-    radius_rotor="${radius_rotor}"
-    time_constant="${time_constant}"
+    direction="ccw"
+    motor_constant="${motor_constant}"
+    moment_constant="${moment_constant}"
+    parent="base_link"
+    mass_rotor="${mass_rotor}"
+    radius_rotor="${radius_rotor}"
+    time_constant_up="${time_constant_up}"
+    time_constant_down="${time_constant_down}"
     max_rot_velocity="${max_rot_velocity}"
     motor_number="3"

File: mmuav_description/urdf/mmuav.gazebo.xacro (robot description, xacro)
@@ -138,3 +138,6 @@
     <origin xyz="-0.0 0.0 0" rpy="0.0 0.0 0.0" />
   </xacro:odometry_plugin_macro>
+  <gazebo reference="base_link">
+    <dampingFactor>0.0002</dampingFactor>
+  </gazebo>
 </robot>

File: mmuav_description/urdf/multirotor_base.urdf.xacro (robot description, xacro)
@@ -60,5 +60,5 @@
   <!-- Rotor joint and link -->
   <xacro:macro name="vertical_rotor"
-    params="robot_namespace suffix direction motor_constant moment_constant parent mass_rotor radius_rotor time_constant max_rot_velocity motor_number rotor_drag_coefficient rolling_moment_coefficient color *origin *inertia">
+    params="robot_namespace suffix direction motor_constant moment_constant parent mass_rotor radius_rotor time_constant_up time_constant_down max_rot_velocity motor_number rotor_drag_coefficient rolling_moment_coefficient color *origin *inertia">
     <joint name="rotor_${motor_number}_joint" type="continuous">
       <xacro:insert_block name="origin" />
@@ -96,5 +96,6 @@
         <linkName>rotor_${motor_number}</linkName>
         <turningDirection>${direction}</turningDirection>
-        <timeConstant>${time_constant}</timeConstant>
+        <timeConstantUp>${time_constant_up}</timeConstantUp>
+        <timeConstantDown>${time_constant_down}</timeConstantDown>
         <maxRotVelocity>${max_rot_velocity}</maxRotVelocity>
         <motorConstant>${motor_constant}</motorConstant>
@@ -378,5 +379,5 @@
       <child link="dynamixel_1_${suffix}" />
       <xacro:insert_block name="origin"/>
-      <limit upper="3.14" lower="-3.14" effort="400" velocity="1"/>
+      <limit upper="3.14" lower="-3.14" effort="10000000" velocity="20"/>
       <xacro:insert_block name="axis"/>
       <dynamics damping="0.07" friction="0.0"/>
@@ -396,5 +397,5 @@
       <child link="dynamixel_2_${suffix}" />
       <origin xyz="0 0 0" rpy="0 0 0"/>
-      <limit upper="3.14" lower="-3.14" effort="200" velocity="1"/>
+      <limit upper="3.14" lower="-3.14" effort="10000000" velocity="20"/>
       <axis xyz="0 1 0" />
       <dynamics damping="0.07" friction="0.0"/>
@@ -409,5 +410,5 @@
       <child link="link_gripper2_${suffix}" />
       <origin xyz="0.01265148 0.00103883 0.00134042" rpy="0 0 0"/>
-      <limit upper="3.14" lower="-3.14" effort="20" velocity="1"/>
+      <limit upper="3.14" lower="-3.14" effort="10000000" velocity="20"/>
       <axis xyz="0 1 0" />
       <dynamics damping="0.07" friction="0.0"/>

Commit message: Added bottom camera for manipulator motion visualization.

File: mmuav_description/urdf/mmuav.base.urdf.xacro (robot description, xacro)
@@ -216,3 +216,20 @@
     joint_name="joint_q3_passive_right">
   </xacro:transmisija>
+  <!-- Camera properties -->
+  <xacro:property name="camera_link" value="0.05" />
+  <xacro:property name="camera_inertia">
+    <inertia
+    ixx="1e-8"
+    iyy="1e-8"
+    izz="1e-8"
+    ixy="0.0" ixz="0.0" iyz="0.0" />
+  </xacro:property>
+  <xacro:property name="camera_mass" value="1e-5"/>
+  <xacro:cam
+    camera_link="${camera_link}"
+    camera_mass="${camera_mass}"
+    parent="base_link">
+    <origin xyz="0 0 -0.5" rpy="0 ${-PI/2} 0"/>
+    <xacro:insert_block name="camera_inertia"/>
+  </xacro:cam>
 </robot>

File: mmuav_description/urdf/multirotor_base.urdf.xacro (robot description, xacro)
@@ -153,42 +153,49 @@
     </link>
   </xacro:macro>
-   <!-- camera -->
-  <xacro:macro name="camera_macro" params="robot_namespace">
-    <!-- joint -->
+  <!-- Camera macro. Adds a box representing a camera below the UAV
+  @param camera_link Length of the camera box
+  @param camera_mass Mass of the camera
+  @param parent Parent link on which the camera will be fixed
+  @param *origin Block argument defining the origin of the camera with
+  reference to the parent link.
+  @param *inertia Block argument defining camera inertia.
+  -->
+  <xacro:macro name="cam" params="camera_link camera_mass parent *origin *inertia">
+    <!-- Camera link -->
+    <link name="camera_box">
+      <!--collision>
+        <origin xyz="0 0 0" rpy="0 0 0"/>
+        <geometry>
+          <box size="${camera_link} ${camera_link} ${camera_link}"/>
+        </geometry>
+      </collision-->
+      <visual>
+        <origin xyz="0 0 0" rpy="0 0 0"/>
+        <geometry>
+          <box size="${camera_link} ${camera_link} ${camera_link}"/>
+        </geometry>
+        <material name="red"/>
+      </visual>
+      <inertial>
+        <mass value="${camera_mass}" />
+        <origin xyz="0 0 0" rpy="0 0 0"/>
+        <xacro:insert_block name="inertia"/>
+      </inertial>
+    </link>
+    <!-- Camera joint with reference to the parent link -->
     <joint name="camera_joint" type="fixed">
-      <axis xyz="0 1 0" />
-      <origin xyz="0 0 0.2" rpy="0 0 0" />
-      <parent link="base_link" />
-      <child link="camera_link" />
-    </joint>
-    <!-- link -->
-    <link name="camera_link">
-      <collision>
-        <origin xyz="0 0 0" rpy="0 0 0" />
-        <geometry>
-          <box size="0.1 0.1 0.1" />
-        </geometry>
-      </collision>
-      <visual>
-        <origin xyz="0 0 0" rpy="0 0 0" />
-        <geometry>
-          <box size="0.1 0.1 0.1" />
-        </geometry>
-        <material name="red" />
-      </visual>
-      <inertial>
-        <mass value="1e-5" />
-        <origin xyz="0 0 0" rpy="0 0 0" />
-        <inertia ixx="1e-6" ixy="0" ixz="0" iyy="1e-6" iyz="0" izz="1e-6" />
-      </inertial>
-    </link>
-    <gazebo reference="camera_link">
+      <xacro:insert_block name="origin"/>
+      <parent link="${parent}"/>
+      <child link="camera_box"/>
+    </joint>
+    <!-- camera -->
+    <gazebo reference="camera_box">
       <sensor type="camera" name="camera1">
         <update_rate>30.0</update_rate>
         <camera name="head">
-          <horizontal_fov>2</horizontal_fov>
+          <horizontal_fov>1.3962634</horizontal_fov>
           <image>
             <width>800</width>
-            <height>600</height>
+            <height>800</height>
             <format>R8G8B8</format>
           </image>
@@ -206,8 +213,8 @@
           <alwaysOn>true</alwaysOn>
           <updateRate>0.0</updateRate>
-          <cameraName>${robot_namespace}/camera1</cameraName>
+          <cameraName>morus/camera1</cameraName>
           <imageTopicName>image_raw</imageTopicName>
           <cameraInfoTopicName>camera_info</cameraInfoTopicName>
-          <frameName>camera_link</frameName>
+          <frameName>camera_box</frameName>
           <hackBaseline>0.07</hackBaseline>
           <distortionK1>0.0</distortionK1>

Commit message: initial_commit

File: mmuav_description/urdf/mmuav.base.urdf.xacro (robot description, xacro)
@@ -3,5 +3,5 @@
   <!-- Properties -->
   <xacro:property name="rotor_velocity_slowdown_sim" value="10" />
-  <xacro:property name="body_mesh_file" value="3DR_ArducopterArms.dae" />
+  <xacro:property name="body_mesh_file" value="3DR_ArducopterExtendedLegs.dae" />
   <xacro:property name="mass" value="2.5" />  <!-- [kg] -->
   <xacro:property name="body_width" value="0.471" /> <!-- [m] -->
@@ -24,9 +24,4 @@
   <xacro:property name="cos45" value="0.7071" />
   <xacro:property name="PI" value="3.14" />
-    <!-- Manipulator properties-->
-  <xacro:property name="link_length" value="0.5" />
-  <xacro:property name="link_mass" value="0.1"/>
-  <xacro:property name="link_width" value="0.05" />
-  <xacro:property name="link_mesh_file" value="AX12.dae" />
   <!-- Property Blocks -->
   <xacro:property name="body_inertia">
@@ -77,5 +72,5 @@
       dim_y = "0.1"
       dim_z = "0.05">
-      <origin xyz="0 -0.325 -0.1" rpy="0 0 0" />
+      <origin xyz="0 -0.325 -0.075" rpy="0 0 0" />
       <xacro:insert_block name="land_gear_inertia"/>
   </xacro:landing_gear>
@@ -87,5 +82,5 @@
       dim_y = "0.1"
       dim_z = "0.05">
-      <origin xyz="0 0.325 -0.1" rpy="0 0 0" />
+      <origin xyz="0 0.325 -0.075" rpy="0 0 0" />
       <xacro:insert_block name="land_gear_inertia"/>
   </xacro:landing_gear>
@@ -169,53 +164,43 @@
    <!-- Adding left manipulator -->
   <xacro:manipulator
-    link_length="${link_length}"
-    link_width="${link_width}"
-    link_mass="${link_mass}"
-    link_mesh_file="${link_mesh_file}"
     parent="base_link"
     suffix="left">
     <axis xyz="0 1 0" />
-    <!-- origin xyz="${-0.11188*sin45} ${0.11206*cos45} -0.07349" rpy="-1.57079632679 0 0"/ -->
-    <origin xyz="0 0.158342 -0.07349" rpy="-1.57079632679 0 0"/>
+    <origin xyz="0 -0.1583424671 -0.07349" rpy="0 ${PI} 0"/>
   </xacro:manipulator>
      <!-- Adding right manipulator -->
   <xacro:manipulator
-    link_length="${link_length}"
-    link_width="${link_width}"
-    link_mass="${link_mass}"
-    link_mesh_file="${link_mesh_file}"
     parent="base_link"
     suffix="right">
     <axis xyz="0 1 0" />
-    <!--origin xyz="${0.11205**sin45} ${-0.11188*cos45} -0.07349" rpy="-1.57079632679 0 0"/ -->
-    <origin xyz="0 -0.158342 -0.07349" rpy="-1.57079632679 0 0"/>
+    <origin xyz="0 0.1583424671 -0.07349" rpy="0 ${PI} ${PI}"/>
   </xacro:manipulator>
   <!-- Add transmission for joints-->
   <xacro:transmisija
     trans_number="0"
-    joint_name="joint_q1_left">
+    joint_name="joint_dynamixel1_left">
+  </xacro:transmisija>
+  <xacro:transmisija
+    trans_number="1"
+    joint_name="joint_dynamixel2_left">
+  </xacro:transmisija>
+  <xacro:transmisija
+    trans_number="2"
+    joint_name="joint_dynamixel1_right">
   </xacro:transmisija>
   <xacro:transmisija
     trans_number="3"
-    joint_name="joint_q1_right">
-  </xacro:transmisija>
-  <xacro:transmisija
-    trans_number="1"
-    joint_name="joint_q2_left">
+    joint_name="joint_dynamixel2_right">
   </xacro:transmisija>
   <xacro:transmisija
     trans_number="4"
-    joint_name="joint_q2_right">
+    joint_name="joint_gripper2_right">
   </xacro:transmisija>
   <xacro:transmisija
     trans_number="5"
-    joint_name="joint_q3_passive_left">
-  </xacro:transmisija >
-  <xacro:transmisija
-    trans_number="6"
-    joint_name="joint_q3_passive_right">
+    joint_name="joint_gripper2_left">
   </xacro:transmisija>
   <!-- Camera properties -->
-  <xacro:property name="camera_link" value="0.05" />
+  <!--xacro:property name="camera_link" value="0.05" />
   <xacro:property name="camera_inertia">
     <inertia
@@ -232,4 +217,4 @@
     <origin xyz="0 0 -0.5" rpy="0 ${-PI/2} 0"/>
     <xacro:insert_block name="camera_inertia"/>
-  </xacro:cam>
+  </xacro:cam-->
 </robot>

File: mmuav_description/urdf/mmuav.gazebo.xacro (robot description, xacro)
@@ -80,5 +80,5 @@
   </gazebo-->
     <!-- Mount first generic pose sensor-->
-  <xacro:odometry_plugin_macro
+  <!--xacro:odometry_plugin_macro
     namespace="$(arg name)"
     odometry_sensor_suffix="2"
@@ -106,6 +106,6 @@
     odometry_map=""
     image_scale="0.1">
-    <inertia ixx="0.00001" ixy="0.0" ixz="0.0" iyy="0.00001" iyz="0.0" izz="0.00001" /> <!-- [kg m^2] [kg m^2] [kg m^2] [kg m^2] [kg m^2] [kg m^2] -->
-    <origin xyz="-0.0 0.0 0" rpy="0.0 0.0 0.0" />
+    <inertia ixx="0.00001" ixy="0.0" ixz="0.0" iyy="0.00001" iyz="0.0" izz="0.00001" /--> <!-- [kg m^2] [kg m^2] [kg m^2] [kg m^2] [kg m^2] [kg m^2] -->
+    <!--origin xyz="-0.0 0.0 0" rpy="0.0 0.0 0.0" />
   </xacro:odometry_plugin_macro>
   <xacro:odometry_plugin_macro
@@ -135,7 +135,75 @@
     odometry_map=""
     image_scale="0.1">
-    <inertia ixx="0.00001" ixy="0.0" ixz="0.0" iyy="0.00001" iyz="0.0" izz="0.00001" /> <!-- [kg m^2] [kg m^2] [kg m^2] [kg m^2] [kg m^2] [kg m^2] -->
-    <origin xyz="-0.0 0.0 0" rpy="0.0 0.0 0.0" />
-  </xacro:odometry_plugin_macro>
+    <inertia ixx="0.00001" ixy="0.0" ixz="0.0" iyy="0.00001" iyz="0.0" izz="0.00001" /--> <!-- [kg m^2] [kg m^2] [kg m^2] [kg m^2] [kg m^2] [kg m^2] -->
+    <!--origin xyz="-0.0 0.0 0" rpy="0.0 0.0 0.0" />
+  </xacro:odometry_plugin_macro-->
+  <gazebo reference="link_manipulator2uav_left">
+    <gravity>true</gravity>
+    <self_collide>false</self_collide>
+  </gazebo>
+  <gazebo reference="link_manipulator2uav_right">
+    <gravity>true</gravity>
+    <self_collide>false</self_collide>
+  </gazebo>
+  <gazebo reference="link_dynamixel1_left">
+    <gravity>true</gravity>
+    <self_collide>false</self_collide>
+  </gazebo>
+  <gazebo reference="link_dynamixel1_right">
+    <gravity>true</gravity>
+    <self_collide>false</self_collide>
+  </gazebo>
+  <gazebo reference="link_F3_left">
+    <gravity>true</gravity>
+    <self_collide>false</self_collide>
+  </gazebo>
+  <gazebo reference="link_F3_right">
+    <gravity>true</gravity>
+    <self_collide>false</self_collide>
+  </gazebo>
+  <gazebo reference="link_F4_left">
+    <gravity>true</gravity>
+    <self_collide>false</self_collide>
+  </gazebo>
+  <gazebo reference="link_F4_right">
+    <gravity>true</gravity>
+    <self_collide>false</self_collide>
+  </gazebo>
+  <gazebo reference="link_dynamixel2_left">
+    <gravity>true</gravity>
+    <self_collide>false</self_collide>
+  </gazebo>
+  <gazebo reference="link_dynamixel2_right">
+    <gravity>true</gravity>
+    <self_collide>false</self_collide>
+  </gazebo>
+  <gazebo reference="link_gripper1_left">
+    <gravity>true</gravity>
+    <self_collide>false</self_collide>
+  </gazebo>
+  <gazebo reference="link_gripper1_right">
+    <gravity>true</gravity>
+    <self_collide>false</self_collide>
+  </gazebo>
+  <gazebo reference="link_gripper2_left">
+    <gravity>true</gravity>
+    <self_collide>false</self_collide>
+  </gazebo>
+  <gazebo reference="link_gripper2_right">
+    <gravity>true</gravity>
+    <self_collide>false</self_collide>
+  </gazebo>
+  <gazebo reference="base_link_inertia">
+    <gravity>true</gravity>
+    <self_collide>false</self_collide>
+  </gazebo>
+  <gazebo reference="land_gear_1">
+    <gravity>true</gravity>
+    <self_collide>false</self_collide>
+  </gazebo>
+  <gazebo reference="land_gear_2">
+    <gravity>true</gravity>
+    <self_collide>false</self_collide>
+  </gazebo>
   <gazebo reference="base_link">
     <dampingFactor>0.0002</dampingFactor>
