Commit message: .

File: mmuav_description/urdf/mmuav.base.urdf.xacro (robot description, xacro)
@@ -232,10 +232,10 @@
       </collision>
     </link>
-    <joint name="joint_screw" type="fixed">
+    <joint name="joint_screw1" type="fixed">
         <origin xyz="0.023 0.006 0.0385" rpy="${PI} 0 ${PI/6}" />
         <parent link="link_gripper2_left"/>
         <child link="link_screw"/>
     </joint>
-    <!--link name='link_screw2'>
+    <link name='link_screw2'>
       <inertial>
         <mass value="0.05" />
@@ -251,5 +251,5 @@
         <parent link="link_gripper2_right"/>
         <child link="link_screw2"/>
-    </joint-->
+    </joint>
   <!-- Camera properties -->
   <!--xacro:property name="camera_link" value="0.05" />

File: mmuav_description/urdf/multirotor_base.urdf.xacro (robot description, xacro)
@@ -387,9 +387,9 @@
     <!--JOINT1 CONTINOUS dynamixel1-->
     <!--_____________________________________________________________-->
-    <joint name="joint_dynamixel1_${suffix}" type="continuous">
+    <joint name="joint_dynamixel1_${suffix}" type="revolute">
       <parent link="link_manipulator2uav_${suffix}"/>
       <child link="link_dynamixel1_${suffix}"/>
       <origin xyz="0 0 0" rpy="${PI} 0 ${-PI/2}" />
-      <!--limit upper="6" lower="-6" effort="15" velocity="6.17"/-->
+      <limit upper="6" lower="-6" effort="15" velocity="6.17"/>
       <axis xyz="0 0 1" />
     </joint>
@@ -413,9 +413,9 @@
     <!--JOINT2 CONTINOUS dynamixel2-->
     <!--_____________________________________________________________-->
-    <joint name="joint_dynamixel2_${suffix}" type="continuous">
+    <joint name="joint_dynamixel2_${suffix}" type="revolute">
       <parent link="link_F4_${suffix}"/>
       <child link="link_dynamixel2_${suffix}"/>
       <origin xyz="0 0 0" rpy="0 0 ${-PI/2}" />
-      <!--limit upper="6" lower="-6" effort="15" velocity="6.17"/-->
+      <limit upper="6" lower="-6" effort="15" velocity="6.17"/>
       <axis xyz="0 0 1" />
     </joint>
@@ -431,9 +431,9 @@
     <!--JOINT3 CONTINOUS gripper-->
     <!--_____________________________________________________________-->
-    <joint name="joint_gripper2_${suffix}" type="continuous">
+    <joint name="joint_gripper2_${suffix}" type="revolute">
       <parent link="link_gripper1_${suffix}"/>
       <child link="link_gripper2_${suffix}"/>
       <origin xyz="0.01265 0.00104 -0.00134" rpy="0 0 ${PI}" />
-      <!--limit upper="6" lower="-6" effort="15" velocity="6.17"/-->
+      <limit upper="6" lower="-6" effort="15" velocity="6.17"/>
       <axis xyz="0 0 1" />
     </joint>
