Commit message: added odometry plugin

File: mmuav_description/urdf/mmuav.gazebo.xacro (robot description, xacro)
@@ -79,3 +79,62 @@
     </plugin>
   </gazebo-->
+    <!-- Mount first generic pose sensor-->
+  <xacro:odometry_plugin_macro
+    namespace="$(arg name)"
+    odometry_sensor_suffix="2"
+    child_frame_id="base"
+    parent_link="link_gripper2_left"
+    pose_topic="link_gripper2_left/pose"
+    pose_with_covariance_topic="link_gripper2_left/pose_with_covariance"
+    position_topic="link_gripper2_left/position"
+    transform_topic="link_gripper2_left/transform"
+    odometry_topic="link_gripper2_left/odometry"
+    parent_frame_id="world"
+    mass_odometry_sensor="0.01"
+    measurement_divisor="10"
+    measurement_delay="10"
+    unknown_delay="0.0"
+    noise_normal_position="0.0 0.0 0.0"
+    noise_normal_quaternion="0.0 0.0 0.0"
+    noise_normal_linear_velocity="0 0 0"
+    noise_normal_angular_velocity="0 0 0"
+    noise_uniform_position="0 0 0"
+    noise_uniform_quaternion="0 0 0"
+    noise_uniform_linear_velocity="0 0 0"
+    noise_uniform_angular_velocity="0 0 0"
+    enable_odometry_map="false"
+    odometry_map=""
+    image_scale="0.1">
+    <inertia ixx="0.00001" ixy="0.0" ixz="0.0" iyy="0.00001" iyz="0.0" izz="0.00001" /> <!-- [kg m^2] [kg m^2] [kg m^2] [kg m^2] [kg m^2] [kg m^2] -->
+    <origin xyz="-0.0 0.0 0" rpy="0.0 0.0 0.0" />
+  </xacro:odometry_plugin_macro>
+  <xacro:odometry_plugin_macro
+    namespace="$(arg name)"
+    odometry_sensor_suffix="3"
+    child_frame_id="base"
+    parent_link="link_gripper2_right"
+    pose_topic="link_gripper2_right/pose"
+    pose_with_covariance_topic="link_gripper2_right/pose_with_covariance"
+    position_topic="link_gripper2_right/position"
+    transform_topic="link_gripper2_right/transform"
+    odometry_topic="link_gripper2_right/odometry"
+    parent_frame_id="world"
+    mass_odometry_sensor="0.01"
+    measurement_divisor="10"
+    measurement_delay="10"
+    unknown_delay="0.0"
+    noise_normal_position="0.0 0.0 0.0"
+    noise_normal_quaternion="0.0 0.0 0.0"
+    noise_normal_linear_velocity="0 0 0"
+    noise_normal_angular_velocity="0 0 0"
+    noise_uniform_position="0 0 0"
+    noise_uniform_quaternion="0 0 0"
+    noise_uniform_linear_velocity="0 0 0"
+    noise_uniform_angular_velocity="0 0 0"
+    enable_odometry_map="false"
+    odometry_map=""
+    image_scale="0.1">
+    <inertia ixx="0.00001" ixy="0.0" ixz="0.0" iyy="0.00001" iyz="0.0" izz="0.00001" /> <!-- [kg m^2] [kg m^2] [kg m^2] [kg m^2] [kg m^2] [kg m^2] -->
+    <origin xyz="-0.0 0.0 0" rpy="0.0 0.0 0.0" />
+  </xacro:odometry_plugin_macro>
 </robot>

Commit message: added screw and forces sensor

File: mmuav_description/urdf/mmuav.gazebo.xacro (robot description, xacro)
@@ -80,14 +80,14 @@
   </gazebo-->
     <!-- Mount first generic pose sensor-->
-  <!--xacro:odometry_plugin_macro
+  <xacro:odometry_plugin_macro
     namespace="$(arg name)"
     odometry_sensor_suffix="2"
     child_frame_id="base"
-    parent_link="link_gripper2_left"
-    pose_topic="link_gripper2_left/pose"
-    pose_with_covariance_topic="link_gripper2_left/pose_with_covariance"
-    position_topic="link_gripper2_left/position"
-    transform_topic="link_gripper2_left/transform"
-    odometry_topic="link_gripper2_left/odometry"
+    parent_link="link_dynamixel1_left"
+    pose_topic="link_dynamixel1_left/pose"
+    pose_with_covariance_topic="link_dynamixel1_left/pose_with_covariance"
+    position_topic="link_dynamixel1_left/position"
+    transform_topic="link_dynamixel1_left/transform"
+    odometry_topic="link_dynamixel1_left/odometry"
     parent_frame_id="base_link"
     mass_odometry_sensor="0.01"
@@ -106,6 +106,6 @@
     odometry_map=""
     image_scale="0.1">
-    <inertia ixx="0.00001" ixy="0.0" ixz="0.0" iyy="0.00001" iyz="0.0" izz="0.00001" /--> <!-- [kg m^2] [kg m^2] [kg m^2] [kg m^2] [kg m^2] [kg m^2] -->
-    <!--origin xyz="-0.0 0.0 0" rpy="0.0 0.0 0.0" />
+    <inertia ixx="0.00001" ixy="0.0" ixz="0.0" iyy="0.00001" iyz="0.0" izz="0.00001" /> <!-- [kg m^2] [kg m^2] [kg m^2] [kg m^2] [kg m^2] [kg m^2] -->
+    <origin xyz="0.0 0.0 0" rpy="0.0 0.0 0.0" />
   </xacro:odometry_plugin_macro>
   <xacro:odometry_plugin_macro
@@ -135,7 +135,7 @@
     odometry_map=""
     image_scale="0.1">
-    <inertia ixx="0.00001" ixy="0.0" ixz="0.0" iyy="0.00001" iyz="0.0" izz="0.00001" /--> <!-- [kg m^2] [kg m^2] [kg m^2] [kg m^2] [kg m^2] [kg m^2] -->
-    <!--origin xyz="-0.0 0.0 0" rpy="0.0 0.0 0.0" />
-  </xacro:odometry_plugin_macro-->
+    <inertia ixx="0.00001" ixy="0.0" ixz="0.0" iyy="0.00001" iyz="0.0" izz="0.00001" /> <!-- [kg m^2] [kg m^2] [kg m^2] [kg m^2] [kg m^2] [kg m^2] -->
+    <origin xyz="0.04903524 0.0 0" rpy="0.0 0.0 0.0" />
+  </xacro:odometry_plugin_macro>
   <gazebo reference="link_manipulator2uav_left">
     <gravity>true</gravity>

File: mmuav_description/urdf/multirotor_base.urdf.xacro (robot description, xacro)
@@ -383,6 +383,6 @@
       <parent link="link_manipulator2uav_${suffix}"/>
       <child link="link_dynamixel1_${suffix}"/>
-      <origin xyz="0 0 0" rpy="${PI} 0 0" />
-      <limit upper="6" lower="-6" effort="1.5" velocity="6.2"/>
+      <origin xyz="0 0 0" rpy="${PI} 0 ${-PI/2}" />
+      <limit upper="6" lower="-6" effort="1.5" velocity="1"/>
       <axis xyz="0 0 1" />
     </joint>
@@ -409,6 +409,6 @@
       <parent link="link_F4_${suffix}"/>
       <child link="link_dynamixel2_${suffix}"/>
-      <origin xyz="0 0 0" rpy="0 0 0" />
-      <limit upper="6" lower="-6" effort="1.5" velocity="6.2"/>
+      <origin xyz="0 0 0" rpy="0 0 ${-PI/2}" />
+      <limit upper="6" lower="-6" effort="1.5" velocity="1"/>
       <axis xyz="0 0 1" />
     </joint>
@@ -427,6 +427,6 @@
       <parent link="link_gripper1_${suffix}"/>
       <child link="link_gripper2_${suffix}"/>
-      <origin xyz="0.01265 0.00104 -0.00134" rpy="0 0 ${PI}" />
-      <limit upper="3.14" lower="3.14" effort="1.5" velocity="6.2"/>
+      <origin xyz="0.01265 0.00104 -0.00134" rpy="0 0 0" />
+      <limit upper="0" lower="0" effort="1.5" velocity="1"/>
       <axis xyz="0 0 1" />
     </joint>

File: mmuav_description/urdf/screw.base.urdf.xacro (robot description, xacro)
@@ -5,5 +5,5 @@
   <xacro:include filename="$(find mmuav_description)/urdf/multirotor_base.urdf.xacro" />
   <xacro:screw>
-    <origin xyz="0 0 0" rpy="0 0 0"/>
+    <origin xyz="0 0 0.1" rpy="0 ${PI} 0"/>
   </xacro:screw>
 </robot>

Commit message: novi bracnh:

File: mmuav_description/urdf/mmuav.gazebo.xacro (robot description, xacro)
@@ -212,8 +212,16 @@
     <gravity>true</gravity>
     <self_collide>true</self_collide>
-    <mu1>0</mu1>
-    <mu2>0</mu2>
+    <mu1>1</mu1>
+    <mu2>1</mu2>
     <maxContacts>1</maxContacts>
     <fdir1 value = "1 0 0"/>
   </gazebo>
+  <gazebo reference="link_force_sensor_top_mount">
+    <gravity>true</gravity>
+    <self_collide>true</self_collide>
+    <mu1>1</mu1>
+    <mu2>1</mu2>
+    <maxContacts>1</maxContacts>
+    <fdir1 value = "1 0 0"/>
+  </gazebo>
 </robot>

File: mmuav_description/urdf/multirotor_base.urdf.xacro (robot description, xacro)
@@ -512,5 +512,5 @@
         <origin xyz="-0.01903 -0.01661 -0.05153" rpy="0 0 0" />
         <geometry>
-          <mesh filename="package://mmuav_description/meshes/forcesensor_mount_top.dae"
+          <mesh filename="package://mmuav_description/meshes/forcesensor_mount_top_without_hole.dae"
             scale="1 1 1" />
         </geometry>
@@ -519,5 +519,5 @@
         <origin xyz="-0.01903 -0.01661 -0.05153" rpy="0 0 0"/>
         <geometry>
-          <mesh filename="package://mmuav_description/meshes/forcesensor_mount_top.dae"
+          <mesh filename="package://mmuav_description/meshes/forcesensor_mount_top_without_hole.dae"
             scale="1 1 1" />
         </geometry>
