Commit message: Switched mmc uav simulation to new time constants.

File: mmuav_description/urdf/mmcuav.base.urdf.xacro (robot description, xacro)
@@ -13,5 +13,6 @@
   <xacro:property name="motor_constant" value="8.54858e-06" /> <!-- [kg*m/s^2] -->
   <xacro:property name="moment_constant" value="0.016" /> <!-- [m] -->
-  <xacro:property name="time_constant" value="0.0125" /> <!-- [s] -->
+  <xacro:property name="time_constant_up" value="0.0125" /> <!-- [s] -->
+  <xacro:property name="time_constant_down" value="0.025" /> <!-- [s] -->
   <xacro:property name="max_rot_velocity" value="1475" /> <!-- [rad/s] -->
   <xacro:property name="sin45" value="0.7071068" />
@@ -82,5 +83,6 @@
     mass_rotor="${mass_rotor}"
     radius_rotor="${radius_rotor}"
-    time_constant="${time_constant}"
+    time_constant_up="${time_constant_up}"
+    time_constant_down="${time_constant_down}"
     max_rot_velocity="${max_rot_velocity}"
     motor_number="0"
@@ -101,5 +103,6 @@
     mass_rotor="${mass_rotor}"
     radius_rotor="${radius_rotor}"
-    time_constant="${time_constant}"
+    time_constant_up="${time_constant_up}"
+    time_constant_down="${time_constant_down}"
     max_rot_velocity="${max_rot_velocity}"
     motor_number="3"
@@ -120,5 +123,6 @@
     mass_rotor="${mass_rotor}"
     radius_rotor="${radius_rotor}"
-    time_constant="${time_constant}"
+    time_constant_up="${time_constant_up}"
+    time_constant_down="${time_constant_down}"
     max_rot_velocity="${max_rot_velocity}"
     motor_number="1"
@@ -139,5 +143,6 @@
     mass_rotor="${mass_rotor}"
     radius_rotor="${radius_rotor}"
-    time_constant="${time_constant}"
+    time_constant_up="${time_constant_up}"
+    time_constant_down="${time_constant_down}"
     max_rot_velocity="${max_rot_velocity}"
     motor_number="2"

Commit message: Added option to tilt propellers in mmcuav.

File: mmuav_description/urdf/mmcuav.base.urdf.xacro (robot description, xacro)
@@ -32,4 +32,5 @@
   <xacro:property name="cos45" value="0.7071" />
   <xacro:property name="PI" value="3.1415926535897931" />
+  <xacro:property name="tilt_angle" value="0.0"/>
   <!-- Property Blocks -->
   <xacro:property name="body_inertia">
@@ -91,5 +92,5 @@
     color="Red">
     <!--<origin xyz="${cos45*arm_length} ${sin45*arm_length} ${rotor_offset_top}" rpy="0 0 0" />-->
-    <origin xyz="${1*arm_length} ${0*arm_length} ${rotor_offset_top}" rpy="0 0 0" />
+    <origin xyz="${1*arm_length} ${0*arm_length} ${rotor_offset_top}" rpy="0 ${-tilt_angle} 0" />
     <xacro:insert_block name="rotor_inertia" />
   </xacro:vertical_rotor>
@@ -111,5 +112,5 @@
     color="Blue">
     <!--<origin xyz="${cos45*arm_length} ${-sin45*arm_length} ${rotor_offset_top}" rpy="0 0 0" />-->
-    <origin xyz="${0*arm_length} ${-1*arm_length} ${rotor_offset_top}" rpy="0 0 0" />
+    <origin xyz="${0*arm_length} ${-1*arm_length} ${rotor_offset_top}" rpy="${-tilt_angle} 0 0" />
     <xacro:insert_block name="rotor_inertia" />
   </xacro:vertical_rotor>
@@ -131,5 +132,5 @@
     color="Blue">
     <!--<origin xyz="${-cos45*arm_length} ${sin45*arm_length} ${rotor_offset_top}" rpy="0 0 0" />-->
-    <origin xyz="${0*arm_length} ${1*arm_length} ${rotor_offset_top}" rpy="0 0 0" />
+    <origin xyz="${0*arm_length} ${1*arm_length} ${rotor_offset_top}" rpy="${tilt_angle} 0 0" />
     <xacro:insert_block name="rotor_inertia" />
   </xacro:vertical_rotor>
@@ -151,5 +152,5 @@
     color="Red">
     <!--<origin xyz="${-cos45*arm_length} ${-sin45*arm_length} ${rotor_offset_top}" rpy="0 0 0" />-->
-    <origin xyz="${-1*arm_length} ${0*arm_length} ${rotor_offset_top}" rpy="0 0 0" />
+    <origin xyz="${-1*arm_length} ${0*arm_length} ${rotor_offset_top}" rpy="0 ${tilt_angle} 0" />
     <xacro:insert_block name="rotor_inertia" />
   </xacro:vertical_rotor>

Commit message: Changed rotors 1 and thrust gain.

File: mmuav_description/urdf/mmcuav.base.urdf.xacro (robot description, xacro)
@@ -12,4 +12,6 @@
   <xacro:property name="radius_rotor" value="0.1524" /> <!-- [m] -->
   <xacro:property name="motor_constant" value="8.54858e-06" /> <!-- [kg*m/s^2] -->
+  <xacro:property name="motor_constant1" value="8.762e-06" /> <!-- [kg*m/s^2] -->
+  <xacro:property name="motor_constant3" value="8.33487e-06" /> <!-- [kg*m/s^2] -->
   <xacro:property name="moment_constant" value="0.016" /> <!-- [m] -->
   <xacro:property name="time_constant_up" value="0.0125" /> <!-- [s] -->
@@ -78,5 +80,5 @@
     suffix="front_left"
     direction="cw"
-    motor_constant="${motor_constant}"
+    motor_constant="${motor_constant1}"
     moment_constant="${moment_constant}"
     parent="base_link"
@@ -118,5 +120,5 @@
     suffix="back_left"
     direction="ccw"
-    motor_constant="${motor_constant}"
+    motor_constant="${motor_constant3}"
     moment_constant="${moment_constant}"
     parent="base_link"

File: mmuav_description/urdf/mmcuav.gazebo.xacro (robot description, xacro)
@@ -69,5 +69,5 @@
     mass_odometry_sensor="0.01"
     measurement_divisor="10"
-    measurement_delay="0.0"
+    measurement_delay="0.001"
     unknown_delay="0.0"
     noise_normal_position="0.0 0.0 0.0"

Commit message: All rotors thrust constants and limits returned to the nominal values.

File: mmuav_description/urdf/mmcuav.base.urdf.xacro (robot description, xacro)
@@ -12,6 +12,6 @@
   <xacro:property name="radius_rotor" value="0.1524" /> <!-- [m] -->
   <xacro:property name="motor_constant" value="8.54858e-06" /> <!-- [kg*m/s^2] -->
-  <xacro:property name="motor_constant1" value="8.762e-06" /> <!-- [kg*m/s^2] -->
-  <xacro:property name="motor_constant3" value="8.33487e-06" /> <!-- [kg*m/s^2] -->
+  <xacro:property name="motor_constant1" value="8.54858e-06" /> <!-- [kg*m/s^2] -->
+  <xacro:property name="motor_constant3" value="8.54858e-06" /> <!-- [kg*m/s^2] -->
   <xacro:property name="moment_constant" value="0.016" /> <!-- [m] -->
   <xacro:property name="time_constant_up" value="0.0125" /> <!-- [s] -->

Commit message: Able to launch UAV with moving masses

File: mmuav_description/urdf/mmcuav.base.urdf.xacro (robot description, xacro)
@@ -157,4 +157,32 @@
   <!-- <xacro:camera_macro robot_namespace="${namespace}">
   </xacro:camera_macro> -->
+  <!-- Added landing gear -->
+  <xacro:property name="land_gear_inertia">
+    <inertia
+    ixx="1e-6"
+    iyy="1e-6"
+    izz="1e-6"
+    ixy="0.0" ixz="0.0"  iyz="0.0" /> <!-- [kg*m^2] [kg*m^2] [kg*m^2] [kg*m^2] [kg*m^2] [kg*m^2] -->
+  </xacro:property>
+  <xacro:landing_gear
+      parent="base_link"
+      gear_num = "1"
+      mass = "1e-6"
+      dim_x = "0.8"
+      dim_y = "0.1"
+      dim_z = "0.05">
+      <origin xyz="0 -0.325 -0.1" rpy="0 0 0" />
+      <xacro:insert_block name="land_gear_inertia"/>
+  </xacro:landing_gear>
+  <xacro:landing_gear
+      parent="base_link"
+      gear_num = "2"
+      mass = "1e-6"
+      dim_x = "0.8"
+      dim_y = "0.1"
+      dim_z = "0.05">
+      <origin xyz="0 0.325 -0.1" rpy="0 0 0" />
+      <xacro:insert_block name="land_gear_inertia"/>
+  </xacro:landing_gear>
   <!-- Instantinate movable mass 0 -->
   <xacro:movable_mass

File: mmuav_description/urdf/mmcuav.gazebo.xacro (robot description, xacro)
@@ -62,4 +62,5 @@
     parent_link="base_link"
     pose_topic="pose"
+    velocity_relative_topic="velocity_relative"
     pose_with_covariance_topic="pose_with_covariance"
     position_topic="position"
