Commit message: Adapted position and height control for velocity topic from rotors_gazebo.

File: mmuav_description/urdf/uav.gazebo.xacro (robot description, xacro)
@@ -62,4 +62,5 @@
     parent_link="base_link"
     pose_topic="pose"
+    velocity_relative_topic="velocity_relative"
     pose_with_covariance_topic="pose_with_covariance"
     position_topic="position"
@@ -68,20 +69,20 @@
     parent_frame_id="world"
     mass_odometry_sensor="0.01"
-    measurement_divisor="10"
-    measurement_delay="10"
+    measurement_divisor="5"
+    measurement_delay="0"
     unknown_delay="0.0"
     noise_normal_position="0.0 0.0 0.0"
     noise_normal_quaternion="0.0 0.0 0.0"
-    noise_normal_linear_velocity="0 0 0"
-    noise_normal_angular_velocity="0 0 0"
-    noise_uniform_position="0 0 0"
-    noise_uniform_quaternion="0 0 0"
-    noise_uniform_linear_velocity="0 0 0"
-    noise_uniform_angular_velocity="0 0 0"
+    noise_normal_linear_velocity="0.0 0.0 0.0"
+    noise_normal_angular_velocity="0.0 0.0 0.0"
+    noise_uniform_position="0.0 0.0 0.0"
+    noise_uniform_quaternion="0.0 0.0 0.0"
+    noise_uniform_linear_velocity="0.0 0.0 0.0"
+    noise_uniform_angular_velocity="0.0 0.0 0.0"
     enable_odometry_map="false"
     odometry_map=""
-    image_scale="0.1">
+    image_scale="">
     <inertia ixx="0.00001" ixy="0.0" ixz="0.0" iyy="0.00001" iyz="0.0" izz="0.00001" /> <!-- [kg m^2] [kg m^2] [kg m^2] [kg m^2] [kg m^2] [kg m^2] -->
-    <origin xyz="-0.0 0.0 0" rpy="0.0 0.0 0.0" />
+    <origin xyz="0.0 0.0 0" rpy="0.0 0.0 0.0" />
   </xacro:odometry_plugin_macro>
 </robot>

Commit message: Add mount_magnet option to uav robot.

File: mmuav_description/urdf/uav.gazebo.xacro (robot description, xacro)
@@ -14,4 +14,6 @@
   <xacro:property name="enable_bag_plugin" value="false" />
   <xacro:property name="bag_file" value="uav.bag" />
+  <xacro:arg name="mount_magnet" default="false" />
+  <xacro:property name="mount_magnet" value="$(arg mount_magnet)" />
   <!-- Instantiate mmuav "mechanics" -->
   <xacro:include filename="$(find mmuav_description)/urdf/uav.base.urdf.xacro" />
@@ -55,4 +57,18 @@
     </plugin>
   </gazebo>
+  <xacro:if value="${mount_magnet}">
+    <gazebo>
+      <plugin name="dipole_magnet" filename="libstorm_gazebo_dipole_magnet.so">
+        <robotNamespace>uav</robotNamespace>
+        <bodyName>base_link</bodyName>
+        <dipole_moment>0 0 970</dipole_moment>
+        <!-- Set to false if not using ROS -->
+        <shouldPublish>true</shouldPublish>
+        <topicNs>magnet</topicNs>
+        <updateRate>100</updateRate>
+        <gain>1.0</gain>
+      </plugin>
+    </gazebo>
+  </xacro:if>
   <!-- Mount first generic pose sensor-->
   <xacro:odometry_plugin_macro

Commit message: Add argument for z axis value and optional disk to separate magnet from UAV

File: mmuav_description/urdf/uav.gazebo.xacro (robot description, xacro)
@@ -16,4 +16,8 @@
   <xacro:arg name="mount_magnet" default="false" />
   <xacro:property name="mount_magnet" value="$(arg mount_magnet)" />
+  <xacro:arg name="mount_magnet_with_disk" default="false" />
+  <xacro:property name="mount_magnet_with_disk" value="$(arg mount_magnet_with_disk)" />
+  <xacro:arg name="magnet_dipole_moment_z" default="970" />
+  <xacro:property name="dp_z" value="$(arg magnet_dipole_moment_z)" />
   <!-- Instantiate mmuav "mechanics" -->
   <xacro:include filename="$(find mmuav_description)/urdf/uav.base.urdf.xacro" />
@@ -58,9 +62,34 @@
   </gazebo>
   <xacro:if value="${mount_magnet}">
+    <xacro:if value="${mount_magnet_with_disk}">
+      <joint name="electromagnet_joint" type="fixed">
+        <axis xyz="0 1 0" />
+        <origin xyz="0.0 0.0 -0.15" rpy="0 0 0"/>
+        <parent link="base_link"/>
+        <child link="electromagnet_actuator"/>
+      </joint>
+      <link name="electromagnet_actuator">
+        <inertial>
+        <origin xyz="0 0 0" rpy="0 0 0" />
+        <mass value="0.025"/>
+        <inertia ixx="0.0001" ixy="0" ixz="0" iyy ="0.0001" iyz = "0" izz = "0.0001" />
+        </inertial>
+        <collision name="collision">
+        <geometry>
+          <cylinder radius="0.08" length="0.035"/>
+        </geometry>
+        </collision>
+        <visual>
+        <geometry>
+          <cylinder radius="0.08" length="0.035"/>
+        </geometry>
+        </visual>
+      </link>
+    </xacro:if>
     <gazebo>
       <plugin name="dipole_magnet" filename="libstorm_gazebo_dipole_magnet.so">
-        <robotNamespace>uav</robotNamespace>
+        <robotNamespace>$(arg name)</robotNamespace>
         <bodyName>base_link</bodyName>
-        <dipole_moment>0 0 970</dipole_moment>
+        <dipole_moment>0 0 ${dp_z}</dipole_moment>
         <!-- Set to false if not using ROS -->
         <shouldPublish>true</shouldPublish>

Commit message: Add example of gimbal mounting

File: mmuav_description/urdf/uav.gazebo.xacro (robot description, xacro)
@@ -131,3 +131,7 @@
     <origin xyz="0.0 0.0 0" rpy="0.0 0.0 0.0" />
   </xacro:odometry_plugin_macro>
+  <!-- mount gimbal -->
+  <!--<xacro:gimbal_macro parent="base_link">
+    <origin xyz="0.25 0 -0.05" rpy="0 0 0"/>
+  </xacro:gimbal_macro> -->
 </robot>

Commit message: added velodyne to uav

File: mmuav_description/urdf/uav.gazebo.xacro (robot description, xacro)
@@ -14,4 +14,6 @@
   <xacro:property name="enable_bag_plugin" value="false" />
   <xacro:property name="bag_file" value="uav.bag" />
+  <xacro:arg name="mount_velodyne" default="false" />
+  <xacro:property name="mount_velodyne" value="$(arg mount_velodyne)" />
   <xacro:arg name="mount_magnet" default="false" />
   <xacro:property name="mount_magnet" value="$(arg mount_magnet)" />
@@ -37,4 +39,7 @@
     <limit upper="0" lower="0" effort="0" velocity="0" />
   </joint>
+  <xacro:property name="horizontal_velodyne_origin">
+    <origin xyz="0 0 -0.025" rpy="3.141592653589793 0.1323284641020683 0." />
+  </xacro:property>
   <!-- Mount an IMU -->
   <gazebo>
@@ -61,4 +66,11 @@
     </plugin>
   </gazebo>
+  <xacro:if value="${mount_velodyne}">
+    <xacro:include filename="$(find velodyne_description)/urdf/VU-8.urdf.xacro"/>
+    <VU-8 parent="base_link" name="velodyne" topic="$(arg name)/velodyne_points" hz="10" samples="440" gpu="false"
+            min_range="1" lasers="16">
+        <xacro:insert_block name="horizontal_velodyne_origin"/>
+    </VU-8>
+  </xacro:if>
   <xacro:if value="${mount_magnet}">
     <xacro:if value="${mount_magnet_with_disk}">

Commit message: Add option to choose realistic or ground truth feedback.

File: mmuav_description/urdf/uav.gazebo.xacro (robot description, xacro)
@@ -28,4 +28,6 @@
   <xacro:arg name="manipulator_tool" default="none" />
   <xacro:property name="manipulator_tool" value="$(arg manipulator_tool)" />
+  <xacro:arg name="odometry_type" default="ground_truth" />
+  <xacro:property name="odometry_type" value="$(arg odometry_type)" />
   <xacro:arg name="collision_bitmask" default="-1" />
   <xacro:property name="collision_bitmask" value="$(arg collision_bitmask)" />
@@ -154,34 +156,68 @@
   </xacro:if>
   <!-- Mount first generic pose sensor-->
-  <xacro:odometry_plugin_macro
-    namespace="$(arg name)"
-    odometry_sensor_suffix="1"
-    child_frame_id="base"
-    parent_link="base_link"
-    pose_topic="pose"
-    velocity_relative_topic="velocity_relative"
-    pose_with_covariance_topic="pose_with_covariance"
-    position_topic="position"
-    transform_topic="transform"
-    odometry_topic="odometry"
-    parent_frame_id="world"
-    mass_odometry_sensor="0.01"
-    measurement_divisor="5"
-    measurement_delay="0"
-    unknown_delay="0.0"
-    noise_normal_position="0.0 0.0 0.0"
-    noise_normal_quaternion="0.0 0.0 0.0"
-    noise_normal_linear_velocity="0.0 0.0 0.0"
-    noise_normal_angular_velocity="0.0 0.0 0.0"
-    noise_uniform_position="0.0 0.0 0.0"
-    noise_uniform_quaternion="0.0 0.0 0.0"
-    noise_uniform_linear_velocity="0.0 0.0 0.0"
-    noise_uniform_angular_velocity="0.0 0.0 0.0"
-    enable_odometry_map="false"
-    odometry_map=""
-    image_scale="">
-    <inertia ixx="0.00001" ixy="0.0" ixz="0.0" iyy="0.00001" iyz="0.0" izz="0.00001" /> <!-- [kg m^2] [kg m^2] [kg m^2] [kg m^2] [kg m^2] [kg m^2] -->
-    <origin xyz="0.0 0.0 0" rpy="0.0 0.0 0.0" />
-  </xacro:odometry_plugin_macro>
+  <xacro:if value="${'ground_truth' == odometry_type}">
+    <xacro:odometry_plugin_macro
+      namespace="$(arg name)"
+      odometry_sensor_suffix="1"
+      child_frame_id="base"
+      parent_link="base_link"
+      pose_topic="pose"
+      velocity_relative_topic="velocity_relative"
+      pose_with_covariance_topic="pose_with_covariance"
+      position_topic="position"
+      transform_topic="transform"
+      odometry_topic="odometry"
+      parent_frame_id="world"
+      mass_odometry_sensor="0.01"
+      measurement_divisor="5"
+      measurement_delay="0"
+      unknown_delay="0.0"
+      noise_normal_position="0.0 0.0 0.0"
+      noise_normal_quaternion="0.0 0.0 0.0"
+      noise_normal_linear_velocity="0.0 0.0 0.0"
+      noise_normal_angular_velocity="0.0 0.0 0.0"
+      noise_uniform_position="0.0 0.0 0.0"
+      noise_uniform_quaternion="0.0 0.0 0.0"
+      noise_uniform_linear_velocity="0.0 0.0 0.0"
+      noise_uniform_angular_velocity="0.0 0.0 0.0"
+      enable_odometry_map="false"
+      odometry_map=""
+      image_scale="">
+      <inertia ixx="0.00001" ixy="0.0" ixz="0.0" iyy="0.00001" iyz="0.0" izz="0.00001" /> <!-- [kg m^2] [kg m^2] [kg m^2] [kg m^2] [kg m^2] [kg m^2] -->
+      <origin xyz="0.0 0.0 0" rpy="0.0 0.0 0.0" />
+    </xacro:odometry_plugin_macro>
+  </xacro:if>
+  <xacro:if value="${'realistic' == odometry_type}">
+    <xacro:odometry_plugin_macro
+      namespace="$(arg name)"
+      odometry_sensor_suffix="1"
+      child_frame_id="base"
+      parent_link="base_link"
+      pose_topic="pose"
+      velocity_relative_topic="velocity_relative"
+      pose_with_covariance_topic="pose_with_covariance"
+      position_topic="position"
+      transform_topic="transform"
+      odometry_topic="odometry"
+      parent_frame_id="world"
+      mass_odometry_sensor="0.00001"
+      measurement_divisor="10"
+      measurement_delay="10"
+      unknown_delay="0.0"
+      noise_normal_position="0.01 0.01 0.01"
+      noise_normal_quaternion="0.017 0.017 0.017"
+      noise_normal_linear_velocity="0.0 0.0 0.0"
+      noise_normal_angular_velocity="0.0 0.0 0.0"
+      noise_uniform_position="0.0 0.0 0.0"
+      noise_uniform_quaternion="0.0 0.0 0.0"
+      noise_uniform_linear_velocity="0.0 0.0 0.0"
+      noise_uniform_angular_velocity="0.0 0.0 0.0"
+      enable_odometry_map="false"
+      odometry_map=""
+      image_scale="">
+      <inertia ixx="0.00001" ixy="0.0" ixz="0.0" iyy="0.00001" iyz="0.0" izz="0.00001" /> <!-- [kg m^2] [kg m^2] [kg m^2] [kg m^2] [kg m^2] [kg m^2] -->
+      <origin xyz="0.0 0.0 0" rpy="0.0 0.0 0.0" />
+    </xacro:odometry_plugin_macro>
+  </xacro:if>
   <xacro:if value="${'rod_with_camera' == manipulator_tool}">
     <xacro:odometry_plugin_macro

Commit message: Pruned everything currently uneccessary for me, model is spawning

File: mmuav_description/urdf/uav.gazebo.xacro (robot description, xacro)
@@ -12,22 +12,18 @@
     </plugin>
   </gazebo>
+  <!-- Add UAV base and component snippets -->
+  <xacro:include filename="$(find mmuav_description)/urdf/uav.base.urdf.xacro" />
+  <xacro:include filename="$(find rotors_description)/urdf/component_snippets.xacro" />
   <xacro:property name="enable_bag_plugin" value="false" />
   <xacro:property name="bag_file" value="uav.bag" />
   <xacro:arg name="mount_velodyne" default="false" />
   <xacro:property name="mount_velodyne" value="$(arg mount_velodyne)" />
-  <xacro:arg name="mount_magnet" default="false" />
-  <xacro:property name="mount_magnet" value="$(arg mount_magnet)" />
-  <xacro:arg name="mount_magnet_with_disk" default="false" />
-  <xacro:property name="mount_magnet_with_disk" value="$(arg mount_magnet_with_disk)" />
-  <xacro:arg name="magnet_dipole_moment_z" default="970" />
-  <xacro:property name="dp_z" value="$(arg magnet_dipole_moment_z)" />
   <xacro:arg name="mount_stereo_cam" default="false" />
   <xacro:property name="mount_stereo_cam" value="$(arg mount_stereo_cam)" />
   <xacro:arg name="turn_off_all_collisions" default="false" />
   <xacro:property name="turn_off_all_collisions" value="$(arg turn_off_all_collisions)" />
-  <xacro:arg name="manipulator_tool" default="none" />
-  <xacro:property name="manipulator_tool" value="$(arg manipulator_tool)" />
   <xacro:arg name="collision_bitmask" default="-1" />
   <xacro:property name="collision_bitmask" value="$(arg collision_bitmask)" />
+  <!-- Cam properties -->
 	<xacro:property name="front_facing_camera">
 		<origin xyz="0.025 0 0.1" rpy="0 0 0"/>
@@ -45,30 +41,4 @@
     ixy="0.0" ixz="0.0" iyz="0.0" />
   </xacro:property>
-  <!-- Instantiate mmuav "mechanics" -->
-  <xacro:include filename="$(find mmuav_description)/urdf/uav.base.urdf.xacro" />
-  <xacro:include filename="$(find rotors_description)/urdf/component_snippets.xacro" />
-  <!-- Create link and joint for a sensor -->
-  <gazebo reference="pose_sensor1_link">
-    <collision>
-      <surface>
-        <contact>
-          <collide_bitmask>${collision_bitmask}</collide_bitmask>
-        </contact>
-      </surface>
-    </collision>
-  </gazebo>
-  <link name="pose_sensor1_link">
-    <inertial>
-      <inertia ixx="0.00001" ixy="0.0" ixz="0.0" iyy="0.00001" iyz="0.0"
-        izz="0.00001" />
-      <mass value="0.01" />
-    </inertial>
-  </link>
-  <joint name="pose_sensor1_joint" type="revolute">
-    <parent link="base_link" />
-    <origin xyz="0 0 0" rpy="0 0 0" />
-    <child link="pose_sensor1_link" />
-    <limit upper="0" lower="0" effort="0" velocity="0" />
-  </joint>
   <xacro:property name="horizontal_velodyne_origin">
     <origin xyz="0 0 -0.025" rpy="3.141592653589793 0.1323284641020683 0." />
@@ -105,52 +75,4 @@
     </VU-8>
   </xacro:if>
-  <xacro:if value="${mount_magnet}">
-    <xacro:if value="${mount_magnet_with_disk}">
-      <joint name="electromagnet_joint" type="fixed">
-        <axis xyz="0 1 0" />
-        <origin xyz="0.0 0.0 -0.15" rpy="0 0 0"/>
-        <parent link="base_link"/>
-        <child link="electromagnet_actuator"/>
-      </joint>
-      <gazebo reference="electromagnet_actuator">
-        <collision>
-          <surface>
-            <contact>
-              <collide_bitmask>${collision_bitmask}</collide_bitmask>
-            </contact>
-          </surface>
-        </collision>
-      </gazebo>
-      <link name="electromagnet_actuator">
-        <inertial>
-        <origin xyz="0 0 0" rpy="0 0 0" />
-        <mass value="0.025"/>
-        <inertia ixx="0.0001" ixy="0" ixz="0" iyy ="0.0001" iyz = "0" izz = "0.0001" />
-        </inertial>
-        <collision name="collision">
-        <geometry>
-          <cylinder radius="0.08" length="0.035"/>
-        </geometry>
-        </collision>
-        <visual>
-        <geometry>
-          <cylinder radius="0.08" length="0.035"/>
-        </geometry>
-        </visual>
-      </link>
-    </xacro:if>
-    <gazebo>
-      <plugin name="dipole_magnet" filename="libstorm_gazebo_dipole_magnet.so">
-        <robotNamespace>$(arg name)</robotNamespace>
-        <bodyName>base_link</bodyName>
-        <dipole_moment>0 0 ${dp_z}</dipole_moment>
-        <!-- Set to false if not using ROS -->
-        <shouldPublish>true</shouldPublish>
-        <topicNs>magnet</topicNs>
-        <updateRate>100</updateRate>
-        <gain>1.0</gain>
-      </plugin>
-    </gazebo>
-  </xacro:if>
   <!-- Mount first generic pose sensor-->
   <xacro:odometry_plugin_macro
@@ -184,41 +106,4 @@
     <origin xyz="0.0 0.0 0" rpy="0.0 0.0 0.0" />
   </xacro:odometry_plugin_macro>
-  <xacro:if value="${'rod_with_camera' == manipulator_tool}">
-    <xacro:odometry_plugin_macro
-    namespace="$(arg name)"
-    odometry_sensor_suffix="2"
-    child_frame_id="base"
-    parent_link="camera_box"
-    pose_topic="camera/pose"
-    velocity_relative_topic="camera/velocity_relative"
-    pose_with_covariance_topic="camera/pose_with_covariance"
-    position_topic="camera/position"
-    transform_topic="camera/transform"
-    odometry_topic="camera/odometry"
-    parent_frame_id="world"
-    mass_odometry_sensor="1e-5"
-    measurement_divisor="5"
-    measurement_delay="0"
-    unknown_delay="0.0"
-    noise_normal_position="0.0 0.0 0.0"
-    noise_normal_quaternion="0.0 0.0 0.0"
-    noise_normal_linear_velocity="0.0 0.0 0.0"
-    noise_normal_angular_velocity="0.0 0.0 0.0"
-    noise_uniform_position="0.0 0.0 0.0"
-    noise_uniform_quaternion="0.0 0.0 0.0"
-    noise_uniform_linear_velocity="0.0 0.0 0.0"
-    noise_uniform_angular_velocity="0.0 0.0 0.0"
-    enable_odometry_map="false"
-    odometry_map=""
-    image_scale="">
-    <inertia ixx="1e-6" ixy="0.0" ixz="0.0" iyy="1e-6" iyz="0.0" izz="1e-6" /> <!-- [kg m^2] [kg m^2] [kg m^2] [kg m^2] [kg m^2] [kg m^2] -->
-    <!-- This rotation is correction for blender. -->
-    <origin xyz="0.0 0.0 0" rpy="1.57 0.0 -1.57" />
-  </xacro:odometry_plugin_macro>
-  </xacro:if>
-  <!-- mount gimbal -->
-  <!--<xacro:gimbal_macro parent="base_link">
-    <origin xyz="0.25 0 -0.05" rpy="0 0 0"/>
-  </xacro:gimbal_macro> -->
   <xacro:if value="${mount_stereo_cam}">
     <xacro:stereo_cam
@@ -231,12 +116,3 @@
     </xacro:stereo_cam>
   </xacro:if>
-  <!--gazebo reference="rod">
-    <collision>
-      <surface>
-        <contact>
-          <collide_bitmask>0x01</collide_bitmask>
-        </contact>
-      </surface>
-    </collision>
-  </gazebo-->
 </robot>
