Commit message: added joint control

File: mmuav_description/urdf/multirotor_base.urdf.xacro (robot description, xacro)
@@ -24,12 +24,12 @@
         </geometry>
       </visual>
-      <collision>
+      <!--collision>
         <origin xyz="0 0 0" rpy="0 0 0" />
         <geometry>
           <mesh filename="package://mmuav_description/meshes/${mesh_file}"
             scale="1 1 1" />
-          <!--box size="${body_width} ${body_width} ${body_height}" /--> <!-- [m] [m] [m] -->
-        </geometry>
-      </collision>
+          <box size="${body_width} ${body_width} ${body_height}" />
+        </geometry>
+      </collision-->
     </link>
     <!-- IMU -->
@@ -214,9 +214,9 @@
       </visual>
       <collision name='collision'>
-        <origin xyz="0 0 0" rpy="0 0 0"/>
-        <geometry>
-          <mesh filename="package://mmuav_description/meshes/AX12.dae"
-            scale="1 1 1" />
-           <!--box size="0.05 0.041 0.032"/-->
+        <origin xyz="0.01261097 0 0.00120978" rpy="0 0 0"/>
+        <geometry>
+          <!--mesh filename="package://mmuav_description/meshes/AX12.dae"
+            scale="1 1 1" /-->
+           <box size="0.05 0.041 0.032"/>
         </geometry>
       </collision>
@@ -227,11 +227,10 @@
     <link name='link_F3_fixed_${suffix}'>
       <inertial>
-        <mass value="0.055" />
-        <origin xyz="0 0 0" rpy="0 0 0"/>
-        <inertia
-          ixx="0.001"
-          iyy="0"
-          izz="0"
-          ixy="0.0" ixz="0.0" iyz="0.0" />
+        <mass value="0.00323" />
+        <origin xyz="0.00000191 0.00240389 0" rpy="0 0 0"/>
+        <inertia
+          ixx="0.00000047" ixy="0" ixz="0.0"
+          iyx="0" iyy="0.00000065" iyz="0"
+          izx="0.0" izy="0" izz="0.00000020"/>
       </inertial>
       <visual>
@@ -242,12 +241,4 @@
         </geometry>
       </visual>
-      <collision name='collision'>
-        <origin xyz="0 0 0" rpy="0 0 0"/>
-        <geometry>
-          <mesh filename="package://mmuav_description/meshes/F3.dae"
-            scale="1 1 1" />
-           <!--box size="0.05 0.041 0.032"/-->
-        </geometry>
-      </collision>
     </link>
     <!--_____________________________________________________________-->
@@ -256,11 +247,10 @@
     <link name='link_F4_fixed_${suffix}'>
       <inertial>
-        <mass value="0.055" />
-        <origin xyz="0 0 0" rpy="0 0 0"/>
-        <inertia
-          ixx="0"
-          iyy="0"
-          izz="0"
-          ixy="0.0" ixz="0.0" iyz="0.0" />
+        <mass value="0.01" />
+        <origin xyz="0 -0.03040000 -0.00860000" rpy="0 0 0"/>
+        <inertia
+          ixx="0.00000845" ixy="0" ixz="0.0"
+          iyx="0" iyy="0.00000180" iyz="-0.00000279"
+          izx="0.0" izy="-0.00000279" izz="0.00000750"/>
       </inertial>
       <visual>
@@ -271,12 +261,4 @@
         </geometry>
       </visual>
-      <collision name='collision'>
-        <origin xyz="0 0 0" rpy="0 0 0"/>
-        <geometry>
-          <mesh filename="package://mmuav_description/meshes/F4.dae"
-            scale="1 1 1" />
-           <!--box size="0.05 0.041 0.032"/-->
-        </geometry>
-      </collision>
     </link>
     <!--_____________________________________________________________-->
@@ -300,9 +282,9 @@
       </visual>
       <collision name='collision'>
-        <origin xyz="0 0 0" rpy="0 0 0"/>
-        <geometry>
-          <mesh filename="package://mmuav_description/meshes/AX12.dae"
-            scale="1 1 1" />
-           <!--box size="0.05 0.041 0.032"/-->
+        <origin xyz="0.01261097 0 0.00120978" rpy="0 0 0"/>
+        <geometry>
+          <!--mesh filename="package://mmuav_description/meshes/AX12.dae"
+            scale="1 1 1" /-->
+           <box size="0.05 0.041 0.032"/>
         </geometry>
       </collision>
@@ -313,11 +295,10 @@
     <link name='link_gripper1_${suffix}'>
       <inertial>
-        <mass value="0.055" />
-        <origin xyz="0 0 0" rpy="0 0 0"/>
-        <inertia
-          ixx="0"
-          iyy="0"
-          izz="0"
-          ixy="0.0" ixz="0.0" iyz="0.0" />
+        <mass value="0.0109" />
+        <origin xyz="0.00028510 0.00103830 0.00134070" rpy="0 0 0"/>
+        <inertia
+          ixx="0.00000124" ixy="0" ixz="0.0"
+          iyx="0" iyy="0.00000170" iyz="0"
+          izx="0.0" izy="0" izz="0.00000137"/>
       </inertial>
       <visual>
@@ -328,12 +309,4 @@
         </geometry>
       </visual>
-      <collision name='collision'>
-        <origin xyz="0 0 0" rpy="0 0 0"/>
-        <geometry>
-          <mesh filename="package://mmuav_description/meshes/gripper_part1.dae"
-            scale="1 1 1" />
-           <!--box size="0.05 0.041 0.032"/-->
-        </geometry>
-      </collision>
     </link>
     <!--_____________________________________________________________-->
@@ -399,6 +372,7 @@
       <child link="link_gripper2_${suffix}" />
       <origin xyz="0.01265148 0.00103883 0.00134042" rpy="0 0 0"/>
-      <limit upper="1.79769e+308" lower="-1.79769e+308" effort="10" velocity="1"/>
+      <limit upper="1.0471975512" lower="-1.0471975512" effort="10" velocity="1"/>
       <axis xyz="0 1 0" />
+      <dynamics damping="0.0" friction="0.04"/>
     </joint>
   </xacro:macro>

Commit message: Corrected joint offsets for manipulator.

File: mmuav_description/urdf/multirotor_base.urdf.xacro (robot description, xacro)
@@ -343,5 +343,5 @@
       <child link="dynamixel_1_${suffix}" />
       <xacro:insert_block name="origin"/>
-      <limit upper="2" lower="-2" effort="10" velocity="1"/>
+      <limit upper="3.14" lower="-3.14" effort="10" velocity="1"/>
       <xacro:insert_block name="axis"/>
     </joint>
@@ -360,5 +360,5 @@
       <child link="dynamixel_2_${suffix}" />
       <origin xyz="0 0 0" rpy="0 0 0"/>
-      <limit upper="1.79769e+308" lower="-1.79769e+308" effort="10" velocity="1"/>
+      <limit upper="3.14" lower="-3.14" effort="10" velocity="1"/>
       <axis xyz="0 1 0" />
     </joint>
@@ -372,5 +372,5 @@
       <child link="link_gripper2_${suffix}" />
       <origin xyz="0.01265148 0.00103883 0.00134042" rpy="0 0 0"/>
-      <limit upper="1.0471975512" lower="-1.0471975512" effort="10" velocity="1"/>
+      <limit upper="1.57" lower="-1.57" effort="10" velocity="1"/>
       <axis xyz="0 1 0" />
       <dynamics damping="0.0" friction="0.04"/>

Commit message: added position controller, new joint parameters

File: mmuav_description/urdf/multirotor_base.urdf.xacro (robot description, xacro)
@@ -410,5 +410,5 @@
       <child link="link_dynamixel2_${suffix}"/>
       <origin xyz="0 0 0" rpy="0 0 ${-PI/2}" />
-      <limit upper="6" lower="-6" effort="1.5" velocity="1"/>
+      <limit upper="6" lower="-6" effort="0.3" velocity="0.1"/>
       <axis xyz="0 0 1" />
     </joint>
@@ -427,6 +427,6 @@
       <parent link="link_gripper1_${suffix}"/>
       <child link="link_gripper2_${suffix}"/>
-      <origin xyz="0.01265 0.00104 -0.00134" rpy="0 0 0" />
-      <limit upper="0" lower="0" effort="1.5" velocity="1"/>
+      <origin xyz="0.01265 0.00104 -0.00134" rpy="0 0 ${PI}" />
+      <limit upper="6" lower="-6" effort="0.05" velocity="0.01"/>
       <axis xyz="0 0 1" />
     </joint>

Commit message: Added collision object for uav central body. Reduce dynamics damping of the mm joints.

File: mmuav_description/urdf/multirotor_base.urdf.xacro (robot description, xacro)
@@ -24,12 +24,12 @@
         </geometry>
       </visual>
-      <!--collision>
-        <origin xyz="0 0 0" rpy="0 0 0" />
-        <geometry>
-          <mesh filename="package://mmuav_description/meshes/${mesh_file}"
-            scale="1 1 1" />
+      <collision>
+        <origin xyz="0 0 0" rpy="0 0 0" />
+        <geometry>
+          <!--mesh filename="package://mmuav_description/meshes/${mesh_file}"
+            scale="1 1 1" /-->
           <box size="${body_width} ${body_width} ${body_height}" />
         </geometry>
-      </collision-->
+      </collision>
     </link>
     <!-- IMU -->
@@ -430,6 +430,6 @@
       <parent link="${parent}"/>
       <child link="movable_mass_${mass_number}"/>
-      <limit lower="${-path_len/2}" upper="${path_len/2}" effort="10000" velocity="20"/>
-      <dynamics damping="10" />
+      <limit lower="${-path_len/2}" upper="${path_len/2}" effort="50" velocity="5"/>
+      <dynamics damping="0.2" />
     </joint>
     <link name="movable_mass_${mass_number}">

Commit message: Fixed minor errors

File: mmuav_description/urdf/multirotor_base.urdf.xacro (robot description, xacro)
@@ -456,3 +456,114 @@
     </gazebo>
   </xacro:macro>
+  <xacro:macro name="camera_manipulator"
+  params="parent link_mass link_ixx link_iyy link_izz *origin">
+    <material name="blue">
+      <color rgba="0 0 0.8 1"/>
+    </material>
+    <material name="red">
+      <color rgba="1 0 0 1"/>
+    </material>
+    <link name='connector1'>
+      <inertial>
+        <mass value="0.00251" />
+        <origin xyz="0 0 -0.01" rpy="0 0 0"/>
+        <inertia
+          ixx="0.00001176" ixy="0" ixz="0"
+          iyx="0" iyy="0.00001176" iyz="0"
+          izx="0" izy="0" izz="0.00000252"/>
+      </inertial>
+      <visual>
+        <origin xyz="0 0 -0.01" rpy="0 0 0" />
+        <geometry>
+          <cylinder length="0.02" radius="0.02"/>
+        </geometry>
+      </visual>
+    </link>
+    <link name='link1'>
+      <inertial>
+        <mass value="${link_mass}" />
+        <origin xyz="-0.09899494936 0.09899494936 -0.01" rpy="0 0 0"/>
+        <inertia
+          ixx="${link_ixx}" ixy="0" ixz="0"
+          iyx="0" iyy="${link_iyy}" iyz="0"
+          izx="0" izy="0" izz="${link_izz}"/>
+      </inertial>
+      <visual>
+        <origin xyz="-0.09899494936 0.09899494936 -0.01" rpy="0.7853981634 1.570796327 0" />
+        <geometry>
+          <box size="0.02 0.04 0.32"/>
+        </geometry>
+      </visual>
+    </link>
+    <link name='connector2'>
+      <inertial>
+        <mass value="0.00251" />
+        <origin xyz="0 0 0" rpy="0 0 0"/>
+        <inertia
+          ixx="00001176" ixy="0" ixz="0"
+          iyx="0" iyy="0.00001176" iyz="0"
+          izx="0" izy="0" izz="0.00000252"/>
+      </inertial>
+      <visual>
+        <origin xyz="0 0 -0.02" rpy="0 0 0" />
+        <geometry>
+          <cylinder length="0.02" radius="0.02"/>
+        </geometry>
+      </visual>
+    </link>
+    <link name='link2'>
+      <inertial>
+        <mass value="${link_mass}" />
+        <origin xyz="-0.09899494936 0.09899494936 -0.02" rpy="0 0 0"/>
+        <inertia
+          ixx="${link_ixx}" ixy="0" ixz="0"
+          iyx="0" iyy="${link_iyy}" iyz="0"
+          izx="0" izy="0" izz="${link_izz}"/>
+    </inertial>
+      <visual>
+        <origin xyz="-0.09899494936 0.09899494936 -0.02" rpy="0.7853981634 1.570796327 0" />
+        <geometry>
+          <box size="0.02 0.04 0.32"/>
+        </geometry>
+      </visual>
+    </link>
+    <joint name="base_to_connector1" type="fixed">
+      <parent link="${parent}"/>
+      <child link="connector1"/>
+      <xacro:insert_block name="origin"/>
+    </joint>
+    <joint name="connector1_to_link1" type="continuous">
+      <parent link="connector1"/>
+      <child link="link1"/>
+      <origin xyz="0 0 -0.02" rpy="0 0 0"/>
+      <limit upper="3.14" lower="-3.14" effort="10000000" velocity="20"/>
+      <axis xyz="0 0 1" />
+      <dynamics damping="0.00" friction="0.0"/>
+    </joint>
+    <joint name="link1_to_connector2" type="fixed">
+      <parent link="link1"/>
+      <child link="connector2"/>
+      <origin xyz="-0.19798989873 0.19798989873 -0.01" rpy="0 0 0"/>
+    </joint>
+    <joint name="connector2_to_link2" type="continuous">
+      <parent link="connector2"/>
+      <child link="link2"/>
+      <origin xyz="0 0 -0.02" rpy="0 0 0"/>
+      <limit upper="3.14" lower="-3.14" effort="10000000" velocity="20"/>
+      <axis xyz="0 0 1" />
+      <dynamics damping="0.07" friction="0.0"/>
+    </joint>
+    <gazebo reference="link1">
+      <material>Gazebo/Blue</material>
+    </gazebo>
+    <gazebo reference="link2">
+      <material>Gazebo/Blue</material>
+    </gazebo>
+    <gazebo reference="connector1">
+      <material>Gazebo/Red</material>
+    </gazebo>
+    <gazebo reference="connector2">
+      <material>Gazebo/Red</material>
+    </gazebo>
+  </xacro:macro>
 </robot>

File: mmuav_description/urdf/uav.base.urdf.xacro (robot description, xacro)
@@ -147,101 +147,55 @@
     <xacro:insert_block name="rotor_inertia" />
   </xacro:vertical_rotor>
-  <link name='connector1'>
-    <inertial>
-      <mass value="0.0126" />
-      <origin xyz="0 0 -0.04" rpy="0 0 0"/>
-      <inertia
-        ixx="0.00001176" ixy="0" ixz="0"
-        iyx="0" iyy="0.00001176" iyz="0"
-        izx="0" izy="0" izz="0.00000252"/>
-    </inertial>
-    <visual>
-      <origin xyz="0 0 -0.04" rpy="0 0 0" />
-      <geometry>
-        <cylinder length="0.1" radius="0.02"/>
-      </geometry>
-    </visual>
-  </link>
-  <link name='link1'>
-    <inertial>
-      <mass value="0.0256" />
-      <origin xyz="-0.09899494936 0.09899494936 -0.01" rpy="0 0 0"/>
-      <inertia
-        ixx="0.000004266" ixy="0" ixz="0"
-        iyx="0" iyy="0.002" iyz="0"
-        izx="0" izy="0" izz="0.000262827"/>
-    </inertial>
-    <visual>
-      <origin xyz="-0.09899494936 0.09899494936 -0.01" rpy="0.758398 1.5708 0" />
-      <geometry>
-        <box size="0.02 0.04 0.32"/>
-      </geometry>
-    </visual>
-  </link>
-    <link name='connector2'>
-      <inertial>
-        <mass value="0.00251" />
-        <origin xyz="0 0 0" rpy="0 0 0"/>
-        <inertia
-          ixx="0.0000003346" ixy="0" ixz="0"
-          iyx="0" iyy="0.0000003346" iyz="0"
-          izx="0" izy="0" izz="0.000000502"/>
-      </inertial>
-      <visual>
-        <origin xyz="0 0 -0.02" rpy="0 0 0" />
-        <geometry>
-          <cylinder length="0.02" radius="0.02"/>
-        </geometry>
-      </visual>
-    </link>
-    <link name='link2'>
-      <inertial>
-        <mass value="0.0256" />
-        <origin xyz="-0.09899494936 0.09899494936 -0.02" rpy="0 0 0"/>
-        <inertia
-          ixx="0.000004266" ixy="0" ixz="0"
-          iyx="0" iyy="0.002" iyz="0"
-          izx="0" izy="0" izz="0.000262827"/>
-    </inertial>
-      <visual>
-        <origin xyz="-0.09899494936 0.09899494936 -0.02" rpy="0.758398 1.5708 0" />
-        <geometry>
-          <box size="0.02 0.04 0.32"/>
-        </geometry>
-      </visual>
-    </link>
-    <joint name="base_to_connector1" type="fixed">
-      <parent link="base_link"/>
-      <child link="connector1"/>
-      <origin xyz="0 0 0" rpy="0 0 0"/>
-    </joint>
-    <joint name="connector1_to_link1" type="continuous">
-      <parent link="connector1"/>
-      <child link="link1"/>
-      <origin xyz="0 0 -0.09" rpy="0 0 0"/>
-      <limit upper="3.14" lower="-3.14" effort="10000000" velocity="20"/>
-      <axis xyz="0 0 1" />
-      <dynamics damping="0.07" friction="0.0"/>
-    </joint>
-    <joint name="link1_to_connector2" type="fixed">
-      <parent link="link1"/>
-      <child link="connector2"/>
-      <origin xyz="-0.19798989873 0.19798989873 -0.01" rpy="0 0 0"/>
-    </joint>
-    <joint name="connector2_to_link2" type="continuous">
-      <parent link="connector2"/>
-      <child link="link2"/>
-      <origin xyz="0 0 -0.02" rpy="0 0 0"/>
-      <limit upper="3.14" lower="-3.14" effort="10000000" velocity="20"/>
-      <axis xyz="0 0 1" />
-      <dynamics damping="0.07" friction="0.0"/>
-    </joint>
-    <xacro:transmisija
-      trans_number="0"
-      joint_name="connector1_to_link1">
-    </xacro:transmisija>
-    <xacro:transmisija
-      trans_number="1"
-      joint_name="connector2_to_link2">
-    </xacro:transmisija>
+<!--
+  <xacro:camera_manipulator
+    parent="base_link"
+    link_mass="0.25"
+    link_ixx="0.00004167"
+    link_iyy="0.00854167"
+    link_izz="0.00856667" >
+    <origin xyz="0 0 0" rpy="0 0 0"/>
+  </xacro:camera_manipulator>
+-->
+<!--
+  <xacro:camera_manipulator
+    parent="base_link"
+    link_mass="0.05"
+    link_ixx="0.00000833"
+    link_iyy="0.00170833"
+    link_izz="0.00171333" >
+    <origin xyz="0 0 0" rpy="0 0 0"/>
+  </xacro:camera_manipulator>
+-->
+  <xacro:camera_manipulator
+    parent="base_link"
+    link_mass="0.005"
+    link_ixx="0.00000083"
+    link_iyy="0.00017083"
+    link_izz="0.00017133" >
+    <origin xyz="0 0 0" rpy="0 0 0"/>
+  </xacro:camera_manipulator>
+  <xacro:transmisija
+    trans_number="0"
+    joint_name="connector1_to_link1">
+  </xacro:transmisija>
+  <xacro:transmisija
+    trans_number="1"
+    joint_name="connector2_to_link2">
+  </xacro:transmisija>
+  <xacro:property name="camera_link" value="0.05" />
+  <xacro:property name="camera_inertia">
+    <inertia
+    ixx="1e-8"
+    iyy="1e-8"
+    izz="1e-8"
+    ixy="0.0" ixz="0.0" iyz="0.0" />
+  </xacro:property>
+  <xacro:property name="camera_mass" value="1e-5"/>
+  <xacro:cam
+    camera_link="${camera_link}"
+    camera_mass="${camera_mass}"
+    parent="link2">
+    <origin xyz="-0.2121320344 0.2121320344 0.02" rpy="0 0 0"/>
+    <xacro:insert_block name="camera_inertia"/>
+  </xacro:cam>
 </robot>

Commit message: Camera manipulator model build - WIP

File: mmuav_description/urdf/multirotor_base.urdf.xacro (robot description, xacro)
@@ -567,3 +567,28 @@
     </gazebo>
   </xacro:macro>
+  <xacro:macro name="c_manip"
+  params="parent link_mass link_ixx link_iyy link_izz *origin">
+    <link name='connector1'>
+      <inertial>
+        <mass value="0.1" />
+        <origin xyz="0 0 -0.01" rpy="0 0 0"/>
+        <inertia
+          ixx="0.01176" ixy="0" ixz="0"
+          iyx="0" iyy="0.01176" iyz="0"
+          izx="0" izy="0" izz="0.0252"/>
+      </inertial>
+      <visual>
+        <origin xyz="0 0 0" rpy="0 0 0" />
+        <geometry>
+          <mesh filename="package://mmuav_description/meshes/link1.dae"
+            scale="1 1 1" />
+        </geometry>
+      </visual>
+    </link>
+    <joint name="base_to_connector1" type="fixed">
+      <parent link="${parent}"/>
+      <child link="connector1"/>
+      <xacro:insert_block name="origin"/>
+    </joint>
+  </xacro:macro>
 </robot>

File: mmuav_description/urdf/uav.base.urdf.xacro (robot description, xacro)
@@ -167,12 +167,13 @@
   </xacro:camera_manipulator>
 -->
-  <xacro:camera_manipulator
+  <xacro:c_manip
     parent="base_link"
     link_mass="0.005"
-    link_ixx="0.00000083"
+    link_ixx="0.0000083"
     link_iyy="0.00017083"
     link_izz="0.00017133" >
     <origin xyz="0 0 0" rpy="0 0 0"/>
-  </xacro:camera_manipulator>
+  </xacro:c_manip>
+<!--
   <xacro:transmisija
     trans_number="0"
@@ -199,3 +200,4 @@
     <xacro:insert_block name="camera_inertia"/>
   </xacro:cam>
+-->
 </robot>

Commit message: added ttc control

File: mmuav_description/urdf/multirotor_base.urdf.xacro (robot description, xacro)
@@ -24,12 +24,12 @@
         </geometry>
       </visual>
-      <!--collision>
+      <collision>
         <origin xyz="0 0 0" rpy="0 0 0" />
         <geometry>
           <mesh filename="package://mmuav_description/meshes/${mesh_file}"
             scale="1 1 1" />
-          <box size="${body_width} ${body_width} ${body_height}" />
-        </geometry>
-      </collision-->
+          <!--box size="${body_width} ${body_width} ${body_height}" /-->
+        </geometry>
+      </collision>
     </link>
     <!-- IMU -->
@@ -110,4 +110,40 @@
     </gazebo>
     <gazebo reference="rotor_${motor_number}">
+      <material>Gazebo/${color}</material>
+    </gazebo>
+  </xacro:macro>
+  <!-- Macro file for tilted props. It defines joint between prop and body, and link which defines actual joint. Stick
+  is defined in other macro file-->
+  <xacro:macro name="tilt" params="parent motor_number x_axis y_axis color mass length radius *origin">
+    <joint name="tilt_${motor_number}_joint" type="revolute">
+      <xacro:insert_block name="origin"/>
+      <axis xyz="${x_axis} ${y_axis} 0"/>
+      <parent link="${parent}"/>
+      <child link="tilt_${motor_number}"/>
+      <limit lower="-0.785398163" upper="0.785398163" effort="100000" velocity="3"/>
+    </joint>
+    <link name="tilt_${motor_number}">
+      <visual>
+        <origin rpy="0 0 0" xyz="0 0 ${length/2}"/>
+        <geometry>
+          <cylinder length="${length}" radius="${radius}" />
+        </geometry>
+      </visual>
+      <collision>
+        <origin rpy="0 0 0" xyz="0 0 ${length/2}"/>
+        <geometry>
+            <cylinder length="${length}" radius="${radius}" />
+        </geometry>
+      </collision>
+      <inertial>
+          <origin rpy="0 0 0" xyz="0 0 ${length/2}"/>
+          <mass value="${mass}" />
+          <inertia
+            ixx="${5/12 * mass * (3.0 * radius * radius + length * length)}"  ixy="0.0" ixz="0.0"
+            iyx="0.0" iyy="${5/12 * mass * (3.0 * radius * radius + length * length)}" iyz="0.0"
+            izx="0.0" izy="0.0" izz="${5/2 * mass * radius * radius}" />
+      </inertial>
+    </link>
+    <gazebo reference="tilt_${motor_number}">
       <material>Gazebo/${color}</material>
     </gazebo>
