Commit message: added ducted fan control

File: mmuav_description/urdf/multirotor_base.urdf.xacro (robot description, xacro)
@@ -113,4 +113,78 @@
     </gazebo>
   </xacro:macro>
+<!-- ducted fan joint and link -->
+  <xacro:macro name="ducted_fan"
+    params="robot_namespace suffix direction motor_constant moment_constant area_control_flap area_antitorque_flap fluid_density distance_control_flap distance_antitorque_flap thrust_coefficient torque_coefficient slip_velocity_coefficient lift_coefficient_control_flap drag_coefficient_control_flap lift_coefficient_antitorque_flap drag_coefficient_antitorque_flap lift_coefficient_control_flap_at0 drag_coefficient_control_flap_at0 lift_coefficient_antitorque_flap_at0 drag_coefficient_antitorque_flap_at0 parent mass_rotor radius_rotor time_constant_up time_constant_down max_rot_velocity motor_number rotor_drag_coefficient rolling_moment_coefficient color *origin *inertia">
+    <joint name="rotor_${motor_number}_joint" type="continuous">
+      <xacro:insert_block name="origin" />
+      <axis xyz="0 0 1" />
+      <!-- TODO(ff): not currently set because it's not yet supported -->
+      <!-- <limit effort="2000" velocity="${max_rot_velocity}" /> -->
+      <parent link="${parent}" />
+      <child link="rotor_${motor_number}" />
+    </joint>
+    <!-- TODO(ff): not currently set because it's not yet supported -->
+    <!-- <gazebo reference="rotor_${motor_number}_joint"> <axis> <xyz>0 0 1</xyz>
+      <limit> <velocity> ${max_rot_velocity} </velocity> </limit> </axis> </gazebo> -->
+    <link name="rotor_${motor_number}">
+      <inertial>
+        <mass value="${mass_rotor}" /> <!-- [kg] -->
+        <xacro:insert_block name="inertia" />
+      </inertial>
+      <visual>
+        <geometry>
+          <!-- <cylinder length="0.005" radius="${radius_rotor}"/> --> <!-- [m] -->
+          <mesh filename="package://mmuav_description/meshes/propeller_${direction}.dae"
+            scale="0.001 0.001 0.001" />
+          <!-- <box size="${2*radius_rotor} 0.01 0.005"/> -->
+        </geometry>
+      </visual>
+      <collision>
+        <geometry>
+          <cylinder length="0.005" radius="${radius_rotor}" /> <!-- [m] -->
+        </geometry>
+      </collision>
+    </link>
+    <gazebo>
+      <plugin name="${suffix}_motor_model" filename="libmmuav_gazebo_ductedfan_motor_model.so">
+        <jointName>rotor_${motor_number}_joint</jointName>
+        <linkName>rotor_${motor_number}</linkName>
+        <turningDirection>${direction}</turningDirection>
+        <timeConstantUp>${time_constant_up}</timeConstantUp>
+        <timeConstantDown>${time_constant_down}</timeConstantDown>
+        <maxRotVelocity>${max_rot_velocity}</maxRotVelocity>
+        <motorConstant>${motor_constant}</motorConstant>
+        <momentConstant>${moment_constant}</momentConstant>
+        <commandSubTopic>${robot_namespace}/command/motors</commandSubTopic>
+        <motorNumber>${motor_number}</motorNumber>
+        <rotorDragCoefficient>${rotor_drag_coefficient}</rotorDragCoefficient>
+        <rollingMomentCoefficient>${rolling_moment_coefficient}</rollingMomentCoefficient>
+        <motorVelocityTopic>${robot_namespace}/motor_vel/${motor_number}</motorVelocityTopic>
+        <rotorVelocitySlowdownSim>${rotor_velocity_slowdown_sim}</rotorVelocitySlowdownSim>
+        <angleControlFlapRefSubTopic>${robot_namespace}/angle_wing_${motor_number}_ref_value</angleControlFlapRefSubTopic>
+        <angleControlFlapCommandPubTopic>${robot_namespace}/angle_wing_${motor_number}_controller/command</angleControlFlapCommandPubTopic>
+        <angleControlFlapValueSubTopic>${robot_namespace}/angle_wing_${motor_number}_controller/state</angleControlFlapValueSubTopic>
+        <fluidDensity>${fluid_density}</fluidDensity>
+        <areaControlFlap>${area_control_flap}</areaControlFlap>
+        <areaAntitorqueFlap>${area_antitorque_flap}</areaAntitorqueFlap>
+        <distanceControlFlap>${distance_control_flap}</distanceControlFlap>
+        <distanceAntitorqueFlap>${distance_antitorque_flap}</distanceAntitorqueFlap>
+        <thrustCoefficient>${thrust_coefficient}</thrustCoefficient>
+        <torqueCoefficient>${torque_coefficient}</torqueCoefficient>
+        <slipVelocityCoefficient>${slip_velocity_coefficient}</slipVelocityCoefficient>
+        <liftCoefficientControlFlap>${lift_coefficient_control_flap}</liftCoefficientControlFlap>
+        <dragCoefficientControlFlap>${drag_coefficient_control_flap}</dragCoefficientControlFlap>
+        <liftCoefficientAntitorqueFlap>${lift_coefficient_antitorque_flap}</liftCoefficientAntitorqueFlap>
+        <dragCoefficientAntitorqueFlap>${drag_coefficient_antitorque_flap}</dragCoefficientAntitorqueFlap>
+        <liftCoefficientControlFlapAt0>${lift_coefficient_control_flap_at0}</liftCoefficientControlFlapAt0>
+        <dragCoefficientControlFlapAt0>${drag_coefficient_control_flap_at0}</dragCoefficientControlFlapAt0>
+        <liftCoefficientAntitorqueFlapAt0>${lift_coefficient_antitorque_flap_at0}</liftCoefficientAntitorqueFlapAt0>
+        <dragCoefficientAntitorqueFlapAt0>${drag_coefficient_antitorque_flap_at0}</dragCoefficientAntitorqueFlapAt0>
+      </plugin>
+    </gazebo>
+    <gazebo reference="rotor_${motor_number}">
+      <material>Gazebo/${color}</material>
+    </gazebo>
+  </xacro:macro>
   <!-- Macro file for tilted props. It defines joint between prop and body, and link which defines actual joint. Stick
   is defined in other macro file-->
@@ -146,4 +220,37 @@
     </link>
     <gazebo reference="tilt_${motor_number}">
+      <material>Gazebo/${color}</material>
+    </gazebo>
+  </xacro:macro>
+  <!-- Macro file for the wing. It defines joint between base and wing.-->
+  <xacro:macro name="wing"
+     params="robot_namespace parent wing_number mass wing_x wing_y wing_z x_axis y_axis color *origin *inertia">
+    <joint name="wing_${wing_number}_joint" type="revolute">
+    <xacro:insert_block name="origin" />
+      <axis xyz="${x_axis} ${y_axis} 0"/>
+      <parent link="${parent}"/>
+      <child link="wing_${wing_number}"/>
+      <limit lower="-0.785398163" upper="0.785398163" effort="10000" velocity="10"/>
+    </joint>
+    <link name="wing_${wing_number}">
+      <visual>
+        <origin rpy="0 0 0" xyz="0 0 0"/>
+        <geometry>
+          <box size="${1*wing_x} ${1*wing_y} ${1*wing_z}"/>
+        </geometry>
+      </visual>
+      <!--collision>
+        <origin rpy="0 0 0" xyz="0 0 0"/>
+        <geometry>
+          <box size="${wing_x} ${wing_y} ${wing_z}"/>
+        </geometry>
+      </collision-->
+      <inertial>
+        <origin rpy="0 0 0" xyz="0 0 0"/>
+        <mass value="${wing_mass}"/>
+        <xacro:insert_block name="inertia"/>
+      </inertial>
+    </link>
+    <gazebo reference="wing_${wing_number}">
       <material>Gazebo/${color}</material>
     </gazebo>

Commit message: g

File: mmuav_description/urdf/multirotor_base.urdf.xacro (robot description, xacro)
@@ -493,5 +493,5 @@
     <link name='link_gripper2_${suffix}'>
       <inertial>
-        <mass value="0.25" />
+        <mass value="0.5" />
         <!-- origin xyz="0.02116183 0 0" rpy="1.57079632679 0 0"/ -->
         <origin xyz="0.04 0 0" rpy="0 0 0"/>

Commit message: Enable multiple cameras

File: mmuav_description/urdf/multirotor_base.urdf.xacro (robot description, xacro)
@@ -304,5 +304,5 @@
   @param *inertia Block argument defining camera inertia.
   -->
-  <xacro:macro name="cam" params="camera_link camera_mass parent *origin *inertia">
+  <xacro:macro name="cam" params="namespace camera_link camera_mass parent *origin *inertia">
     <!-- Camera link -->
     <link name="camera_box">
@@ -356,5 +356,5 @@
           <alwaysOn>true</alwaysOn>
           <updateRate>0.0</updateRate>
-          <cameraName>mmuav/camera1</cameraName>
+          <cameraName>${namespace}/camera1</cameraName>
           <imageTopicName>image_raw</imageTopicName>
           <cameraInfoTopicName>camera_info</cameraInfoTopicName>

Commit message: Add gimbal macro to base urdf

File: mmuav_description/urdf/multirotor_base.urdf.xacro (robot description, xacro)
@@ -599,3 +599,140 @@
     </gazebo>
   </xacro:macro>
+  <xacro:macro name="gimbal_macro" params="parent *origin">
+        <joint name="gimbal_position" type="fixed">
+            <xacro:insert_block name="origin"/>
+            <parent link="base_link"/>
+            <child link="gimbal_link_1"/>
+        </joint>
+        <gazebo reference="gimbal_position">
+            <preserveFixedJoint>true</preserveFixedJoint>
+        </gazebo>
+        <link name="gimbal_link_1">
+            <inertial>
+                <mass value="0.0001" />
+                <origin xyz="0 0 0" rpy="0 0 0" />
+                <inertia ixx="0.0001" ixy="0" ixz="0" iyy="0.0001" iyz="0" izz="0.0001" />
+            </inertial>
+<!--             <visual>
+                <geometry>
+                <box size="0.01 0.01 0.01" />
+                </geometry>
+            </visual> -->
+        </link>
+        <joint name="gimbal_roll_joint" type="continuous">
+            <parent link="gimbal_link_1" />
+            <child link="gimbal_link_2" />
+            <axis xyz="1 0 0" />
+            <dynamics damping="0.0" friction="0.0" />
+        </joint>
+        <link name="gimbal_link_2">
+            <inertial>
+                <mass value="0.0001" />
+                <origin xyz="0 0 0" rpy="0 0 0" />
+                <inertia ixx="0.0001" ixy="0" ixz="0" iyy="0.0001" iyz="0" izz="0.0001" />
+            </inertial>
+<!--             <visual>
+                <geometry>
+                <box size="0.01 0.01 0.01" />
+                </geometry>
+            </visual> -->
+        </link>
+        <joint name="gimbal_pitch_joint" type="continuous">
+            <parent link="gimbal_link_2" />
+            <child link="gimbal_link_3" />
+            <axis xyz="0 1 0" />
+            <dynamics damping="0.0" friction="0.0" />
+        </joint>
+        <link name="gimbal_link_3">
+            <inertial>
+                <mass value="0.0001" />
+                <origin xyz="0 0 0" rpy="0 0 0" />
+                <inertia ixx="0.0001" ixy="0" ixz="0" iyy="0.0001" iyz="0" izz="0.0001" />
+            </inertial>
+ <!--            <visual>
+                <geometry>
+                <box size="0.01 0.01 0.01" />
+                </geometry>
+            </visual> -->
+        </link>
+        <joint name="gimbal_yaw_joint" type="continuous">
+            <parent link="gimbal_link_3" />
+            <child link="gimbal_link_4" />
+            <axis xyz="0 0 1" />
+            <dynamics damping="0.0" friction="0.0" />
+        </joint>
+        <link name="gimbal_link_4">
+            <inertial>
+                <mass value="0.0001" />
+                <origin xyz="0 0 0" rpy="0 0 ${-PI}" />
+                <inertia ixx="0.0001" ixy="0" ixz="0" iyy="0.0001" iyz="0" izz="0.0001" />
+            </inertial>
+<!--             <visual>
+                <geometry>
+                <box size="0.01 0.01 0.01" />
+                </geometry>
+            </visual> -->
+        </link>
+        <joint name="camera_joint" type="continuous">
+            <parent link="gimbal_link_4" />
+            <child link="camera_link" />
+            <axis xyz="0 0 1" />
+            <dynamics damping="0.0" friction="0.0" />
+        </joint>
+        <link name="camera_link">
+        </link>
+        <joint name="camera_optical_joint" type="fixed">
+            <origin xyz="0 0 0" rpy="${-PI/2} 0.0 ${-PI/2}" />
+            <parent link="camera_link" />
+            <child link="camera_optical_frame"/>
+        </joint>
+        <gazebo reference="camera_optical_joint">
+            <preserveFixedJoint>true</preserveFixedJoint>
+        </gazebo>
+        <link name="camera_optical_frame">
+        </link>
+        <gazebo reference="gimbal_link_4">
+            <sensor type="camera" name="camera_camera_sensor">
+                <update_rate>30</update_rate>
+                <camera>
+                <!-- <pose>0.027 0 -0.027 0 1.57 0</pose> -->
+                <!-- <pose>0.027 0 -0.027 0 1.57 0</pose> -->
+                <pose>0.107 0 -0.127 0 0 0</pose>
+                <horizontal_fov>${94 * PI/180.0}</horizontal_fov>
+                <image>
+                    <format>R8G8B8</format>
+                    <width>640</width>
+                    <height>480</height>
+                </image>
+                <clip>
+                    <near>0.02</near>
+                    <far>300</far>
+                </clip>
+                </camera>
+                <plugin name="camera_controller" filename="libgazebo_ros_camera.so">
+                <cameraName>gimbal</cameraName>
+                <alwaysOn>true</alwaysOn>
+                <updateRate>10</updateRate>
+                <imageTopicName>image_raw</imageTopicName>
+                <cameraInfoTopicName>camera_info</cameraInfoTopicName>
+                <frameName>camera_optical_frame</frameName>
+                </plugin>
+            </sensor>
+        </gazebo>
+        <gazebo>
+          <plugin name="gimbal_controller" filename="libmmuav_gazebo_gimbal.so"/>
+        </gazebo>
+        <xacro:transmisija
+          trans_number="g1"
+          joint_name="gimbal_roll_joint">
+        </xacro:transmisija>
+        <xacro:transmisija
+          trans_number="g2"
+          joint_name="gimbal_pitch_joint">
+        </xacro:transmisija>
+        <xacro:transmisija
+          trans_number="g3"
+          joint_name="gimbal_yaw_joint">
+        </xacro:transmisija>
+    </xacro:macro>
 </robot>

Commit message: Add gimbal macro to urdf

File: mmuav_description/urdf/multirotor_base.urdf.xacro (robot description, xacro)
@@ -304,5 +304,5 @@
   @param *inertia Block argument defining camera inertia.
   -->
-  <xacro:macro name="cam" params="camera_link camera_mass parent *origin *inertia">
+  <xacro:macro name="cam" params="namespace camera_link camera_mass parent *origin *inertia">
     <!-- Camera link -->
     <link name="camera_box">
@@ -356,5 +356,5 @@
           <alwaysOn>true</alwaysOn>
           <updateRate>0.0</updateRate>
-          <cameraName>mmuav/camera1</cameraName>
+          <cameraName>${namespace}/camera1</cameraName>
           <imageTopicName>image_raw</imageTopicName>
           <cameraInfoTopicName>camera_info</cameraInfoTopicName>
@@ -599,3 +599,140 @@
     </gazebo>
   </xacro:macro>
+  <xacro:macro name="gimbal_macro" params="parent *origin">
+        <joint name="gimbal_position" type="fixed">
+            <xacro:insert_block name="origin"/>
+            <parent link="base_link"/>
+            <child link="gimbal_link_1"/>
+        </joint>
+        <gazebo reference="gimbal_position">
+            <preserveFixedJoint>true</preserveFixedJoint>
+        </gazebo>
+        <link name="gimbal_link_1">
+            <inertial>
+                <mass value="0.0001" />
+                <origin xyz="0 0 0" rpy="0 0 0" />
+                <inertia ixx="0.0001" ixy="0" ixz="0" iyy="0.0001" iyz="0" izz="0.0001" />
+            </inertial>
+<!--             <visual>
+                <geometry>
+                <box size="0.01 0.01 0.01" />
+                </geometry>
+            </visual> -->
+        </link>
+        <joint name="gimbal_roll_joint" type="continuous">
+            <parent link="gimbal_link_1" />
+            <child link="gimbal_link_2" />
+            <axis xyz="1 0 0" />
+            <dynamics damping="0.0" friction="0.0" />
+        </joint>
+        <link name="gimbal_link_2">
+            <inertial>
+                <mass value="0.0001" />
+                <origin xyz="0 0 0" rpy="0 0 0" />
+                <inertia ixx="0.0001" ixy="0" ixz="0" iyy="0.0001" iyz="0" izz="0.0001" />
+            </inertial>
+<!--             <visual>
+                <geometry>
+                <box size="0.01 0.01 0.01" />
+                </geometry>
+            </visual> -->
+        </link>
+        <joint name="gimbal_pitch_joint" type="continuous">
+            <parent link="gimbal_link_2" />
+            <child link="gimbal_link_3" />
+            <axis xyz="0 1 0" />
+            <dynamics damping="0.0" friction="0.0" />
+        </joint>
+        <link name="gimbal_link_3">
+            <inertial>
+                <mass value="0.0001" />
+                <origin xyz="0 0 0" rpy="0 0 0" />
+                <inertia ixx="0.0001" ixy="0" ixz="0" iyy="0.0001" iyz="0" izz="0.0001" />
+            </inertial>
+ <!--            <visual>
+                <geometry>
+                <box size="0.01 0.01 0.01" />
+                </geometry>
+            </visual> -->
+        </link>
+        <joint name="gimbal_yaw_joint" type="continuous">
+            <parent link="gimbal_link_3" />
+            <child link="gimbal_link_4" />
+            <axis xyz="0 0 1" />
+            <dynamics damping="0.0" friction="0.0" />
+        </joint>
+        <link name="gimbal_link_4">
+            <inertial>
+                <mass value="0.0001" />
+                <origin xyz="0 0 0" rpy="0 0 ${-PI}" />
+                <inertia ixx="0.0001" ixy="0" ixz="0" iyy="0.0001" iyz="0" izz="0.0001" />
+            </inertial>
+<!--             <visual>
+                <geometry>
+                <box size="0.01 0.01 0.01" />
+                </geometry>
+            </visual> -->
+        </link>
+        <joint name="camera_joint" type="continuous">
+            <parent link="gimbal_link_4" />
+            <child link="camera_link" />
+            <axis xyz="0 0 1" />
+            <dynamics damping="0.0" friction="0.0" />
+        </joint>
+        <link name="camera_link">
+        </link>
+        <joint name="camera_optical_joint" type="fixed">
+            <origin xyz="0 0 0" rpy="${-PI/2} 0.0 ${-PI/2}" />
+            <parent link="camera_link" />
+            <child link="camera_optical_frame"/>
+        </joint>
+        <gazebo reference="camera_optical_joint">
+            <preserveFixedJoint>true</preserveFixedJoint>
+        </gazebo>
+        <link name="camera_optical_frame">
+        </link>
+        <gazebo reference="gimbal_link_4">
+            <sensor type="camera" name="camera_camera_sensor">
+                <update_rate>30</update_rate>
+                <camera>
+                <!-- <pose>0.027 0 -0.027 0 1.57 0</pose> -->
+                <!-- <pose>0.027 0 -0.027 0 1.57 0</pose> -->
+                <pose>0.107 0 -0.127 0 0 0</pose>
+                <horizontal_fov>${94 * PI/180.0}</horizontal_fov>
+                <image>
+                    <format>R8G8B8</format>
+                    <width>640</width>
+                    <height>480</height>
+                </image>
+                <clip>
+                    <near>0.02</near>
+                    <far>300</far>
+                </clip>
+                </camera>
+                <plugin name="camera_controller" filename="libgazebo_ros_camera.so">
+                <cameraName>gimbal</cameraName>
+                <alwaysOn>true</alwaysOn>
+                <updateRate>10</updateRate>
+                <imageTopicName>image_raw</imageTopicName>
+                <cameraInfoTopicName>camera_info</cameraInfoTopicName>
+                <frameName>camera_optical_frame</frameName>
+                </plugin>
+            </sensor>
+        </gazebo>
+        <gazebo>
+          <plugin name="gimbal_controller" filename="libmmuav_gazebo_gimbal.so"/>
+        </gazebo>
+        <xacro:transmisija
+          trans_number="g1"
+          joint_name="gimbal_roll_joint">
+        </xacro:transmisija>
+        <xacro:transmisija
+          trans_number="g2"
+          joint_name="gimbal_pitch_joint">
+        </xacro:transmisija>
+        <xacro:transmisija
+          trans_number="g3"
+          joint_name="gimbal_yaw_joint">
+        </xacro:transmisija>
+    </xacro:macro>
 </robot>

Commit message: Revert cam macro changes

File: mmuav_description/urdf/multirotor_base.urdf.xacro (robot description, xacro)
@@ -304,5 +304,5 @@
   @param *inertia Block argument defining camera inertia.
   -->
-  <xacro:macro name="cam" params="namespace camera_link camera_mass parent *origin *inertia">
+  <xacro:macro name="cam" params="camera_link camera_mass parent *origin *inertia">
     <!-- Camera link -->
     <link name="camera_box">
@@ -356,5 +356,5 @@
           <alwaysOn>true</alwaysOn>
           <updateRate>0.0</updateRate>
-          <cameraName>${namespace}/camera1</cameraName>
+          <cameraName>mmuav/camera1</cameraName>
           <imageTopicName>image_raw</imageTopicName>
           <cameraInfoTopicName>camera_info</cameraInfoTopicName>

Commit message: Change order of rotations in the URDF

File: mmuav_description/urdf/multirotor_base.urdf.xacro (robot description, xacro)
@@ -620,8 +620,8 @@
             </visual> -->
         </link>
-        <joint name="gimbal_roll_joint" type="continuous">
+        <joint name="gimbal_yaw_joint" type="continuous">
             <parent link="gimbal_link_1" />
             <child link="gimbal_link_2" />
-            <axis xyz="1 0 0" />
+            <axis xyz="0 0 1" />
             <dynamics damping="0.0" friction="0.0" />
         </joint>
@@ -656,8 +656,8 @@
             </visual> -->
         </link>
-        <joint name="gimbal_yaw_joint" type="continuous">
+        <joint name="gimbal_roll_joint" type="continuous">
             <parent link="gimbal_link_3" />
             <child link="gimbal_link_4" />
-            <axis xyz="0 0 1" />
+            <axis xyz="1 0 0" />
             <dynamics damping="0.0" friction="0.0" />
         </joint>
