Commit message: Add stereo camera to UAV

File: mmuav_description/urdf/multirotor_base.urdf.xacro (robot description, xacro)
@@ -366,4 +366,89 @@
           <distortionT1>0.0</distortionT1>
           <distortionT2>0.0</distortionT2>
+        </plugin>
+      </sensor>
+    </gazebo>
+  </xacro:macro>
+  <!-- Stereo tCamera macro. Adds a box representing a camera below the UAV
+  @param camera_link Length of the camera box
+  @param camera_mass Mass of the camera
+  @param parent Parent link on which the camera will be fixed
+  @param *origin Block argument defining the origin of the camera with
+  reference to the parent link.
+  @param *inertia Block argument defining camera inertia.
+  -->
+  <xacro:macro name="stereo_cam" params="namespace camera_link camera_mass parent *origin *inertia">
+    <!-- Camera link -->
+    <link name="camera_box">
+      <!--collision>
+        <origin xyz="0 0 0" rpy="0 0 0"/>
+        <geometry>
+          <box size="${camera_link} ${camera_link} ${camera_link}"/>
+        </geometry>
+      </collision-->
+      <visual>
+        <origin xyz="0 0 0" rpy="0 1.57 0"/>
+        <geometry>
+          <!--box size="${camera_link} ${camera_link} ${camera_link}"/-->
+          <mesh filename="package://mmuav_description/meshes/asus_xtion_pro_camera.dae" scale="1 1 1" />
+        </geometry>
+      </visual>
+      <inertial>
+        <mass value="${camera_mass}" />
+        <xacro:insert_block name="inertia"/>
+      </inertial>
+    </link>
+    <!-- Camera joint with reference to the parent link -->
+    <joint name="camera_joint" type="fixed">
+      <xacro:insert_block name="origin"/>
+      <parent link="${parent}"/>
+      <child link="camera_box"/>
+    </joint>
+    <!-- camera -->
+    <gazebo reference="camera_box">
+      <sensor type="depth" name="camera">
+        <update_rate>30.0</update_rate>
+        <camera name="head">
+          <horizontal_fov>1.3962634</horizontal_fov>
+          <image>
+            <width>640</width>
+            <height>480</height>
+            <format>R8G8B8</format>
+          </image>
+          <clip>
+            <near>0.02</near>
+            <far>300</far>
+          </clip>
+          <noise>
+            <type>gaussian</type>
+            <mean>0.0</mean>
+            <stddev>0.007</stddev>
+          </noise>
+        </camera>
+        <plugin name="camera_plugin" filename="libgazebo_ros_openni_kinect.so">
+          <baseline>0.2</baseline>
+          <alwaysOn>true</alwaysOn>
+          <!-- Keep this zero, update_rate in the parent <sensor> tag
+            will control the frame rate. -->
+          <updateRate>0.0</updateRate>
+          <cameraName>${namespace}/camera_ir</cameraName>
+          <imageTopicName>/${namespace}/camera/color/image_raw</imageTopicName>
+          <cameraInfoTopicName>/${namespace}/camera/color/camera_info</cameraInfoTopicName>
+          <depthImageTopicName>/${namespace}/camera/depth/image_raw</depthImageTopicName>
+          <depthImageCameraInfoTopicName>/${namespace}/camera/depth/camera_info</depthImageCameraInfoTopicName>
+          <pointCloudTopicName>/${namespace}/camera/depth_registered/points</pointCloudTopicName>
+          <frameName>camera_box</frameName>
+          <pointCloudCutoff>0.3</pointCloudCutoff>
+          <pointCloudCutoffMax>10.0</pointCloudCutoffMax>
+          <distortionK1>0</distortionK1>
+          <distortionK2>0</distortionK2>
+          <distortionK3>0</distortionK3>
+          <distortionT1>0</distortionT1>
+          <distortionT2>0</distortionT2>
+          <CxPrime>0</CxPrime>
+          <Cx>0</Cx>
+          <Cy>0</Cy>
+          <focalLength>0</focalLength>
+          <hackBaseline>0</hackBaseline>
         </plugin>
       </sensor>

File: mmuav_description/urdf/uav.gazebo.xacro (robot description, xacro)
@@ -22,4 +22,21 @@
   <xacro:arg name="magnet_dipole_moment_z" default="970" />
   <xacro:property name="dp_z" value="$(arg magnet_dipole_moment_z)" />
+  <xacro:arg name="mount_stereo_cam" default="false" />
+  <xacro:property name="mount_stereo_cam" value="$(arg mount_stereo_cam)" />
+	<xacro:property name="front_facing_camera">
+		<origin xyz="0.025 0 0.1" rpy="0 0 0"/>
+	</xacro:property>
+	<xacro:property name="down_facing_camera">
+	  <origin xyz="0 0.2 -0.3" rpy="-1.570796 1.570796 0"/>
+	</xacro:property>
+  <xacro:property name="camera_mass" value="1e-5"/>
+	<xacro:property name="camera_size" value="0.05" />
+  <xacro:property name="camera_inertia">
+    <inertia
+    ixx="1e-12"
+    iyy="1e-12"
+    izz="1e-12"
+    ixy="0.0" ixz="0.0" iyz="0.0" />
+  </xacro:property>
   <!-- Instantiate mmuav "mechanics" -->
   <xacro:include filename="$(find mmuav_description)/urdf/uav.base.urdf.xacro" />
@@ -147,3 +164,13 @@
     <origin xyz="0.25 0 -0.05" rpy="0 0 0"/>
   </xacro:gimbal_macro> -->
+  <xacro:if value="${mount_stereo_cam}">
+    <xacro:stereo_cam
+      namespace="$(arg name)"
+      camera_link="${camera_size}"
+      camera_mass="${camera_mass}"
+      parent="base_link">
+      <xacro:insert_block name="front_facing_camera"/>
+      <xacro:insert_block name="camera_inertia"/>
+    </xacro:stereo_cam>
+  </xacro:if>
 </robot>

Commit message: Add rod with camera manipulator tool.

File: mmuav_description/urdf/multirotor_base.urdf.xacro (robot description, xacro)
@@ -304,5 +304,5 @@
   @param *inertia Block argument defining camera inertia.
   -->
-  <xacro:macro name="cam" params="namespace camera_link camera_mass parent *origin *inertia">
+  <xacro:macro name="cam" params="namespace camera_name camera_link camera_mass parent *origin *inertia">
     <!-- Camera link -->
     <link name="camera_box">
@@ -356,5 +356,5 @@
           <alwaysOn>true</alwaysOn>
           <updateRate>0.0</updateRate>
-          <cameraName>${namespace}/camera1</cameraName>
+          <cameraName>${namespace}/${camera_name}</cameraName>
           <imageTopicName>image_raw</imageTopicName>
           <cameraInfoTopicName>camera_info</cameraInfoTopicName>

File: mmuav_description/urdf/uav.base.urdf.xacro (robot description, xacro)
@@ -236,5 +236,5 @@
       </plugin>
     </gazebo>
-    <xacro:if value="${'rod' == manipulator_tool}">
+    <xacro:if value="${'rod' == manipulator_tool or 'rod_with_camera' == manipulator_tool}">
       <!-- Rod link -->
       <link name="rod">
@@ -273,4 +273,25 @@
         <child link="rod"/>
       </joint>
+      <!-- Add camera only if requested -->
+      <xacro:if value="${'rod_with_camera' == manipulator_tool}">
+        <xacro:property name="rod_camera_link" value="0.02" />
+        <xacro:property name="rod_camera_inertia">
+          <inertia
+          ixx="1e-8"
+          iyy="1e-8"
+          izz="1e-8"
+          ixy="0.0" ixz="0.0" iyz="0.0" />
+        </xacro:property>
+        <xacro:property name="rod_camera_mass" value="1e-5"/>
+        <xacro:cam
+          namespace="$(arg name)"
+          camera_name="rod_camera"
+          camera_link="${rod_camera_link}"
+          camera_mass="${rod_camera_mass}"
+          parent="rod">
+          <origin xyz="0.3 0 0" rpy="${PI} 0 0"/>
+          <xacro:insert_block name="rod_camera_inertia"/>
+        </xacro:cam>
+      </xacro:if>
     </xacro:if>
   </xacro:if>

Commit message: Add option to turn off all collision. Default is false.

File: mmuav_description/urdf/multirotor_base.urdf.xacro (robot description, xacro)
@@ -2,4 +2,6 @@
 <robot xmlns:xacro="http://ros.org/wiki/xacro">
   <!-- Main multirotor link -->
+  <xacro:arg name="turn_off_all_collisions" default="false" />
+  <xacro:property name="turn_off_all_collisions" value="$(arg turn_off_all_collisions)" />
   <xacro:macro name="multirotor_base_macro"
     params="robot_namespace mass body_width body_height mesh_file *origin *inertia">
@@ -24,12 +26,14 @@
         </geometry>
       </visual>
-      <collision>
-        <origin xyz="0 0 0" rpy="0 0 0" />
-        <geometry>
-          <mesh filename="package://mmuav_description/meshes/${mesh_file}"
-            scale="1 1 1" />
-          <!--box size="${body_width} ${body_width} ${body_height}" /-->
-        </geometry>
-      </collision>
+      <xacro:unless value="${turn_off_all_collisions}">
+        <collision>
+          <origin xyz="0 0 0" rpy="0 0 0" />
+          <geometry>
+            <mesh filename="package://mmuav_description/meshes/${mesh_file}"
+              scale="1 1 1" />
+            <!--box size="${body_width} ${body_width} ${body_height}" /-->
+          </geometry>
+        </collision>
+      </xacro:unless>
     </link>
     <!-- IMU -->
@@ -85,9 +89,11 @@
         </geometry>
       </visual>
-      <collision>
-        <geometry>
-          <cylinder length="0.005" radius="${radius_rotor}" /> <!-- [m] -->
-        </geometry>
-      </collision>
+      <xacro:unless value="${turn_off_all_collisions}">
+        <collision>
+          <geometry>
+            <cylinder length="0.005" radius="${radius_rotor}" /> <!-- [m] -->
+          </geometry>
+        </collision>
+      </xacro:unless>
     </link>
     <gazebo>
@@ -140,9 +146,11 @@
         </geometry>
       </visual>
-      <collision>
-        <geometry>
-          <cylinder length="0.005" radius="${radius_rotor}" /> <!-- [m] -->
-        </geometry>
-      </collision>
+      <xacro:unless value="${turn_off_all_collisions}">
+        <collision>
+          <geometry>
+            <cylinder length="0.005" radius="${radius_rotor}" /> <!-- [m] -->
+          </geometry>
+        </collision>
+      </xacro:unless>
     </link>
     <gazebo>
@@ -204,10 +212,12 @@
         </geometry>
       </visual>
-      <collision>
-        <origin rpy="0 0 0" xyz="0 0 ${length/2}"/>
-        <geometry>
-            <cylinder length="${length}" radius="${radius}" />
-        </geometry>
-      </collision>
+      <xacro:unless value="${turn_off_all_collisions}">
+        <collision>
+          <origin rpy="0 0 0" xyz="0 0 ${length/2}"/>
+          <geometry>
+              <cylinder length="${length}" radius="${radius}" />
+          </geometry>
+        </collision>
+      </xacro:unless>
       <inertial>
           <origin rpy="0 0 0" xyz="0 0 ${length/2}"/>
@@ -283,10 +293,12 @@
         </geometry>
       </visual>
-      <collision>
-        <origin rpy="0 0 0" xyz="0 0 0"/>
-        <geometry>
-          <box size="${dim_x} ${dim_y} ${dim_z}"/>
-        </geometry>
-      </collision>
+      <xacro:unless value="${turn_off_all_collisions}">
+        <collision>
+          <origin rpy="0 0 0" xyz="0 0 0"/>
+          <geometry>
+            <box size="${dim_x} ${dim_y} ${dim_z}"/>
+          </geometry>
+        </collision>
+      </xacro:unless>
       <inertial>
          <origin rpy="0 0 0" xyz="0 0 0"/>
@@ -668,10 +680,12 @@
         </geometry>
       </visual>
-      <collision>
-        <origin rpy="0 0 0" xyz="0 0 ${0*dimension/2}"/>
-        <geometry>
-          <box size="${1*dimension} ${1*dimension} ${1*dimension}"/>
-        </geometry>
-      </collision>
+      <xacro:unless value="${turn_off_all_collisions}">
+        <collision>
+          <origin rpy="0 0 0" xyz="0 0 ${0*dimension/2}"/>
+          <geometry>
+            <box size="${1*dimension} ${1*dimension} ${1*dimension}"/>
+          </geometry>
+        </collision>
+      </xacro:unless>
       <inertial>
         <origin rpy="0 0 0" xyz="0 0 ${0*dimension/2}"/>

File: mmuav_description/urdf/uav.base.urdf.xacro (robot description, xacro)
@@ -6,4 +6,6 @@
   <xacro:arg name="manipulator_tool" default="none" />
   <xacro:property name="manipulator_tool" value="$(arg manipulator_tool)" />
+  <xacro:arg name="turn_off_all_collisions" default="false" />
+  <xacro:property name="turn_off_all_collisions" value="$(arg turn_off_all_collisions)" />
   <!-- Properties -->
   <xacro:property name="rotor_velocity_slowdown_sim" value="15" />
@@ -252,10 +254,12 @@
           <material name="red"/>
         </visual>
-        <collision>
-          <origin xyz="0.15 0 0" rpy="0 0 0"/>
-          <geometry>
-              <box size="0.3 0.01 0.01"/>
-          </geometry>
-        </collision>
+        <xacro:unless value="${turn_off_all_collisions}">
+          <collision>
+            <origin xyz="0.15 0 0" rpy="0 0 0"/>
+            <geometry>
+                <box size="0.3 0.01 0.01"/>
+            </geometry>
+          </collision>
+        </xacro:unless>
         <inertial>
           <mass value="0.00001" />
@@ -372,10 +376,12 @@
           <material name="red"/>
         </visual>
-        <collision>
-          <origin xyz="0.15 0 0" rpy="0 0 0"/>
-          <geometry>
-              <box size="0.3 0.01 0.01"/>
-          </geometry>
-        </collision>
+        <xacro:unless value="${turn_off_all_collisions}">
+          <collision>
+            <origin xyz="0.15 0 0" rpy="0 0 0"/>
+            <geometry>
+                <box size="0.3 0.01 0.01"/>
+            </geometry>
+          </collision>
+        </xacro:unless>
         <inertial>
           <mass value="0.00001" />

File: mmuav_description/urdf/uav.gazebo.xacro (robot description, xacro)
@@ -24,4 +24,6 @@
   <xacro:arg name="mount_stereo_cam" default="false" />
   <xacro:property name="mount_stereo_cam" value="$(arg mount_stereo_cam)" />
+  <xacro:arg name="turn_off_all_collisions" default="false" />
+  <xacro:property name="turn_off_all_collisions" value="$(arg turn_off_all_collisions)" />
 	<xacro:property name="front_facing_camera">
 		<origin xyz="0.025 0 0.1" rpy="0 0 0"/>
