Commit message: Add collision bitmask to urdf and launch files.

File: mmuav_description/urdf/multirotor_base.urdf.xacro (robot description, xacro)
@@ -4,6 +4,17 @@
   <xacro:arg name="turn_off_all_collisions" default="false" />
   <xacro:property name="turn_off_all_collisions" value="$(arg turn_off_all_collisions)" />
+  <xacro:arg name="collision_bitmask" default="-1" />
+  <xacro:property name="collision_bitmask" value="$(arg collision_bitmask)" />
   <xacro:macro name="multirotor_base_macro"
     params="robot_namespace mass body_width body_height mesh_file *origin *inertia">
+    <gazebo reference="base_link">
+      <collision>
+        <surface>
+          <contact>
+            <collide_bitmask>${collision_bitmask}</collide_bitmask>
+          </contact>
+        </surface>
+      </collision>
+    </gazebo>
     <link name="base_link"></link>
     <joint name="base_joint" type="fixed">
@@ -12,4 +23,13 @@
       <child link="base_link_inertia" />
     </joint>
+    <gazebo reference="base_link_inertia">
+      <collision>
+        <surface>
+          <contact>
+            <collide_bitmask>${collision_bitmask}</collide_bitmask>
+          </contact>
+        </surface>
+      </collision>
+    </gazebo>
     <link name="base_link_inertia">
       <inertial>
@@ -38,4 +58,13 @@
     </link>
     <!-- IMU -->
+    <gazebo reference="imu_link">
+      <collision>
+        <surface>
+          <contact>
+            <collide_bitmask>${collision_bitmask}</collide_bitmask>
+          </contact>
+        </surface>
+      </collision>
+    </gazebo>
     <link name="imu_link">
       <inertial>
@@ -76,4 +105,13 @@
     <!-- <gazebo reference="rotor_${motor_number}_joint"> <axis> <xyz>0 0 1</xyz>
       <limit> <velocity> ${max_rot_velocity} </velocity> </limit> </axis> </gazebo> -->
+    <gazebo reference="rotor_${motor_number}">
+      <collision>
+        <surface>
+          <contact>
+            <collide_bitmask>${collision_bitmask}</collide_bitmask>
+          </contact>
+        </surface>
+      </collision>
+    </gazebo>
     <link name="rotor_${motor_number}">
       <inertial>
@@ -133,4 +171,13 @@
     <!-- <gazebo reference="rotor_${motor_number}_joint"> <axis> <xyz>0 0 1</xyz>
       <limit> <velocity> ${max_rot_velocity} </velocity> </limit> </axis> </gazebo> -->
+    <gazebo reference="rotor_${motor_number}">
+      <collision>
+        <surface>
+          <contact>
+            <collide_bitmask>${collision_bitmask}</collide_bitmask>
+          </contact>
+        </surface>
+      </collision>
+    </gazebo>
     <link name="rotor_${motor_number}">
       <inertial>
@@ -205,4 +252,13 @@
       <limit lower="-0.785398163" upper="0.785398163" effort="100000" velocity="3"/>
     </joint>
+    <gazebo reference="tilt_${motor_number}">
+      <collision>
+        <surface>
+          <contact>
+            <collide_bitmask>${collision_bitmask}</collide_bitmask>
+          </contact>
+        </surface>
+      </collision>
+    </gazebo>
     <link name="tilt_${motor_number}">
       <visual>
@@ -243,4 +299,13 @@
       <limit lower="-0.785398163" upper="0.785398163" effort="10000" velocity="10"/>
     </joint>
+    <gazebo reference="wing_${wing_number}">
+      <collision>
+        <surface>
+          <contact>
+            <collide_bitmask>${collision_bitmask}</collide_bitmask>
+          </contact>
+        </surface>
+      </collision>
+    </gazebo>
     <link name="wing_${wing_number}">
       <visual>
@@ -286,4 +351,13 @@
       <child link="land_gear_${gear_num}"/>
     </joint>
+    <gazebo reference="land_gear_${gear_num}">
+      <collision>
+        <surface>
+          <contact>
+            <collide_bitmask>${collision_bitmask}</collide_bitmask>
+          </contact>
+        </surface>
+      </collision>
+    </gazebo>
     <link name="land_gear_${gear_num}">
       <visual>
@@ -318,4 +392,13 @@
   <xacro:macro name="cam" params="namespace camera_name camera_link camera_mass parent *origin *inertia">
     <!-- Camera link -->
+    <gazebo reference="camera_box">
+      <collision>
+        <surface>
+          <contact>
+            <collide_bitmask>${collision_bitmask}</collide_bitmask>
+          </contact>
+        </surface>
+      </collision>
+    </gazebo>
     <link name="camera_box">
       <!--collision>
@@ -349,8 +432,8 @@
         <update_rate>30.0</update_rate>
         <camera name="head">
-          <horizontal_fov>1.3962634</horizontal_fov>
+          <horizontal_fov>1.0</horizontal_fov>
           <image>
-            <width>1920</width>
-            <height>1080</height>
+            <width>640</width>
+            <height>480</height>
             <format>R8G8B8</format>
           </image>
@@ -392,4 +475,13 @@
   <xacro:macro name="stereo_cam" params="namespace camera_link camera_mass parent *origin *inertia">
     <!-- Camera link -->
+    <gazebo reference="camera_box">
+      <collision>
+        <surface>
+          <contact>
+            <collide_bitmask>${collision_bitmask}</collide_bitmask>
+          </contact>
+        </surface>
+      </collision>
+    </gazebo>
     <link name="camera_box">
       <!--collision>
@@ -424,6 +516,6 @@
           <horizontal_fov>1.3962634</horizontal_fov>
           <image>
-            <width>640</width>
-            <height>480</height>
+            <width>1920</width>
+            <height>1080</height>
             <format>R8G8B8</format>
           </image>
@@ -472,4 +564,13 @@
     <!--LINK1 Dynamixel-->
     <!--_____________________________________________________________-->
+    <gazebo reference="dynamixel_1_${suffix}">
+      <collision>
+        <surface>
+          <contact>
+            <collide_bitmask>${collision_bitmask}</collide_bitmask>
+          </contact>
+        </surface>
+      </collision>
+    </gazebo>
     <link name='dynamixel_1_${suffix}'>
       <inertial>
@@ -500,4 +601,13 @@
     <!--LINK1 F3-->
     <!--_____________________________________________________________-->
+    <gazebo reference="link_F3_fixed_${suffix}">
+      <collision>
+        <surface>
+          <contact>
+            <collide_bitmask>${collision_bitmask}</collide_bitmask>
+          </contact>
+        </surface>
+      </collision>
+    </gazebo>
     <link name='link_F3_fixed_${suffix}'>
       <inertial>
@@ -520,4 +630,13 @@
     <!--LINK1 F4-->
     <!--_____________________________________________________________-->
+    <gazebo reference="link_F4_fixed_${suffix}">
+      <collision>
+        <surface>
+          <contact>
+            <collide_bitmask>${collision_bitmask}</collide_bitmask>
+          </contact>
+        </surface>
+      </collision>
+    </gazebo>
     <link name='link_F4_fixed_${suffix}'>
       <inertial>
@@ -540,4 +659,13 @@
     <!--LINK2 Dynamixel-->
     <!--_____________________________________________________________-->
+    <gazebo reference="dynamixel_2_${suffix}">
+      <collision>
+        <surface>
+          <contact>
+            <collide_bitmask>${collision_bitmask}</collide_bitmask>
+          </contact>
+        </surface>
+      </collision>
+    </gazebo>
     <link name='dynamixel_2_${suffix}'>
       <inertial>
@@ -568,4 +696,13 @@
     <!--GRIPPER PART1-->
     <!--_____________________________________________________________-->
+    <gazebo reference="link_gripper1_${suffix}">
+      <collision>
+        <surface>
+          <contact>
+            <collide_bitmask>${collision_bitmask}</collide_bitmask>
+          </contact>
+        </surface>
+      </collision>
+    </gazebo>
     <link name='link_gripper1_${suffix}'>
       <inertial>
@@ -588,4 +725,13 @@
     <!--GRIPPER PART2-->
     <!--_____________________________________________________________-->
+    <gazebo reference="link_gripper2_${suffix}">
+      <collision>
+        <surface>
+          <contact>
+            <collide_bitmask>${collision_bitmask}</collide_bitmask>
+          </contact>
+        </surface>
+      </collision>
+    </gazebo>
     <link name='link_gripper2_${suffix}'>
       <inertial>
@@ -673,4 +819,13 @@
       <dynamics damping="10" />
     </joint>
+    <gazebo reference="movable_mass_${mass_number}">
+      <collision>
+        <surface>
+          <contact>
+            <collide_bitmask>${collision_bitmask}</collide_bitmask>
+          </contact>
+        </surface>
+      </collision>
+    </gazebo>
     <link name="movable_mass_${mass_number}">
       <visual>
@@ -706,4 +861,13 @@
         <gazebo reference="gimbal_position">
             <preserveFixedJoint>true</preserveFixedJoint>
+        </gazebo>
+        <gazebo reference="gimbal_link_1">
+          <collision>
+            <surface>
+              <contact>
+                <collide_bitmask>${collision_bitmask}</collide_bitmask>
+              </contact>
+            </surface>
+          </collision>
         </gazebo>
         <link name="gimbal_link_1">
@@ -725,4 +889,13 @@
             <dynamics damping="0.0" friction="0.0" />
         </joint>
+        <gazebo reference="gimbal_link_2">
+          <collision>
+            <surface>
+              <contact>
+                <collide_bitmask>${collision_bitmask}</collide_bitmask>
+              </contact>
+            </surface>
+          </collision>
+        </gazebo>
         <link name="gimbal_link_2">
             <inertial>
@@ -743,4 +916,13 @@
             <dynamics damping="0.0" friction="0.0" />
         </joint>
+        <gazebo reference="gimbal_link_3">
+          <collision>
+            <surface>
+              <contact>
+                <collide_bitmask>${collision_bitmask}</collide_bitmask>
+              </contact>
+            </surface>
+          </collision>
+        </gazebo>
         <link name="gimbal_link_3">
             <inertial>
@@ -761,4 +943,13 @@
             <dynamics damping="0.0" friction="0.0" />
         </joint>
+        <gazebo reference="gimbal_link_4">
+          <collision>
+            <surface>
+              <contact>
+                <collide_bitmask>${collision_bitmask}</collide_bitmask>
+              </contact>
+            </surface>
+          </collision>
+        </gazebo>
         <link name="gimbal_link_4">
             <inertial>
@@ -779,4 +970,13 @@
             <dynamics damping="0.0" friction="0.0" />
         </joint>
+        <gazebo reference="camera_link">
+          <collision>
+            <surface>
+              <contact>
+                <collide_bitmask>${collision_bitmask}</collide_bitmask>
+              </contact>
+            </surface>
+          </collision>
+        </gazebo>
         <link name="camera_link">
         </link>
@@ -788,4 +988,13 @@
         <gazebo reference="camera_optical_joint">
             <preserveFixedJoint>true</preserveFixedJoint>
+        </gazebo>
+        <gazebo reference="camera_optical_frame">
+          <collision>
+            <surface>
+              <contact>
+                <collide_bitmask>${collision_bitmask}</collide_bitmask>
+              </contact>
+            </surface>
+          </collision>
         </gazebo>
         <link name="camera_optical_frame">

File: mmuav_description/urdf/uav.base.urdf.xacro (robot description, xacro)
@@ -8,4 +8,6 @@
   <xacro:arg name="turn_off_all_collisions" default="false" />
   <xacro:property name="turn_off_all_collisions" value="$(arg turn_off_all_collisions)" />
+  <xacro:arg name="collision_bitmask" default="-1" />
+  <xacro:property name="collision_bitmask" value="$(arg collision_bitmask)" />
   <!-- Properties -->
   <xacro:property name="rotor_velocity_slowdown_sim" value="15" />
@@ -240,4 +242,13 @@
     <xacro:if value="${'rod' == manipulator_tool or 'rod_with_camera' == manipulator_tool or 'rod_with_kinect' == manipulator_tool}">
       <!-- Rod link -->
+      <gazebo reference="rod">
+        <collision>
+          <surface>
+            <contact>
+              <collide_bitmask>${collision_bitmask}</collide_bitmask>
+            </contact>
+          </surface>
+        </collision>
+      </gazebo>
       <link name="rod">
         <!--collision>
@@ -273,4 +284,6 @@
       <gazebo reference="rod">
         <material>Gazebo/Red</material>
+        <mu1>10.8</mu1>
+        <mu2>10.8</mu2>
       </gazebo>
       <!-- Rod joint with reference to the parent link -->
@@ -385,4 +398,13 @@
     </gazebo>
     <xacro:if value="${'rod' == manipulator_tool}">
+      <gazebo reference="rod">
+        <collision>
+          <surface>
+            <contact>
+              <collide_bitmask>${collision_bitmask}</collide_bitmask>
+            </contact>
+          </surface>
+        </collision>
+      </gazebo>
       <!-- Rod link -->
       <link name="rod">

File: mmuav_description/urdf/uav.gazebo.xacro (robot description, xacro)
@@ -28,4 +28,6 @@
   <xacro:arg name="manipulator_tool" default="none" />
   <xacro:property name="manipulator_tool" value="$(arg manipulator_tool)" />
+  <xacro:arg name="collision_bitmask" default="-1" />
+  <xacro:property name="collision_bitmask" value="$(arg collision_bitmask)" />
 	<xacro:property name="front_facing_camera">
 		<origin xyz="0.025 0 0.1" rpy="0 0 0"/>
@@ -47,4 +49,13 @@
   <xacro:include filename="$(find rotors_description)/urdf/component_snippets.xacro" />
   <!-- Create link and joint for a sensor -->
+  <gazebo reference="pose_sensor1_link">
+    <collision>
+      <surface>
+        <contact>
+          <collide_bitmask>${collision_bitmask}</collide_bitmask>
+        </contact>
+      </surface>
+    </collision>
+  </gazebo>
   <link name="pose_sensor1_link">
     <inertial>
@@ -102,4 +113,13 @@
         <child link="electromagnet_actuator"/>
       </joint>
+      <gazebo reference="electromagnet_actuator">
+        <collision>
+          <surface>
+            <contact>
+              <collide_bitmask>${collision_bitmask}</collide_bitmask>
+            </contact>
+          </surface>
+        </collision>
+      </gazebo>
       <link name="electromagnet_actuator">
         <inertial>
@@ -211,3 +231,12 @@
     </xacro:stereo_cam>
   </xacro:if>
+  <!--gazebo reference="rod">
+    <collision>
+      <surface>
+        <contact>
+          <collide_bitmask>0x01</collide_bitmask>
+        </contact>
+      </surface>
+    </collision>
+  </gazebo-->
 </robot>

Commit message: Rotate kinect camera visual properly.

File: mmuav_description/urdf/multirotor_base.urdf.xacro (robot description, xacro)
@@ -492,5 +492,5 @@
       </collision-->
       <visual>
-        <origin xyz="0 0 0" rpy="0 1.57 0"/>
+        <origin xyz="0 0 0" rpy="0 0 0"/>
         <geometry>
           <!--box size="${camera_link} ${camera_link} ${camera_link}"/-->
