Commit message: Pruned everything uneccessary from models

File: mmuav_description/urdf/multirotor_base.urdf.xacro (robot description, xacro)
@@ -558,4 +558,12 @@
       </sensor>
     </gazebo>
+  </xacro:macro>
+  <xacro:macro name="gimbal" params="parent">
+  <!-- Camera joint with reference to the parent link -->
+    <joint name="gimbal_joint" type="fixed">
+      <origin xyz="0 0 0" rpy="0 0 0"/>
+      <parent link="${parent}"/>
+      <child link="gimbal_base_link"/>
+    </joint>
   </xacro:macro>
   <xacro:macro name="manipulator"

File: mmuav_description/urdf/uav.base.urdf.xacro (robot description, xacro)
@@ -1,9 +1,4 @@
 <?xml version="1.0"?>
 <robot name="uav" xmlns:xacro="http://ros.org/wiki/xacro">
-  <!-- Arguments -->
-  <xacro:arg name="manipulator_type" default="none" />
-  <xacro:property name="manipulator_type" value="$(arg manipulator_type)" />
-  <xacro:arg name="manipulator_tool" default="none" />
-  <xacro:property name="manipulator_tool" value="$(arg manipulator_tool)" />
   <xacro:arg name="turn_off_all_collisions" default="false" />
   <xacro:property name="turn_off_all_collisions" value="$(arg turn_off_all_collisions)" />
@@ -29,6 +24,4 @@
   <xacro:property name="rotor_drag_coefficient" value="8.06428e-05" />
   <xacro:property name="rolling_moment_coefficient" value="0.000001" />
-  <!-- aditional arm properties -->
-  <xacro:property name="arm_offset" value="0.1" /> <!-- [m] 0.0457-->
   <!-- Moving masses properties -->
   <xacro:property name="mm_mass" value="0.208" />
@@ -57,12 +50,4 @@
   <!-- Included URDF Files -->
   <xacro:include filename="$(find mmuav_description)/urdf/multirotor_base.urdf.xacro" />
-  <!-- Moving mass inertia block -->
-  <xacro:property name="movable_mass_inertia">
-     <inertia
-     ixx="${mm_mass * (mm_path_len/2 * mm_path_len/2)}"
-     iyy="${mm_mass * (mm_path_len/2 * mm_path_len/2)}"
-     izz="${mm_mass * (mm_path_len/2 * mm_path_len/2)}"
-     ixy="0.0" ixz="0.0"  iyz="0.0" /> <!-- [kg*m^2] [kg*m^2] [kg*m^2] [kg*m^2] [kg*m^2] [kg*m^2] -->
-  </xacro:property>
   <!-- IMU inertia (Pixhawk) -->
   <xacro:property name="imu_inertia">
@@ -164,304 +149,3 @@
     <xacro:insert_block name="rotor_inertia" />
   </xacro:vertical_rotor>
-<!--
-  <xacro:cam
-      namespace="$(arg name)"
-      parent="base_link"
-      camera_link="0.01"
-      camera_mass="0.01">
-      <origin xyz="0 0 -0.2" rpy="0 ${PI/2} ${-PI/4}"/>
-      <inertia ixx="0.001"  ixy="0.0"  ixz="0.0"
-               iyy="0.001"  iyz="0.0"  izz="0.001" />
-    </xacro:cam>
--->
-  <xacro:if value="${'wp_manipulator' == manipulator_type}">
-    <!-- Try to include manipulator -->
-    <xacro:include filename="$(find aerial_manipulators_description)/urdf/manipulator_base.urdf.xacro" />
-    <xacro:wp_manipulator parent="base_link">
-      <origin xyz="0 0 0.075" rpy="${pi/2} 0 ${pi}"/>
-    </xacro:wp_manipulator>
-    <xacro:transmisija
-      trans_number="1"
-      joint_name="joint1">
-    </xacro:transmisija>
-    <xacro:transmisija
-      trans_number="2"
-      joint_name="joint2">
-    </xacro:transmisija>
-    <xacro:transmisija
-      trans_number="3"
-      joint_name="joint3">
-    </xacro:transmisija>
-    <xacro:transmisija
-      trans_number="4"
-      joint_name="joint4">
-    </xacro:transmisija>
-    <xacro:transmisija
-      trans_number="5"
-      joint_name="joint5">
-    </xacro:transmisija>
-    <xacro:if value="${'camera' == manipulator_tool}">
-      <xacro:property name="camera_link" value="0.02" />
-      <xacro:property name="camera_inertia">
-        <inertia
-        ixx="1e-8"
-        iyy="1e-8"
-        izz="1e-8"
-        ixy="0.0" ixz="0.0" iyz="0.0" />
-      </xacro:property>
-      <xacro:property name="camera_mass" value="1e-5"/>
-      <xacro:cam
-        camera_link="${camera_link}"
-        camera_mass="${camera_mass}"
-        parent="end_effector_base">
-        <origin xyz="0 0 0" rpy="${PI} 0 0"/>
-        <xacro:insert_block name="camera_inertia"/>
-      </xacro:cam>
-    </xacro:if>
-    <!-- Enable the Joint Feedback -->
-    <gazebo reference="joint5">
-      <stopCfm>0.08</stopCfm>
-      <stopErp>0.2</stopErp>
-      <implicitSpringDamper>true</implicitSpringDamper>
-      <provideFeedback>true</provideFeedback>
-    </gazebo>
-    <!-- The ft_sensor plugin  -->
-    <gazebo>
-      <plugin name="ft_sensor" filename="libgazebo_ros_ft_sensor.so">
-        <updateRate>1000.0</updateRate>
-        <robotNamespace>$(arg name)/wp_manipulator</robotNamespace>
-        <topicName>force_sensor/ft_sensor</topicName>
-        <jointName>joint5</jointName>
-        <noise>
-          <type>gaussian</type>
-          <mean>0.0</mean>
-          <stddev>0.0001</stddev> <!-- change this to simulate noise -->
-        </noise>
-      </plugin>
-    </gazebo>
-    <xacro:if value="${'rod' == manipulator_tool or 'rod_with_camera' == manipulator_tool or 'rod_with_kinect' == manipulator_tool}">
-      <!-- Rod link -->
-      <gazebo reference="rod">
-        <collision>
-          <surface>
-            <contact>
-              <collide_bitmask>${collision_bitmask}</collide_bitmask>
-            </contact>
-          </surface>
-        </collision>
-      </gazebo>
-      <link name="rod">
-        <!--collision>
-          <origin xyz="0 0 0" rpy="0 0 0"/>
-          <geometry>
-            <box size="${camera_link} ${camera_link} ${camera_link}"/>
-          </geometry>
-        </collision-->
-        <visual>
-          <origin xyz="0.15 0 0" rpy="0 0 0"/>
-          <geometry>
-            <box size="0.3 0.01 0.01"/>
-          </geometry>
-          <material name="red"/>
-        </visual>
-        <xacro:unless value="${turn_off_all_collisions}">
-          <collision>
-            <origin xyz="0.15 0 0" rpy="0 0 0"/>
-            <geometry>
-                <box size="0.3 0.01 0.01"/>
-            </geometry>
-          </collision>
-        </xacro:unless>
-        <inertial>
-          <mass value="0.00001" />
-          <origin xyz="0.15 0 0" rpy="0 0 0"/>
-          <inertia
-            ixx="0" ixy="0" ixz="0"
-            iyx="0" iyy="0" iyz="0"
-            izx="0" izy="0" izz="0"/>
-        </inertial>
-      </link>
-      <gazebo reference="rod">
-        <material>Gazebo/Red</material>
-        <mu1>10.8</mu1>
-        <mu2>10.8</mu2>
-      </gazebo>
-      <!-- Rod joint with reference to the parent link -->
-      <joint name="rod_joint" type="fixed">
-        <origin xyz="0 0 0" rpy="0 0 0" />
-        <parent link="end_effector_base"/>
-        <child link="rod"/>
-      </joint>
-      <!-- Add camera only if requested -->
-      <xacro:if value="${'rod_with_camera' == manipulator_tool}">
-        <xacro:property name="rod_camera_link" value="0.02" />
-        <xacro:property name="rod_camera_inertia">
-          <inertia
-          ixx="1e-8"
-          iyy="1e-8"
-          izz="1e-8"
-          ixy="0.0" ixz="0.0" iyz="0.0" />
-        </xacro:property>
-        <xacro:property name="rod_camera_mass" value="1e-5"/>
-        <xacro:cam
-          namespace="$(arg name)"
-          camera_name="rod_camera"
-          camera_link="${rod_camera_link}"
-          camera_mass="${rod_camera_mass}"
-          parent="rod">
-          <origin xyz="0.3 0 0" rpy="${PI} 0 0"/>
-          <xacro:insert_block name="rod_camera_inertia"/>
-        </xacro:cam>
-      </xacro:if>
-      <!-- Add stereo camera only if requested -->
-      <xacro:if value="${'rod_with_kinect' == manipulator_tool}">
-        <xacro:property name="rod_camera_link" value="0.02" />
-        <xacro:property name="rod_camera_inertia">
-          <inertia
-          ixx="1e-8"
-          iyy="1e-8"
-          izz="1e-8"
-          ixy="0.0" ixz="0.0" iyz="0.0" />
-        </xacro:property>
-        <xacro:property name="rod_camera_mass" value="1e-5"/>
-        <xacro:property name="rod_kinect_transform">
-          <origin xyz="0.3 0 0.0" rpy="${PI} 0 0"/>
-        </xacro:property>
-        <xacro:stereo_cam
-          namespace="$(arg name)"
-          camera_link="${rod_camera_link}"
-          camera_mass="${rod_camera_mass}"
-          parent="rod">
-          <xacro:insert_block name="rod_kinect_transform"/>
-          <xacro:insert_block name="rod_camera_inertia"/>
-        </xacro:stereo_cam>
-      </xacro:if>
-    </xacro:if>
-  </xacro:if>
-  <xacro:if value="${'wp_manipulator_3rx' == manipulator_type}">
-    <!-- Try to include manipulator -->
-    <xacro:include filename="$(find aerial_manipulators_description)/urdf/manipulator_base.urdf.xacro" />
-    <xacro:wp_manipulator_3rx parent="base_link">
-      <!--origin xyz="0 0 0.2" rpy="${pi/2} 0 0"/-->
-      <origin xyz="0 0 0.2" rpy="0 0 0"/>
-    </xacro:wp_manipulator_3rx>
-    <xacro:transmisija
-      trans_number="1"
-      joint_name="joint1">
-    </xacro:transmisija>
-    <xacro:transmisija
-      trans_number="2"
-      joint_name="joint2">
-    </xacro:transmisija>
-    <xacro:transmisija
-      trans_number="3"
-      joint_name="joint3">
-    </xacro:transmisija>
-    <xacro:if value="${'camera' == manipulator_tool}">
-      <xacro:property name="camera_link" value="0.02" />
-      <xacro:property name="camera_inertia">
-        <inertia
-        ixx="1e-8"
-        iyy="1e-8"
-        izz="1e-8"
-        ixy="0.0" ixz="0.0" iyz="0.0" />
-      </xacro:property>
-      <xacro:property name="camera_mass" value="1e-5"/>
-      <xacro:cam
-        camera_link="${camera_link}"
-        camera_mass="${camera_mass}"
-        parent="end_effector_base">
-        <origin xyz="0 0 0" rpy="${PI} 0 0"/>
-        <xacro:insert_block name="camera_inertia"/>
-      </xacro:cam>
-    </xacro:if>
-    <!-- Enable the Joint Feedback -->
-    <gazebo reference="joint3">
-      <stopCfm>0.08</stopCfm>
-      <stopErp>0.2</stopErp>
-      <implicitSpringDamper>true</implicitSpringDamper>
-      <provideFeedback>true</provideFeedback>
-    </gazebo>
-    <!-- The ft_sensor plugin  -->
-    <gazebo>
-      <plugin name="ft_sensor" filename="libgazebo_ros_ft_sensor.so">
-        <updateRate>1000.0</updateRate>
-        <robotNamespace>$(arg name)/wp_manipulator</robotNamespace>
-        <topicName>force_sensor/ft_sensor</topicName>
-        <jointName>joint3</jointName>
-        <noise>
-          <type>gaussian</type>
-          <mean>0.0</mean>
-          <stddev>0.0001</stddev> <!-- change this to simulate noise -->
-        </noise>
-      </plugin>
-    </gazebo>
-    <xacro:if value="${'rod' == manipulator_tool}">
-      <gazebo reference="rod">
-        <collision>
-          <surface>
-            <contact>
-              <collide_bitmask>${collision_bitmask}</collide_bitmask>
-            </contact>
-          </surface>
-        </collision>
-      </gazebo>
-      <!-- Rod link -->
-      <link name="rod">
-        <!--collision>
-          <origin xyz="0 0 0" rpy="0 0 0"/>
-          <geometry>
-            <box size="${camera_link} ${camera_link} ${camera_link}"/>
-          </geometry>
-        </collision-->
-        <visual>
-          <origin xyz="0.15 0 0" rpy="0 0 0"/>
-          <geometry>
-            <box size="0.3 0.01 0.01"/>
-          </geometry>
-          <material name="red"/>
-        </visual>
-        <xacro:unless value="${turn_off_all_collisions}">
-          <collision>
-            <origin xyz="0.15 0 0" rpy="0 0 0"/>
-            <geometry>
-                <box size="0.3 0.01 0.01"/>
-            </geometry>
-          </collision>
-        </xacro:unless>
-        <inertial>
-          <mass value="0.00001" />
-          <origin xyz="0.15 0 0" rpy="0 0 0"/>
-          <inertia
-            ixx="0" ixy="0" ixz="0"
-            iyx="0" iyy="0" iyz="0"
-            izx="0" izy="0" izz="0"/>
-        </inertial>
-      </link>
-      <!-- Rod joint with reference to the parent link -->
-      <joint name="rod_joint" type="fixed">
-        <origin xyz="0 0 0" rpy="0 0 0" />
-        <parent link="end_effector_base"/>
-        <child link="rod"/>
-      </joint>
-    </xacro:if>
-  </xacro:if>
-  <!-- <xacro:camera_macro robot_namespace="${namespace}">
-  </xacro:camera_macro> -->
-  <!--xacro:transmisija
-    trans_number="0"
-    joint_name="stick_to_movable_mass_0">
-  </xacro:transmisija>
-  <xacro:transmisija
-    trans_number="1"
-    joint_name="stick_to_movable_mass_1">
-  </xacro:transmisija>
-  <xacro:transmisija
-    trans_number="2"
-    joint_name="stick_to_movable_mass_2">
-  </xacro:transmisija>
-  <xacro:transmisija
-    trans_number="3"
-    joint_name="stick_to_movable_mass_3">
-  </xacro:transmisija-->
 </robot>

File: mmuav_description/urdf/uav.gazebo.xacro (robot description, xacro)
@@ -12,22 +12,18 @@
     </plugin>
   </gazebo>
+  <!-- Add UAV base and component snippets -->
+  <xacro:include filename="$(find mmuav_description)/urdf/uav.base.urdf.xacro" />
+  <xacro:include filename="$(find rotors_description)/urdf/component_snippets.xacro" />
   <xacro:property name="enable_bag_plugin" value="false" />
   <xacro:property name="bag_file" value="uav.bag" />
   <xacro:arg name="mount_velodyne" default="false" />
   <xacro:property name="mount_velodyne" value="$(arg mount_velodyne)" />
-  <xacro:arg name="mount_magnet" default="false" />
-  <xacro:property name="mount_magnet" value="$(arg mount_magnet)" />
-  <xacro:arg name="mount_magnet_with_disk" default="false" />
-  <xacro:property name="mount_magnet_with_disk" value="$(arg mount_magnet_with_disk)" />
-  <xacro:arg name="magnet_dipole_moment_z" default="970" />
-  <xacro:property name="dp_z" value="$(arg magnet_dipole_moment_z)" />
   <xacro:arg name="mount_stereo_cam" default="false" />
   <xacro:property name="mount_stereo_cam" value="$(arg mount_stereo_cam)" />
   <xacro:arg name="turn_off_all_collisions" default="false" />
   <xacro:property name="turn_off_all_collisions" value="$(arg turn_off_all_collisions)" />
-  <xacro:arg name="manipulator_tool" default="none" />
-  <xacro:property name="manipulator_tool" value="$(arg manipulator_tool)" />
   <xacro:arg name="collision_bitmask" default="-1" />
   <xacro:property name="collision_bitmask" value="$(arg collision_bitmask)" />
+  <!-- Cam properties -->
 	<xacro:property name="front_facing_camera">
 		<origin xyz="0.025 0 0.1" rpy="0 0 0"/>
@@ -45,30 +41,4 @@
     ixy="0.0" ixz="0.0" iyz="0.0" />
   </xacro:property>
-  <!-- Instantiate mmuav "mechanics" -->
-  <xacro:include filename="$(find mmuav_description)/urdf/uav.base.urdf.xacro" />
-  <xacro:include filename="$(find rotors_description)/urdf/component_snippets.xacro" />
-  <!-- Create link and joint for a sensor -->
-  <gazebo reference="pose_sensor1_link">
-    <collision>
-      <surface>
-        <contact>
-          <collide_bitmask>${collision_bitmask}</collide_bitmask>
-        </contact>
-      </surface>
-    </collision>
-  </gazebo>
-  <link name="pose_sensor1_link">
-    <inertial>
-      <inertia ixx="0.00001" ixy="0.0" ixz="0.0" iyy="0.00001" iyz="0.0"
-        izz="0.00001" />
-      <mass value="0.01" />
-    </inertial>
-  </link>
-  <joint name="pose_sensor1_joint" type="revolute">
-    <parent link="base_link" />
-    <origin xyz="0 0 0" rpy="0 0 0" />
-    <child link="pose_sensor1_link" />
-    <limit upper="0" lower="0" effort="0" velocity="0" />
-  </joint>
   <xacro:property name="horizontal_velodyne_origin">
     <origin xyz="0 0 -0.025" rpy="3.141592653589793 0.1323284641020683 0." />
@@ -105,52 +75,4 @@
     </VU-8>
   </xacro:if>
-  <xacro:if value="${mount_magnet}">
-    <xacro:if value="${mount_magnet_with_disk}">
-      <joint name="electromagnet_joint" type="fixed">
-        <axis xyz="0 1 0" />
-        <origin xyz="0.0 0.0 -0.15" rpy="0 0 0"/>
-        <parent link="base_link"/>
-        <child link="electromagnet_actuator"/>
-      </joint>
-      <gazebo reference="electromagnet_actuator">
-        <collision>
-          <surface>
-            <contact>
-              <collide_bitmask>${collision_bitmask}</collide_bitmask>
-            </contact>
-          </surface>
-        </collision>
-      </gazebo>
-      <link name="electromagnet_actuator">
-        <inertial>
-        <origin xyz="0 0 0" rpy="0 0 0" />
-        <mass value="0.025"/>
-        <inertia ixx="0.0001" ixy="0" ixz="0" iyy ="0.0001" iyz = "0" izz = "0.0001" />
-        </inertial>
-        <collision name="collision">
-        <geometry>
-          <cylinder radius="0.08" length="0.035"/>
-        </geometry>
-        </collision>
-        <visual>
-        <geometry>
-          <cylinder radius="0.08" length="0.035"/>
-        </geometry>
-        </visual>
-      </link>
-    </xacro:if>
-    <gazebo>
-      <plugin name="dipole_magnet" filename="libstorm_gazebo_dipole_magnet.so">
-        <robotNamespace>$(arg name)</robotNamespace>
-        <bodyName>base_link</bodyName>
-        <dipole_moment>0 0 ${dp_z}</dipole_moment>
-        <!-- Set to false if not using ROS -->
-        <shouldPublish>true</shouldPublish>
-        <topicNs>magnet</topicNs>
-        <updateRate>100</updateRate>
-        <gain>1.0</gain>
-      </plugin>
-    </gazebo>
-  </xacro:if>
   <!-- Mount first generic pose sensor-->
   <xacro:odometry_plugin_macro
@@ -184,6 +106,5 @@
     <origin xyz="0.0 0.0 0" rpy="0.0 0.0 0.0" />
   </xacro:odometry_plugin_macro>
-  <xacro:if value="${'rod_with_camera' == manipulator_tool}">
-    <xacro:odometry_plugin_macro
+  <xacro:odometry_plugin_macro
     namespace="$(arg name)"
     odometry_sensor_suffix="2"
@@ -214,11 +135,8 @@
     <inertia ixx="1e-6" ixy="0.0" ixz="0.0" iyy="1e-6" iyz="0.0" izz="1e-6" /> <!-- [kg m^2] [kg m^2] [kg m^2] [kg m^2] [kg m^2] [kg m^2] -->
     <!-- This rotation is correction for blender. -->
+    <!-- Find out why this correction exists-->
     <origin xyz="0.0 0.0 0" rpy="1.57 0.0 -1.57" />
   </xacro:odometry_plugin_macro>
   </xacro:if>
-  <!-- mount gimbal -->
-  <!--<xacro:gimbal_macro parent="base_link">
-    <origin xyz="0.25 0 -0.05" rpy="0 0 0"/>
-  </xacro:gimbal_macro> -->
   <xacro:if value="${mount_stereo_cam}">
     <xacro:stereo_cam
@@ -231,12 +149,3 @@
     </xacro:stereo_cam>
   </xacro:if>
-  <!--gazebo reference="rod">
-    <collision>
-      <surface>
-        <contact>
-          <collide_bitmask>0x01</collide_bitmask>
-        </contact>
-      </surface>
-    </collision>
-  </gazebo-->
 </robot>
