Commit message: Removed 100% uneccessary files, added init wp_manipulator

File: mmuav_description/urdf/multirotor_base.urdf.xacro (robot description, xacro)
@@ -1051,4 +1051,4 @@
           joint_name="gimbal_yaw_joint">
         </xacro:transmisija>
-    </xacro:macro>
+  </xacro:macro>
 </robot>

File: mmuav_description/urdf/uav.base.urdf.xacro (robot description, xacro)
@@ -1,4 +1,4 @@
-<?xml version="1.0"?>
-<robot name="uav" xmlns:xacro="http://ros.org/wiki/xacro">
+<?xml version='1.0' encoding='utf-8'?>
+<robot name="uav_base" xmlns:xacro="http://ros.org/wiki/xacro">
   <xacro:arg name="turn_off_all_collisions" default="false" />
   <xacro:property name="turn_off_all_collisions" value="$(arg turn_off_all_collisions)" />

File: mmuav_description/urdf/uav.gazebo.xacro (robot description, xacro)
@@ -1,118 +1,116 @@
-<?xml version="1.0"?>
+<?xml version='1.0' encoding='utf-8'?>
 <robot name="uav" xmlns:xacro="http://ros.org/wiki/xacro">
-  <!--
-  It seems that the xacro:property does not allow to use substitution args. Therefore, instead xacro parameter ${namespace}, subsitution argument is used $(arg name). This is
-  <xacro:property name="namespace" value="$(arg name)" />
-  -->
-  <gazebo>
-    <plugin name="gazebo_ros_control" filename="libgazebo_ros_control.so">
-      <robotNamespace>/$(arg name)</robotNamespace>
-      <robotParam>/$(arg name)/robot_description </robotParam>
-      <robotSimType>gazebo_ros_control/DefaultRobotHWSim</robotSimType>
-    </plugin>
-  </gazebo>
-  <!-- Add UAV base and component snippets -->
-  <xacro:include filename="$(find mmuav_description)/urdf/uav.base.urdf.xacro" />
-  <xacro:include filename="$(find rotors_description)/urdf/component_snippets.xacro" />
-  <xacro:property name="enable_bag_plugin" value="false" />
-  <xacro:property name="bag_file" value="uav.bag" />
-  <xacro:arg name="mount_velodyne" default="false" />
-  <xacro:property name="mount_velodyne" value="$(arg mount_velodyne)" />
-  <xacro:arg name="mount_stereo_cam" default="false" />
-  <xacro:property name="mount_stereo_cam" value="$(arg mount_stereo_cam)" />
-  <xacro:arg name="turn_off_all_collisions" default="false" />
-  <xacro:property name="turn_off_all_collisions" value="$(arg turn_off_all_collisions)" />
-  <xacro:arg name="collision_bitmask" default="-1" />
-  <xacro:property name="collision_bitmask" value="$(arg collision_bitmask)" />
-  <!-- Cam properties -->
-	<xacro:property name="front_facing_camera">
-		<origin xyz="0.025 0 0.1" rpy="0 0 0"/>
-	</xacro:property>
-	<xacro:property name="down_facing_camera">
-	  <origin xyz="0 0.2 -0.3" rpy="-1.570796 1.570796 0"/>
-	</xacro:property>
-  <xacro:property name="camera_mass" value="1e-5"/>
-	<xacro:property name="camera_size" value="0.05" />
-  <xacro:property name="camera_inertia">
-    <inertia
-    ixx="1e-12"
-    iyy="1e-12"
-    izz="1e-12"
-    ixy="0.0" ixz="0.0" iyz="0.0" />
-  </xacro:property>
-  <xacro:property name="horizontal_velodyne_origin">
-    <origin xyz="0 0 -0.025" rpy="3.141592653589793 0.1323284641020683 0." />
-  </xacro:property>
-  <!-- Mount an IMU -->
-  <gazebo>
-    <!-- IMU -->
-    <plugin filename="libhector_gazebo_ros_imu.so" name="imu_ros">
-      <!-- parameters according to http://wiki.ros.org/hector_gazebo_plugins#GazeboRosImu -->
-      <!-- robotNamespace>${namespace}</robotNamespace -->
-      <robotNamespace>$(arg name)</robotNamespace>
-      <bodyName>imu_link</bodyName> <!-- (string, required): name of the body which holds the IMU sensor -->
-      <topicName>imu</topicName> <!-- (string): name of the sensor output topic and prefix of service names (defaults to imu) -->
-      <accelOffset>0.0 0.0 0.0</accelOffset> <!-- (Vector3): constant acceleration offset -->
-      <accelDrift>0.0 0.0 0.0</accelDrift> <!-- (Vector3): standard deviation of the acceleration drift error -->
-      <accelDriftFrequency>0.0 0.0 0.0</accelDriftFrequency> <!-- (Vector3): mean frequency of the acceleration drift staviti na nulu-->
-      <accelGaussianNoise>0.001 0.001 0.001</accelGaussianNoise> <!-- (Vector3): standard deviation of the additive Gaussian acceleration noise -->
-      <rateOffset>0.0 0.0 0.0</rateOffset> <!-- (Vector3): constant rate offset -->
-      <rateDrift>0.0 0.0 0.0</rateDrift> <!-- (Vector3): standard deviation of the rate drift error -->
-      <rateDriftFrequency>0.0 0.0 0.0</rateDriftFrequency> <!-- (Vector3): mean frequency of the rate drift  staviti na nulu-->
-      <rateGaussianNoise>0.0001 0.0001 0.0001</rateGaussianNoise> <!-- (Vector3): standard deviation of the additive Gaussian rate noise -->
-      <headingOffset>0.0</headingOffset> <!-- (double): constant heading offset -->
-      <headingDrift>0.0</headingDrift> <!-- (double): standard deviation of the heading drift error -->
-      <headingDriftFrequency>0.0</headingDriftFrequency> <!-- (double): mean frequency of the heading drift  staviti na nulu-->
-      <headingGaussianNoise>0.0</headingGaussianNoise> <!-- (double): standard deviation of the heading additive Gaussian noise -->
-      <rpyOffsets>0.0 0.0 0.0</rpyOffsets> <!-- (Vector3): if non-zero, used to calculate accelOffset and headingOffset so that resulting roll, pitch and yaw errors correspond to this values when the platform is leveled (for compatibility with gazebo_plugins) -->
-    </plugin>
-  </gazebo>
-  <xacro:if value="${mount_velodyne}">
-    <xacro:include filename="$(find velodyne_description)/urdf/VU-8.urdf.xacro"/>
-    <VU-8 parent="base_link" name="velodyne" topic="$(arg name)/velodyne_points" hz="10" samples="440" gpu="false"
-            min_range="1" lasers="16">
-        <xacro:insert_block name="horizontal_velodyne_origin"/>
-    </VU-8>
-  </xacro:if>
-  <!-- Mount first generic pose sensor-->
-  <xacro:odometry_plugin_macro
-    namespace="$(arg name)"
-    odometry_sensor_suffix="1"
-    child_frame_id="base"
-    parent_link="base_link"
-    pose_topic="pose"
-    velocity_relative_topic="velocity_relative"
-    pose_with_covariance_topic="pose_with_covariance"
-    position_topic="position"
-    transform_topic="transform"
-    odometry_topic="odometry"
-    parent_frame_id="world"
-    mass_odometry_sensor="0.01"
-    measurement_divisor="5"
-    measurement_delay="0"
-    unknown_delay="0.0"
-    noise_normal_position="0.0 0.0 0.0"
-    noise_normal_quaternion="0.0 0.0 0.0"
-    noise_normal_linear_velocity="0.0 0.0 0.0"
-    noise_normal_angular_velocity="0.0 0.0 0.0"
-    noise_uniform_position="0.0 0.0 0.0"
-    noise_uniform_quaternion="0.0 0.0 0.0"
-    noise_uniform_linear_velocity="0.0 0.0 0.0"
-    noise_uniform_angular_velocity="0.0 0.0 0.0"
-    enable_odometry_map="false"
-    odometry_map=""
-    image_scale="">
-    <inertia ixx="0.00001" ixy="0.0" ixz="0.0" iyy="0.00001" iyz="0.0" izz="0.00001" /> <!-- [kg m^2] [kg m^2] [kg m^2] [kg m^2] [kg m^2] [kg m^2] -->
-    <origin xyz="0.0 0.0 0" rpy="0.0 0.0 0.0" />
-  </xacro:odometry_plugin_macro>
-  <xacro:if value="${mount_stereo_cam}">
-    <xacro:stereo_cam
+  <!--xacro:macro name="uav"-->
+    <!-- TODO: Fix uav:xacro -->
+    <!-- Add UAV base and component snippets -->
+    <xacro:include filename="$(find mmuav_description)/urdf/uav.base.urdf.xacro" />
+    <xacro:include filename="$(find rotors_description)/urdf/component_snippets.xacro" />
+    <xacro:arg name="mount_velodyne" default="false" />
+    <xacro:property name="mount_velodyne" value="$(arg mount_velodyne)" />
+    <xacro:arg name="mount_stereo_cam" default="false" />
+    <xacro:property name="mount_stereo_cam" value="$(arg mount_stereo_cam)" />
+    <xacro:arg name="turn_off_all_collisions" default="false" />
+    <xacro:property name="turn_off_all_collisions" value="$(arg turn_off_all_collisions)" />
+    <xacro:arg name="collision_bitmask" default="-1" />
+    <xacro:property name="collision_bitmask" value="$(arg collision_bitmask)" />
+    <!-- Cam properties -->
+    <xacro:property name="front_facing_camera">
+      <origin xyz="0.025 0 0.1" rpy="0 0 0"/>
+    </xacro:property>
+    <xacro:property name="down_facing_camera">
+      <origin xyz="0 0.2 -0.3" rpy="-1.570796 1.570796 0"/>
+    </xacro:property>
+    <xacro:property name="camera_mass" value="1e-5"/>
+    <xacro:property name="camera_size" value="0.05" />
+    <xacro:property name="camera_inertia">
+      <inertia
+      ixx="1e-12"
+      iyy="1e-12"
+      izz="1e-12"
+      ixy="0.0" ixz="0.0" iyz="0.0" />
+    </xacro:property>
+    <xacro:property name="horizontal_velodyne_origin">
+      <origin xyz="0 0 -0.025" rpy="3.141592653589793 0.1323284641020683 0." />
+    </xacro:property>
+    <!-- Mount first generic pose sensor-->
+    <xacro:odometry_plugin_macro
       namespace="$(arg name)"
-      camera_link="${camera_size}"
-      camera_mass="${camera_mass}"
-      parent="base_link">
-      <xacro:insert_block name="front_facing_camera"/>
-      <xacro:insert_block name="camera_inertia"/>
-    </xacro:stereo_cam>
-  </xacro:if>
+      odometry_sensor_suffix="1"
+      child_frame_id="base"
+      parent_link="base_link"
+      pose_topic="pose"
+      velocity_relative_topic="velocity_relative"
+      pose_with_covariance_topic="pose_with_covariance"
+      position_topic="position"
+      transform_topic="transform"
+      odometry_topic="odometry"
+      parent_frame_id="world"
+      mass_odometry_sensor="0.01"
+      measurement_divisor="5"
+      measurement_delay="0"
+      unknown_delay="0.0"
+      noise_normal_position="0.0 0.0 0.0"
+      noise_normal_quaternion="0.0 0.0 0.0"
+      noise_normal_linear_velocity="0.0 0.0 0.0"
+      noise_normal_angular_velocity="0.0 0.0 0.0"
+      noise_uniform_position="0.0 0.0 0.0"
+      noise_uniform_quaternion="0.0 0.0 0.0"
+      noise_uniform_linear_velocity="0.0 0.0 0.0"
+      noise_uniform_angular_velocity="0.0 0.0 0.0"
+      enable_odometry_map="false"
+      odometry_map=""
+      image_scale="">
+      <inertia ixx="0.00001" ixy="0.0" ixz="0.0" iyy="0.00001" iyz="0.0" izz="0.00001" /> <!-- [kg m^2] [kg m^2] [kg m^2] [kg m^2] [kg m^2] [kg m^2] -->
+      <origin xyz="0.0 0.0 0" rpy="0.0 0.0 0.0" />
+    </xacro:odometry_plugin_macro>
+    <!-- Mount stereo cam -->
+    <xacro:if value="${mount_stereo_cam}">
+      <xacro:stereo_cam
+        namespace="$(arg name)"
+        camera_link="${camera_size}"
+        camera_mass="${camera_mass}"
+        parent="base_link">
+        <xacro:insert_block name="front_facing_camera"/>
+        <xacro:insert_block name="camera_inertia"/>
+      </xacro:stereo_cam>
+    </xacro:if>
+    <xacro:if value="${mount_velodyne}">
+      <xacro:include filename="$(find velodyne_description)/urdf/VU-8.urdf.xacro"/>
+      <VU-8 parent="base_link" name="velodyne" topic="$(arg name)/velodyne_points" hz="10" samples="440" gpu="false"
+              min_range="1" lasers="16">
+          <xacro:insert_block name="horizontal_velodyne_origin"/>
+      </VU-8>
+    </xacro:if>
+    <gazebo>
+      <plugin name="gazebo_ros_control" filename="libgazebo_ros_control.so">
+        <robotNamespace>/$(arg name)</robotNamespace>
+        <robotParam>/$(arg name)/robot_description </robotParam>
+        <robotSimType>gazebo_ros_control/DefaultRobotHWSim</robotSimType>
+      </plugin>
+    </gazebo>
+    <!-- Mount an IMU -->
+    <gazebo>
+      <!-- IMU -->
+      <plugin filename="libhector_gazebo_ros_imu.so" name="imu_ros">
+        <!-- parameters according to http://wiki.ros.org/hector_gazebo_plugins#GazeboRosImu -->
+        <!-- robotNamespace>${namespace}</robotNamespace -->
+        <robotNamespace>$(arg name)</robotNamespace>
+        <bodyName>imu_link</bodyName> <!-- (string, required): name of the body which holds the IMU sensor -->
+        <topicName>imu</topicName> <!-- (string): name of the sensor output topic and prefix of service names (defaults to imu) -->
+        <accelOffset>0.0 0.0 0.0</accelOffset> <!-- (Vector3): constant acceleration offset -->
+        <accelDrift>0.0 0.0 0.0</accelDrift> <!-- (Vector3): standard deviation of the acceleration drift error -->
+        <accelDriftFrequency>0.0 0.0 0.0</accelDriftFrequency> <!-- (Vector3): mean frequency of the acceleration drift staviti na nulu-->
+        <accelGaussianNoise>0.001 0.001 0.001</accelGaussianNoise> <!-- (Vector3): standard deviation of the additive Gaussian acceleration noise -->
+        <rateOffset>0.0 0.0 0.0</rateOffset> <!-- (Vector3): constant rate offset -->
+        <rateDrift>0.0 0.0 0.0</rateDrift> <!-- (Vector3): standard deviation of the rate drift error -->
+        <rateDriftFrequency>0.0 0.0 0.0</rateDriftFrequency> <!-- (Vector3): mean frequency of the rate drift  staviti na nulu-->
+        <rateGaussianNoise>0.0001 0.0001 0.0001</rateGaussianNoise> <!-- (Vector3): standard deviation of the additive Gaussian rate noise -->
+        <headingOffset>0.0</headingOffset> <!-- (double): constant heading offset -->
+        <headingDrift>0.0</headingDrift> <!-- (double): standard deviation of the heading drift error -->
+        <headingDriftFrequency>0.0</headingDriftFrequency> <!-- (double): mean frequency of the heading drift  staviti na nulu-->
+        <headingGaussianNoise>0.0</headingGaussianNoise> <!-- (double): standard deviation of the heading additive Gaussian noise -->
+        <rpyOffsets>0.0 0.0 0.0</rpyOffsets> <!-- (Vector3): if non-zero, used to calculate accelOffset and headingOffset so that resulting roll, pitch and yaw errors correspond to this values when the platform is leveled (for compatibility with gazebo_plugins) -->
+      </plugin>
+    </gazebo>
+  <!--/xacro:macro-->
 </robot>

File: mmuav_description/urdf/uav_wp_manipulator.gazebo.xacro (robot description, xacro)
@@ -1,26 +1,25 @@
-<?xml version="1.0"?>
+<?xml version='1.0' encoding='utf-8'?>
 <robot name="uav_wp_manipulator" xmlns:xacro="http://ros.org/wiki/xacro">
     <xacro:include filename="$(find mmuav_description)/urdf/uav.gazebo.xacro" />
-    <xacro:include filename="$(find aerial_manipulators/urdf/wp_manipulator.gazebo.xacro)" />
-        <xacro:arg name="gazebo" value="${gazebo}"
-    </xacro:include>
+    <!--xacro:include filename="$(find aerial_manipulators_description)/urdf/wp_manipulator.gazebo.xacro" /-->
     <!-- aditional arm properties -->
-    <xacro:property name="arm_offset_z" value="0.1" /> <!-- [m] 0.0457-->
-    <link name="world">
+    <!--xacro:property name="arm_offset_z" value="0.1" /-->
+    <!-- [m] 0.0457-->
+    <!--link name="world">
     </link>
     <joint name="world_base_joint" type="floating">
         <parent link="world"/>
         <child link="base_link"/>
-    </joint>
+    </joint-->
     <!-- uav -->
-    <xacro:uav enable_bag_plugin=${enable_bag_plugin}
-        mount_velodyne=${mount_velodyne}
-        mount_stereo_cam=${mount_stereo_cam}
-        turn_off_all_collisions=${turn_off_all_collisions}
-        collision_bitmask=${collision_bitmask} />
+    <xacro:uav
+        mount_velodyne="${arg mount_velodyne}"
+        mount_stereo_cam="${arg mount_stereo_cam}"
+        turn_off_all_collisions="${arg turn_off_all_collisions}"
+        collision_bitmask="${arg collision_bitmask}" >
     </xacro:uav>
     <!-- wp_manipulator -->
-    <xacro:wp_manipulator parent="base_link">
-        <origin xyz="0 0 ${arm_offset_z} rpy="0 0 0" />
-    </xacro:wp_manipulator>
+    <!--xacro:wp_manipulator parent="base_link">
+        <origin xyz="0 0 ${arm_offset_z}" rpy="0 0 0" />
+    </xacro:wp_manipulator-->
 </robot>
