Commit message: Dodavanje manipulatora na letjelicu

File: mmuav_description/urdf/uav.base.urdf.xacro (robot description, xacro)
@@ -1,4 +1,4 @@
 <?xml version="1.0"?>
-<robot name="mmcuav" xmlns:xacro="http://ros.org/wiki/xacro">
+<robot name="uav" xmlns:xacro="http://ros.org/wiki/xacro">
   <!-- Properties -->
   <xacro:property name="rotor_velocity_slowdown_sim" value="15" />
@@ -48,12 +48,4 @@
   <!-- Included URDF Files -->
   <xacro:include filename="$(find mmuav_description)/urdf/multirotor_base.urdf.xacro" />
-  <!-- Moving mass inertia block -->
-  <xacro:property name="movable_mass_inertia">
-     <inertia
-     ixx="${mm_mass * (mm_path_len/2 * mm_path_len/2)}"
-     iyy="${mm_mass * (mm_path_len/2 * mm_path_len/2)}"
-     izz="${mm_mass * (mm_path_len/2 * mm_path_len/2)}"
-     ixy="0.0" ixz="0.0"  iyz="0.0" /> <!-- [kg*m^2] [kg*m^2] [kg*m^2] [kg*m^2] [kg*m^2] [kg*m^2] -->
-  </xacro:property>
   <!-- IMU inertia (Pixhawk) -->
   <xacro:property name="imu_inertia">
@@ -155,5 +147,125 @@
     <xacro:insert_block name="rotor_inertia" />
   </xacro:vertical_rotor>
-  <!-- <xacro:camera_macro robot_namespace="${namespace}">
-  </xacro:camera_macro> -->
+  <link name='link01'>
+    <inertial>
+      <mass value="0.001" />
+      <origin xyz="0 0 -0.03" rpy="0 0 0"/>
+      <inertia
+        ixx="0.05" ixy="0" ixz="0"
+        iyx="0" iyy="0.05" iyz="0"
+        izx="0" izy="0" izz="0.05"/>
+    </inertial>
+    <visual>
+      <origin xyz="0 0 -0.03" rpy="0 0 0" />
+      <geometry>
+        <cylinder length="0.08" radius="0.015"/>
+      </geometry>
+    </visual>
+  </link>
+  <link name='con1'>
+    <inertial>
+      <mass value="0.001" />
+      <origin xyz="0 0 -0.07" rpy="0 0 0"/>
+      <inertia
+        ixx="0.05" ixy="0" ixz="0"
+        iyx="0" iyy="0.05" iyz="0"
+        izx="0" izy="0" izz="0.05"/>
+    </inertial>
+    <visual>
+      <origin xyz="0 0 -0.07" rpy="0 0 0" />
+      <geometry>
+        <sphere radius="0.015"/>
+      </geometry>
+    </visual>
+  </link>
+  <link name='link12'>
+    <inertial>
+      <mass value="0.001" />
+      <origin xyz="-0.113137 0.113137 -0.07" rpy="0 0 0"/>
+      <inertia
+        ixx="0.05" ixy="0" ixz="0"
+        iyx="0" iyy="0.05" iyz="0"
+        izx="0" izy="0" izz="0.05"/>
+    </inertial>
+    <visual>
+      <origin xyz="-0.113137 0.113137 -0.07" rpy="0.758398 1.5708 0" />
+      <geometry>
+        <cylinder length="0.32" radius="0.015"/>
+      </geometry>
+    </visual>
+  </link>
+  <link name='con2'>
+    <inertial>
+      <mass value="0.001" />
+      <origin xyz="-0.226274 0.226274 -0.07" rpy="0 0 0"/>
+      <inertia
+        ixx="0.5" ixy="0" ixz="0"
+        iyx="0" iyy="0.5" iyz="0"
+        izx="0" izy="0" izz="0.5"/>
+    </inertial>
+    <visual>
+      <origin xyz="-0.226274 0.226274 -0.07" rpy="0 0 0" />
+      <geometry>
+        <sphere radius="0.015"/>
+      </geometry>
+    </visual>
+  </link>
+  <link name='link23'>
+    <inertial>
+      <mass value="0.001" />
+      <origin xyz="-0.282843 0.282843 -0.07" rpy="0 0 0"/>
+      <inertia
+        ixx="0.5" ixy="0" ixz="0"
+        iyx="0" iyy="0.5" iyz="0"
+        izx="0" izy="0" izz="0.5"/>
+    </inertial>
+    <visual>
+      <origin xyz="-0.282843 0.282843 -0.07" rpy="0.758398 1.5708 0" />
+      <geometry>
+        <cylinder length="0.16" radius="0.015"/>
+      </geometry>
+    </visual>
+  </link>
+  <joint name="base_to_link01" type="fixed">
+    <parent link="base_link"/>
+    <child link="link01"/>
+  </joint>
+  <joint name="link01_to_con1" type="fixed">
+    <parent link="link01"/>
+    <child link="con1"/>
+  </joint>
+  <joint name="con1_to_link12" type="continuous">
+    <parent link="con1"/>
+    <child link="link12"/>
+    <limit upper="3.14" lower="-3.14" effort="10000000" velocity="20"/>
+    <axis xyz="0 0 1" />
+    <dynamics damping="0.07" friction="0.0"/>
+  </joint>
+  <joint name="link12_to_con2" type="fixed">
+    <parent link="link12"/>
+    <child link="con2"/>
+  </joint>
+  <joint name="con2_to_link23" type="continuous">
+    <parent link="con2"/>
+    <child link="link23"/>
+    <origin xyz="0 0 0" rpy="0 0 0"/>
+    <limit upper="3.14" lower="-3.14" effort="10000000" velocity="20"/>
+    <axis xyz="0 0 1" />
+    <dynamics damping="0.07" friction="0.0"/>
+  </joint>
+  <!--
+  <origin xyz="0 0 -0.3" rpy="0 0 0"/>
+  <origin xyz="0 0 -0.07" rpy="0 0 0"/>
+  <origin xyz="0 0 -0.07" rpy="0 0 0"/>
+  <origin xyz="-0.226274 0.226274 -0.07" rpy="0 0 -0.07"/>
+  <origin xyz="-0.226274 0.226274 -0.07" rpy="0 0 0"/>
+  -->
+  <xacro:transmisija
+    trans_number="0"
+    joint_name="con1_to_link12">
+  </xacro:transmisija>
+  <xacro:transmisija
+    trans_number="1"
+    joint_name="con2_to_link23">
+  </xacro:transmisija>
 </robot>

File: mmuav_description/urdf/uav.gazebo.xacro (robot description, xacro)
@@ -1,4 +1,4 @@
 <?xml version="1.0"?>
-<robot name="mmcuav" xmlns:xacro="http://ros.org/wiki/xacro">
+<robot name="uav" xmlns:xacro="http://ros.org/wiki/xacro">
   <!--
   It seems that the xacro:property does not allow to use substitution args. Therefore, instead xacro parameter ${namespace}, subsitution argument is used $(arg name). This is
@@ -13,7 +13,7 @@
   </gazebo>
   <xacro:property name="enable_bag_plugin" value="false" />
-  <xacro:property name="bag_file" value="mmuav.bag" />
+  <xacro:property name="bag_file" value="uav.bag" />
   <!-- Instantiate mmuav "mechanics" -->
-  <xacro:include filename="$(find mmuav_description)/urdf/mmcuav.base.urdf.xacro" />
+  <xacro:include filename="$(find mmuav_description)/urdf/uav.base.urdf.xacro" />
   <xacro:include filename="$(find rotors_description)/urdf/component_snippets.xacro" />
   <!-- Create link and joint for a sensor -->

Commit message: Adding camera manipulator to uav

File: mmuav_description/urdf/uav.base.urdf.xacro (robot description, xacro)
@@ -48,12 +48,4 @@
   <!-- Included URDF Files -->
   <xacro:include filename="$(find mmuav_description)/urdf/multirotor_base.urdf.xacro" />
-  <!-- Moving mass inertia block -->
-  <xacro:property name="movable_mass_inertia">
-     <inertia
-     ixx="${mm_mass * (mm_path_len/2 * mm_path_len/2)}"
-     iyy="${mm_mass * (mm_path_len/2 * mm_path_len/2)}"
-     izz="${mm_mass * (mm_path_len/2 * mm_path_len/2)}"
-     ixy="0.0" ixz="0.0"  iyz="0.0" /> <!-- [kg*m^2] [kg*m^2] [kg*m^2] [kg*m^2] [kg*m^2] [kg*m^2] -->
-  </xacro:property>
   <!-- IMU inertia (Pixhawk) -->
   <xacro:property name="imu_inertia">
@@ -155,21 +147,125 @@
     <xacro:insert_block name="rotor_inertia" />
   </xacro:vertical_rotor>
-  <!-- <xacro:camera_macro robot_namespace="${namespace}">
-  </xacro:camera_macro> -->
-  <!--xacro:transmisija
+  <link name='link01'>
+    <inertial>
+      <mass value="0.001" />
+      <origin xyz="0 0 -0.03" rpy="0 0 0"/>
+      <inertia
+        ixx="0.05" ixy="0" ixz="0"
+        iyx="0" iyy="0.05" iyz="0"
+        izx="0" izy="0" izz="0.05"/>
+    </inertial>
+    <visual>
+      <origin xyz="0 0 -0.03" rpy="0 0 0" />
+      <geometry>
+        <cylinder length="0.08" radius="0.015"/>
+      </geometry>
+    </visual>
+  </link>
+  <link name='con1'>
+    <inertial>
+      <mass value="0.001" />
+      <origin xyz="0 0 -0.07" rpy="0 0 0"/>
+      <inertia
+        ixx="0.05" ixy="0" ixz="0"
+        iyx="0" iyy="0.05" iyz="0"
+        izx="0" izy="0" izz="0.05"/>
+    </inertial>
+    <visual>
+      <origin xyz="0 0 -0.07" rpy="0 0 0" />
+      <geometry>
+        <sphere radius="0.015"/>
+      </geometry>
+    </visual>
+  </link>
+  <link name='link12'>
+    <inertial>
+      <mass value="0.001" />
+      <origin xyz="-0.113137 0.113137 -0.07" rpy="0 0 0"/>
+      <inertia
+        ixx="0.05" ixy="0" ixz="0"
+        iyx="0" iyy="0.05" iyz="0"
+        izx="0" izy="0" izz="0.05"/>
+    </inertial>
+    <visual>
+      <origin xyz="-0.113137 0.113137 -0.07" rpy="0.758398 1.5708 0" />
+      <geometry>
+        <cylinder length="0.32" radius="0.015"/>
+      </geometry>
+    </visual>
+  </link>
+  <link name='con2'>
+    <inertial>
+      <mass value="0.001" />
+      <origin xyz="-0.226274 0.226274 -0.07" rpy="0 0 0"/>
+      <inertia
+        ixx="0.5" ixy="0" ixz="0"
+        iyx="0" iyy="0.5" iyz="0"
+        izx="0" izy="0" izz="0.5"/>
+    </inertial>
+    <visual>
+      <origin xyz="-0.226274 0.226274 -0.07" rpy="0 0 0" />
+      <geometry>
+        <sphere radius="0.015"/>
+      </geometry>
+    </visual>
+  </link>
+  <link name='link23'>
+    <inertial>
+      <mass value="0.001" />
+      <origin xyz="-0.282843 0.282843 -0.07" rpy="0 0 0"/>
+      <inertia
+        ixx="0.5" ixy="0" ixz="0"
+        iyx="0" iyy="0.5" iyz="0"
+        izx="0" izy="0" izz="0.5"/>
+    </inertial>
+    <visual>
+      <origin xyz="-0.282843 0.282843 -0.07" rpy="0.758398 1.5708 0" />
+      <geometry>
+        <cylinder length="0.16" radius="0.015"/>
+      </geometry>
+    </visual>
+  </link>
+  <joint name="base_to_link01" type="fixed">
+    <parent link="base_link"/>
+    <child link="link01"/>
+  </joint>
+  <joint name="link01_to_con1" type="fixed">
+    <parent link="link01"/>
+    <child link="con1"/>
+  </joint>
+  <joint name="con1_to_link12" type="continuous">
+    <parent link="con1"/>
+    <child link="link12"/>
+    <limit upper="3.14" lower="-3.14" effort="10000000" velocity="20"/>
+    <axis xyz="0 0 1" />
+    <dynamics damping="0.07" friction="0.0"/>
+  </joint>
+  <joint name="link12_to_con2" type="fixed">
+    <parent link="link12"/>
+    <child link="con2"/>
+  </joint>
+  <joint name="con2_to_link23" type="continuous">
+    <parent link="con2"/>
+    <child link="link23"/>
+    <origin xyz="0 0 0" rpy="0 0 0"/>
+    <limit upper="3.14" lower="-3.14" effort="10000000" velocity="20"/>
+    <axis xyz="0 0 1" />
+    <dynamics damping="0.07" friction="0.0"/>
+  </joint>
+  <!--
+  <origin xyz="0 0 -0.3" rpy="0 0 0"/>
+  <origin xyz="0 0 -0.07" rpy="0 0 0"/>
+  <origin xyz="0 0 -0.07" rpy="0 0 0"/>
+  <origin xyz="-0.226274 0.226274 -0.07" rpy="0 0 -0.07"/>
+  <origin xyz="-0.226274 0.226274 -0.07" rpy="0 0 0"/>
+  -->
+  <xacro:transmisija
     trans_number="0"
-    joint_name="stick_to_movable_mass_0">
+    joint_name="con1_to_link12">
   </xacro:transmisija>
   <xacro:transmisija
     trans_number="1"
-    joint_name="stick_to_movable_mass_1">
+    joint_name="con2_to_link23">
   </xacro:transmisija>
-  <xacro:transmisija
-    trans_number="2"
-    joint_name="stick_to_movable_mass_2">
-  </xacro:transmisija>
-  <xacro:transmisija
-    trans_number="3"
-    joint_name="stick_to_movable_mass_3">
-  </xacro:transmisija-->
 </robot>

Commit message: Fixing camera manip urdf and yaml

File: mmuav_description/urdf/uav.base.urdf.xacro (robot description, xacro)
@@ -147,8 +147,24 @@
     <xacro:insert_block name="rotor_inertia" />
   </xacro:vertical_rotor>
-  <link name='link01'>
+    <link name='connector1'>
+      <inertial>
+        <mass value="0.001" />
+        <origin xyz="0 0 -0.04" rpy="0 0 0"/>
+        <inertia
+          ixx="0.05" ixy="0" ixz="0"
+          iyx="0" iyy="0.05" iyz="0"
+          izx="0" izy="0" izz="0.05"/>
+      </inertial>
+      <visual>
+        <origin xyz="0 0 -0.04" rpy="0 0 0" />
+        <geometry>
+          <cylinder length="0.1" radius="0.02"/>
+        </geometry>
+      </visual>
+    </link>
+  <link name='link1'>
     <inertial>
       <mass value="0.001" />
-      <origin xyz="0 0 -0.03" rpy="0 0 0"/>
+      <origin xyz="-0.09899494936 0.09899494936 -0.01" rpy="0 0 0"/>
       <inertia
         ixx="0.05" ixy="0" ixz="0"
@@ -157,115 +173,75 @@
     </inertial>
     <visual>
-      <origin xyz="0 0 -0.03" rpy="0 0 0" />
+      <origin xyz="-0.09899494936 0.09899494936 -0.01" rpy="0.758398 1.5708 0" />
       <geometry>
-        <cylinder length="0.08" radius="0.015"/>
+        <box size="0.02 0.04 0.32"/>
       </geometry>
     </visual>
   </link>
-  <link name='con1'>
-    <inertial>
-      <mass value="0.001" />
-      <origin xyz="0 0 -0.07" rpy="0 0 0"/>
-      <inertia
-        ixx="0.05" ixy="0" ixz="0"
-        iyx="0" iyy="0.05" iyz="0"
-        izx="0" izy="0" izz="0.05"/>
-    </inertial>
-    <visual>
-      <origin xyz="0 0 -0.07" rpy="0 0 0" />
-      <geometry>
-        <sphere radius="0.015"/>
-      </geometry>
-    </visual>
-  </link>
-  <link name='link12'>
-    <inertial>
-      <mass value="0.001" />
-      <origin xyz="-0.113137 0.113137 -0.07" rpy="0 0 0"/>
-      <inertia
-        ixx="0.05" ixy="0" ixz="0"
-        iyx="0" iyy="0.05" iyz="0"
-        izx="0" izy="0" izz="0.05"/>
-    </inertial>
-    <visual>
-      <origin xyz="-0.113137 0.113137 -0.07" rpy="0.758398 1.5708 0" />
-      <geometry>
-        <cylinder length="0.32" radius="0.015"/>
-      </geometry>
-    </visual>
-  </link>
-  <link name='con2'>
-    <inertial>
-      <mass value="0.001" />
-      <origin xyz="-0.226274 0.226274 -0.07" rpy="0 0 0"/>
-      <inertia
-        ixx="0.5" ixy="0" ixz="0"
-        iyx="0" iyy="0.5" iyz="0"
-        izx="0" izy="0" izz="0.5"/>
-    </inertial>
-    <visual>
-      <origin xyz="-0.226274 0.226274 -0.07" rpy="0 0 0" />
-      <geometry>
-        <sphere radius="0.015"/>
-      </geometry>
-    </visual>
-  </link>
-  <link name='link23'>
-    <inertial>
-      <mass value="0.001" />
-      <origin xyz="-0.282843 0.282843 -0.07" rpy="0 0 0"/>
-      <inertia
-        ixx="0.5" ixy="0" ixz="0"
-        iyx="0" iyy="0.5" iyz="0"
-        izx="0" izy="0" izz="0.5"/>
-    </inertial>
-    <visual>
-      <origin xyz="-0.282843 0.282843 -0.07" rpy="0.758398 1.5708 0" />
-      <geometry>
-        <cylinder length="0.16" radius="0.015"/>
-      </geometry>
-    </visual>
-  </link>
-  <joint name="base_to_link01" type="fixed">
-    <parent link="base_link"/>
-    <child link="link01"/>
-  </joint>
-  <joint name="link01_to_con1" type="fixed">
-    <parent link="link01"/>
-    <child link="con1"/>
-  </joint>
-  <joint name="con1_to_link12" type="continuous">
-    <parent link="con1"/>
-    <child link="link12"/>
-    <limit upper="3.14" lower="-3.14" effort="10000000" velocity="20"/>
-    <axis xyz="0 0 1" />
-    <dynamics damping="0.07" friction="0.0"/>
-  </joint>
-  <joint name="link12_to_con2" type="fixed">
-    <parent link="link12"/>
-    <child link="con2"/>
-  </joint>
-  <joint name="con2_to_link23" type="continuous">
-    <parent link="con2"/>
-    <child link="link23"/>
-    <origin xyz="0 0 0" rpy="0 0 0"/>
-    <limit upper="3.14" lower="-3.14" effort="10000000" velocity="20"/>
-    <axis xyz="0 0 1" />
-    <dynamics damping="0.07" friction="0.0"/>
-  </joint>
-  <!--
-  <origin xyz="0 0 -0.3" rpy="0 0 0"/>
-  <origin xyz="0 0 -0.07" rpy="0 0 0"/>
-  <origin xyz="0 0 -0.07" rpy="0 0 0"/>
-  <origin xyz="-0.226274 0.226274 -0.07" rpy="0 0 -0.07"/>
-  <origin xyz="-0.226274 0.226274 -0.07" rpy="0 0 0"/>
-  -->
-  <xacro:transmisija
-    trans_number="0"
-    joint_name="con1_to_link12">
-  </xacro:transmisija>
-  <xacro:transmisija
-    trans_number="1"
-    joint_name="con2_to_link23">
-  </xacro:transmisija>
+    <link name='connector2'>
+      <inertial>
+        <mass value="0.001" />
+        <origin xyz="0 0 0" rpy="0 0 0"/>
+        <inertia
+          ixx="0.05" ixy="0" ixz="0"
+          iyx="0" iyy="0.05" iyz="0"
+          izx="0" izy="0" izz="0.05"/>
+      </inertial>
+      <visual>
+        <origin xyz="0 0 -0.02" rpy="0 0 0" />
+        <geometry>
+          <cylinder length="0.02" radius="0.02"/>
+        </geometry>
+      </visual>
+    </link>
+    <link name='link2'>
+      <inertial>
+        <mass value="0.001" />
+        <origin xyz="-0.09899494936 0.09899494936 -0.02" rpy="0 0 0"/>
+        <inertia
+          ixx="0.05" ixy="0" ixz="0"
+          iyx="0" iyy="0.05" iyz="0"
+          izx="0" izy="0" izz="0.05"/>
+      </inertial>
+      <visual>
+        <origin xyz="-0.09899494936 0.09899494936 -0.02" rpy="0.758398 1.5708 0" />
+        <geometry>
+          <box size="0.02 0.04 0.32"/>
+        </geometry>
+      </visual>
+    </link>
+    <joint name="base_to_connector1" type="fixed">
+      <parent link="base_link"/>
+      <child link="connector1"/>
+      <origin xyz="0 0 0" rpy="0 0 0"/>
+    </joint>
+    <joint name="connecto1_to_link1" type="continuous">
+      <parent link="connector1"/>
+      <child link="link1"/>
+      <origin xyz="0 0 -0.09" rpy="0 0 0"/>
+      <limit upper="3.14" lower="-3.14" effort="10000000" velocity="20"/>
+      <axis xyz="0 0 1" />
+      <dynamics damping="0.07" friction="0.0"/>
+    </joint>
+    <joint name="link1_to_connector2" type="fixed">
+      <parent link="link1"/>
+      <child link="connector2"/>
+      <origin xyz="-0.19798989873 0.19798989873 -0.01" rpy="0 0 0"/>
+    </joint>
+    <joint name="connector2_to_link2" type="continuous">
+      <parent link="connector2"/>
+      <child link="link2"/>
+      <origin xyz="0 0 -0.02" rpy="0 0 0"/>
+      <limit upper="3.14" lower="-3.14" effort="10000000" velocity="20"/>
+      <axis xyz="0 0 1" />
+      <dynamics damping="0.07" friction="0.0"/>
+    </joint>
+    <xacro:transmisija
+      trans_number="0"
+      joint_name="connecto1_to_link1">
+    </xacro:transmisija>
+    <xacro:transmisija
+      trans_number="1"
+      joint_name="connector2_to_link2">
+    </xacro:transmisija>
 </robot>

Commit message: Fixing typos

File: mmuav_description/urdf/uav.base.urdf.xacro (robot description, xacro)
@@ -216,5 +216,5 @@
       <origin xyz="0 0 0" rpy="0 0 0"/>
     </joint>
-    <joint name="connecto1_to_link1" type="continuous">
+    <joint name="connector1_to_link1" type="continuous">
       <parent link="connector1"/>
       <child link="link1"/>
@@ -239,5 +239,5 @@
     <xacro:transmisija
       trans_number="0"
-      joint_name="connecto1_to_link1">
+      joint_name="connector1_to_link1">
     </xacro:transmisija>
     <xacro:transmisija

Commit message: Adjusting mass and inertia matrix

File: mmuav_description/urdf/uav.base.urdf.xacro (robot description, xacro)
@@ -149,10 +149,10 @@
     <link name='connector1'>
       <inertial>
-        <mass value="0.001" />
+        <mass value="0.0126" />
         <origin xyz="0 0 -0.04" rpy="0 0 0"/>
         <inertia
-          ixx="0.05" ixy="0" ixz="0"
-          iyx="0" iyy="0.05" iyz="0"
-          izx="0" izy="0" izz="0.05"/>
+          ixx="0.00001176" ixy="0" ixz="0"
+          iyx="0" iyy="0.00001176" iyz="0"
+          izx="0" izy="0" izz="0.00000252"/>
       </inertial>
       <visual>
@@ -165,10 +165,10 @@
   <link name='link1'>
     <inertial>
-      <mass value="0.001" />
+      <mass value="0.0256" />
       <origin xyz="-0.09899494936 0.09899494936 -0.01" rpy="0 0 0"/>
       <inertia
-        ixx="0.05" ixy="0" ixz="0"
-        iyx="0" iyy="0.05" iyz="0"
-        izx="0" izy="0" izz="0.05"/>
+        ixx="0.000004266" ixy="0" ixz="0"
+        iyx="0" iyy="0.002" iyz="0"
+        izx="0" izy="0" izz="0.000262827"/>
     </inertial>
     <visual>
@@ -181,10 +181,10 @@
     <link name='connector2'>
       <inertial>
-        <mass value="0.001" />
+        <mass value="0.00251" />
         <origin xyz="0 0 0" rpy="0 0 0"/>
         <inertia
-          ixx="0.05" ixy="0" ixz="0"
-          iyx="0" iyy="0.05" iyz="0"
-          izx="0" izy="0" izz="0.05"/>
+          ixx="0.0000003346" ixy="0" ixz="0"
+          iyx="0" iyy="0.0000003346" iyz="0"
+          izx="0" izy="0" izz="0.000000502"/>
       </inertial>
       <visual>
@@ -197,11 +197,11 @@
     <link name='link2'>
       <inertial>
-        <mass value="0.001" />
+        <mass value="0.0256" />
         <origin xyz="-0.09899494936 0.09899494936 -0.02" rpy="0 0 0"/>
         <inertia
-          ixx="0.05" ixy="0" ixz="0"
-          iyx="0" iyy="0.05" iyz="0"
-          izx="0" izy="0" izz="0.05"/>
-      </inertial>
+          ixx="0.000004266" ixy="0" ixz="0"
+          iyx="0" iyy="0.002" iyz="0"
+          izx="0" izy="0" izz="0.000262827"/>
+    </inertial>
       <visual>
         <origin xyz="-0.09899494936 0.09899494936 -0.02" rpy="0.758398 1.5708 0" />

Commit message: Switched to regular UAV, added landing gear

File: mmuav_description/urdf/uav.base.urdf.xacro (robot description, xacro)
@@ -155,21 +155,31 @@
     <xacro:insert_block name="rotor_inertia" />
   </xacro:vertical_rotor>
-  <!-- <xacro:camera_macro robot_namespace="${namespace}">
-  </xacro:camera_macro> -->
-  <!--xacro:transmisija
-    trans_number="0"
-    joint_name="stick_to_movable_mass_0">
-  </xacro:transmisija>
-  <xacro:transmisija
-    trans_number="1"
-    joint_name="stick_to_movable_mass_1">
-  </xacro:transmisija>
-  <xacro:transmisija
-    trans_number="2"
-    joint_name="stick_to_movable_mass_2">
-  </xacro:transmisija>
-  <xacro:transmisija
-    trans_number="3"
-    joint_name="stick_to_movable_mass_3">
-  </xacro:transmisija-->
+  <!-- Added landing gear -->
+  <xacro:property name="land_gear_inertia">
+    <inertia
+    ixx="1e-6"
+    iyy="1e-6"
+    izz="1e-6"
+    ixy="0.0" ixz="0.0"  iyz="0.0" /> <!-- [kg*m^2] [kg*m^2] [kg*m^2] [kg*m^2] [kg*m^2] [kg*m^2] -->
+  </xacro:property>
+  <xacro:landing_gear
+      parent="base_link"
+      gear_num = "1"
+      mass = "1e-6"
+      dim_x = "0.8"
+      dim_y = "0.1"
+      dim_z = "0.05">
+      <origin xyz="0 -0.325 -0.1" rpy="0 0 0" />
+      <xacro:insert_block name="land_gear_inertia"/>
+  </xacro:landing_gear>
+  <xacro:landing_gear
+      parent="base_link"
+      gear_num = "2"
+      mass = "1e-6"
+      dim_x = "0.8"
+      dim_y = "0.1"
+      dim_z = "0.05">
+      <origin xyz="0 0.325 -0.1" rpy="0 0 0" />
+      <xacro:insert_block name="land_gear_inertia"/>
+  </xacro:landing_gear>
 </robot>

Commit message: Add manipulator option to the uav.

File: mmuav_description/urdf/uav.base.urdf.xacro (robot description, xacro)
@@ -1,4 +1,7 @@
 <?xml version="1.0"?>
 <robot name="uav" xmlns:xacro="http://ros.org/wiki/xacro">
+  <!-- Arguments -->
+  <xacro:arg name="manipulator_type" default="none" />
+  <xacro:property name="manipulator_type" value="$(arg manipulator_type)" />
   <!-- Properties -->
   <xacro:property name="rotor_velocity_slowdown_sim" value="15" />
@@ -155,4 +158,31 @@
     <xacro:insert_block name="rotor_inertia" />
   </xacro:vertical_rotor>
+  <xacro:if value="${'cmanip' == manipulator_type}">
+    <!-- Try to include manipulator -->
+    <xacro:include filename="$(find aerial_manipulators)/urdf/manipulator_base.urdf.xacro" />
+    <xacro:cmanip parent="base_link">
+      <origin xyz="0 0 0.075" rpy="${pi/2} 0 ${pi}"/>
+    </xacro:cmanip>
+    <xacro:transmisija
+      trans_number="1"
+      joint_name="link0_to_link1">
+    </xacro:transmisija>
+    <xacro:transmisija
+      trans_number="2"
+      joint_name="link1_to_link2">
+    </xacro:transmisija>
+    <xacro:transmisija
+      trans_number="3"
+      joint_name="link2_to_link3">
+    </xacro:transmisija>
+    <xacro:transmisija
+      trans_number="4"
+      joint_name="link3_to_link4">
+    </xacro:transmisija>
+    <xacro:transmisija
+      trans_number="5"
+      joint_name="link4_to_link5">
+    </xacro:transmisija>
+  </xacro:if>
   <!-- <xacro:camera_macro robot_namespace="${namespace}">
   </xacro:camera_macro> -->
