Commit message: Enable camera on the UAV

File: mmuav_description/urdf/uav.base.urdf.xacro (robot description, xacro)
@@ -155,6 +155,13 @@
     <xacro:insert_block name="rotor_inertia" />
   </xacro:vertical_rotor>
-  <!-- <xacro:camera_macro robot_namespace="${namespace}">
-  </xacro:camera_macro> -->
+  <xacro:cam
+      namespace="$(arg name)"
+      parent="base_link"
+      camera_link="0.01"
+      camera_mass="0.01">
+      <origin xyz="0 0 -0.2" rpy="0 ${PI/2} ${-PI/4}"/>
+      <inertia ixx="0.001"  ixy="0.0"  ixz="0.0"
+               iyy="0.001"  iyz="0.0"  izz="0.001" />
+    </xacro:cam>
   <!--xacro:transmisija
     trans_number="0"

Commit message: Add camera on the end effector link of manipulator

File: mmuav_description/urdf/uav.base.urdf.xacro (robot description, xacro)
@@ -184,4 +184,20 @@
       joint_name="joint5">
     </xacro:transmisija>
+    <xacro:property name="camera_link" value="0.02" />
+    <xacro:property name="camera_inertia">
+      <inertia
+      ixx="1e-8"
+      iyy="1e-8"
+      izz="1e-8"
+      ixy="0.0" ixz="0.0" iyz="0.0" />
+    </xacro:property>
+    <xacro:property name="camera_mass" value="1e-5"/>
+    <xacro:cam
+      camera_link="${camera_link}"
+      camera_mass="${camera_mass}"
+      parent="end_effector_base">
+      <origin xyz="0 0 0" rpy="${PI} 0 0"/>
+      <xacro:insert_block name="camera_inertia"/>
+    </xacro:cam>
   </xacro:if>
   <!-- <xacro:camera_macro robot_namespace="${namespace}">

Commit message: Add option for different toll attachment to manipulator.

File: mmuav_description/urdf/uav.base.urdf.xacro (robot description, xacro)
@@ -4,4 +4,6 @@
   <xacro:arg name="manipulator_type" default="none" />
   <xacro:property name="manipulator_type" value="$(arg manipulator_type)" />
+  <xacro:arg name="manipulator_tool" default="none" />
+  <xacro:property name="manipulator_tool" value="$(arg manipulator_tool)" />
   <!-- Properties -->
   <xacro:property name="rotor_velocity_slowdown_sim" value="15" />
@@ -184,20 +186,22 @@
       joint_name="joint5">
     </xacro:transmisija>
-    <xacro:property name="camera_link" value="0.02" />
-    <xacro:property name="camera_inertia">
-      <inertia
-      ixx="1e-8"
-      iyy="1e-8"
-      izz="1e-8"
-      ixy="0.0" ixz="0.0" iyz="0.0" />
-    </xacro:property>
-    <xacro:property name="camera_mass" value="1e-5"/>
-    <xacro:cam
-      camera_link="${camera_link}"
-      camera_mass="${camera_mass}"
-      parent="end_effector_base">
-      <origin xyz="0 0 0" rpy="${PI} 0 0"/>
-      <xacro:insert_block name="camera_inertia"/>
-    </xacro:cam>
+    <xacro:if value="${'camera' == manipulator_tool}">
+      <xacro:property name="camera_link" value="0.02" />
+      <xacro:property name="camera_inertia">
+        <inertia
+        ixx="1e-8"
+        iyy="1e-8"
+        izz="1e-8"
+        ixy="0.0" ixz="0.0" iyz="0.0" />
+      </xacro:property>
+      <xacro:property name="camera_mass" value="1e-5"/>
+      <xacro:cam
+        camera_link="${camera_link}"
+        camera_mass="${camera_mass}"
+        parent="end_effector_base">
+        <origin xyz="0 0 0" rpy="${PI} 0 0"/>
+        <xacro:insert_block name="camera_inertia"/>
+      </xacro:cam>
+    </xacro:if>>
   </xacro:if>
   <!-- <xacro:camera_macro robot_namespace="${namespace}">

Commit message: Add rod shaped tool.

File: mmuav_description/urdf/uav.base.urdf.xacro (robot description, xacro)
@@ -203,5 +203,37 @@
         <xacro:insert_block name="camera_inertia"/>
       </xacro:cam>
-    </xacro:if>>
+    </xacro:if>
+    <xacro:if value="${'rod' == manipulator_tool}">
+      <!-- Rod link -->
+      <link name="rod">
+        <!--collision>
+          <origin xyz="0 0 0" rpy="0 0 0"/>
+          <geometry>
+            <box size="${camera_link} ${camera_link} ${camera_link}"/>
+          </geometry>
+        </collision-->
+        <visual>
+          <origin xyz="0.15 0 0" rpy="0 0 0"/>
+          <geometry>
+            <box size="0.3 0.01 0.01"/>
+          </geometry>
+          <material name="red"/>
+        </visual>
+        <inertial>
+          <mass value="0.00001" />
+          <origin xyz="0.15 0 0" rpy="0 0 0"/>
+          <inertia
+            ixx="0" ixy="0" ixz="0"
+            iyx="0" iyy="0" iyz="0"
+            izx="0" izy="0" izz="0"/>
+        </inertial>
+      </link>
+      <!-- Rod joint with reference to the parent link -->
+      <joint name="rod_joint" type="fixed">
+        <origin xyz="0 0 0" rpy="0 0 0" />
+        <parent link="end_effector_base"/>
+        <child link="rod"/>
+      </joint>
+    </xacro:if>
   </xacro:if>
   <!-- <xacro:camera_macro robot_namespace="${namespace}">

Commit message: Add collision to wp manipulator rod

File: mmuav_description/urdf/uav.base.urdf.xacro (robot description, xacro)
@@ -220,4 +220,10 @@
           <material name="red"/>
         </visual>
+        <collision>
+          <origin xyz="0.15 0 0" rpy="0 0 0"/>
+          <geometry>
+              <box size="0.3 0.01 0.01"/>
+          </geometry>
+        </collision>
         <inertial>
           <mass value="0.00001" />

Commit message: added new manipulator

File: mmuav_description/urdf/uav.base.urdf.xacro (robot description, xacro)
@@ -275,4 +275,100 @@
     </xacro:if>
   </xacro:if>
+  <xacro:if value="${'wp_manipulator_3rx' == manipulator_type}">
+    <!-- Try to include manipulator -->
+    <xacro:include filename="$(find aerial_manipulators_description)/urdf/manipulator_base.urdf.xacro" />
+    <xacro:wp_manipulator_3rx parent="base_link">
+      <origin xyz="0 0 0.2" rpy="${pi/2} 0 0"/>
+    </xacro:wp_manipulator_3rx>
+    <xacro:transmisija
+      trans_number="1"
+      joint_name="joint1">
+    </xacro:transmisija>
+    <xacro:transmisija
+      trans_number="2"
+      joint_name="joint2">
+    </xacro:transmisija>
+    <xacro:transmisija
+      trans_number="3"
+      joint_name="joint3">
+    </xacro:transmisija>
+    <xacro:if value="${'camera' == manipulator_tool}">
+      <xacro:property name="camera_link" value="0.02" />
+      <xacro:property name="camera_inertia">
+        <inertia
+        ixx="1e-8"
+        iyy="1e-8"
+        izz="1e-8"
+        ixy="0.0" ixz="0.0" iyz="0.0" />
+      </xacro:property>
+      <xacro:property name="camera_mass" value="1e-5"/>
+      <xacro:cam
+        camera_link="${camera_link}"
+        camera_mass="${camera_mass}"
+        parent="end_effector_base">
+        <origin xyz="0 0 0" rpy="${PI} 0 0"/>
+        <xacro:insert_block name="camera_inertia"/>
+      </xacro:cam>
+    </xacro:if>
+    <!-- Enable the Joint Feedback -->
+    <gazebo reference="joint3">
+      <stopCfm>0.08</stopCfm>
+      <stopErp>0.2</stopErp>
+      <implicitSpringDamper>true</implicitSpringDamper>
+      <provideFeedback>true</provideFeedback>
+    </gazebo>
+    <!-- The ft_sensor plugin  -->
+    <gazebo>
+      <plugin name="ft_sensor" filename="libgazebo_ros_ft_sensor.so">
+        <updateRate>1000.0</updateRate>
+        <robotNamespace>$(arg name)/wp_manipulator</robotNamespace>
+        <topicName>force_sensor/ft_sensor</topicName>
+        <jointName>joint3</jointName>
+        <noise>
+          <type>gaussian</type>
+          <mean>0.0</mean>
+          <stddev>0.0001</stddev> <!-- change this to simulate noise -->
+        </noise>
+      </plugin>
+    </gazebo>
+    <xacro:if value="${'rod' == manipulator_tool}">
+      <!-- Rod link -->
+      <link name="rod">
+        <!--collision>
+          <origin xyz="0 0 0" rpy="0 0 0"/>
+          <geometry>
+            <box size="${camera_link} ${camera_link} ${camera_link}"/>
+          </geometry>
+        </collision-->
+        <visual>
+          <origin xyz="0.15 0 0" rpy="0 0 0"/>
+          <geometry>
+            <box size="0.3 0.01 0.01"/>
+          </geometry>
+          <material name="red"/>
+        </visual>
+        <collision>
+          <origin xyz="0.15 0 0" rpy="0 0 0"/>
+          <geometry>
+              <box size="0.3 0.01 0.01"/>
+          </geometry>
+        </collision>
+        <inertial>
+          <mass value="0.00001" />
+          <origin xyz="0.15 0 0" rpy="0 0 0"/>
+          <inertia
+            ixx="0" ixy="0" ixz="0"
+            iyx="0" iyy="0" iyz="0"
+            izx="0" izy="0" izz="0"/>
+        </inertial>
+      </link>
+      <!-- Rod joint with reference to the parent link -->
+      <joint name="rod_joint" type="fixed">
+        <origin xyz="0 0 0" rpy="0 0 0" />
+        <parent link="end_effector_base"/>
+        <child link="rod"/>
+      </joint>
+    </xacro:if>
+  </xacro:if>
   <!-- <xacro:camera_macro robot_namespace="${namespace}">
   </xacro:camera_macro> -->

Commit message: Change manipulator rod color.

File: mmuav_description/urdf/uav.base.urdf.xacro (robot description, xacro)
@@ -267,4 +267,7 @@
         </inertial>
       </link>
+      <gazebo reference="rod">
+        <material>Gazebo/Red</material>
+      </gazebo>
       <!-- Rod joint with reference to the parent link -->
       <joint name="rod_joint" type="fixed">

Commit message: Add kinect camera end effector option.

File: mmuav_description/urdf/uav.base.urdf.xacro (robot description, xacro)
@@ -238,5 +238,5 @@
       </plugin>
     </gazebo>
-    <xacro:if value="${'rod' == manipulator_tool or 'rod_with_camera' == manipulator_tool}">
+    <xacro:if value="${'rod' == manipulator_tool or 'rod_with_camera' == manipulator_tool or 'rod_with_kinect' == manipulator_tool}">
       <!-- Rod link -->
       <link name="rod">
@@ -300,4 +300,27 @@
           <xacro:insert_block name="rod_camera_inertia"/>
         </xacro:cam>
+      </xacro:if>
+      <!-- Add stereo camera only if requested -->
+      <xacro:if value="${'rod_with_kinect' == manipulator_tool}">
+        <xacro:property name="rod_camera_link" value="0.02" />
+        <xacro:property name="rod_camera_inertia">
+          <inertia
+          ixx="1e-8"
+          iyy="1e-8"
+          izz="1e-8"
+          ixy="0.0" ixz="0.0" iyz="0.0" />
+        </xacro:property>
+        <xacro:property name="rod_camera_mass" value="1e-5"/>
+        <xacro:property name="rod_kinect_transform">
+          <origin xyz="0.3 0 0.0" rpy="${PI} ${PI/2} 0"/>
+        </xacro:property>
+        <xacro:stereo_cam
+          namespace="$(arg name)"
+          camera_link="${rod_camera_link}"
+          camera_mass="${rod_camera_mass}"
+          parent="rod">
+          <xacro:insert_block name="rod_kinect_transform"/>
+          <xacro:insert_block name="rod_camera_inertia"/>
+        </xacro:stereo_cam>
       </xacro:if>
     </xacro:if>

Commit message: Add camera pose sensor.

File: mmuav_description/urdf/uav.base.urdf.xacro (robot description, xacro)
@@ -313,5 +313,5 @@
         <xacro:property name="rod_camera_mass" value="1e-5"/>
         <xacro:property name="rod_kinect_transform">
-          <origin xyz="0.3 0 0.0" rpy="${PI} ${PI/2} 0"/>
+          <origin xyz="0.3 0 0.0" rpy="${PI} 0 0"/>
         </xacro:property>
         <xacro:stereo_cam

File: mmuav_description/urdf/uav.gazebo.xacro (robot description, xacro)
@@ -26,4 +26,6 @@
   <xacro:arg name="turn_off_all_collisions" default="false" />
   <xacro:property name="turn_off_all_collisions" value="$(arg turn_off_all_collisions)" />
+  <xacro:arg name="manipulator_tool" default="none" />
+  <xacro:property name="manipulator_tool" value="$(arg manipulator_tool)" />
 	<xacro:property name="front_facing_camera">
 		<origin xyz="0.025 0 0.1" rpy="0 0 0"/>
@@ -162,4 +164,37 @@
     <origin xyz="0.0 0.0 0" rpy="0.0 0.0 0.0" />
   </xacro:odometry_plugin_macro>
+  <xacro:if value="${'rod_with_camera' == manipulator_tool}">
+    <xacro:odometry_plugin_macro
+    namespace="$(arg name)"
+    odometry_sensor_suffix="2"
+    child_frame_id="base"
+    parent_link="camera_box"
+    pose_topic="camera/pose"
+    velocity_relative_topic="camera/velocity_relative"
+    pose_with_covariance_topic="camera/pose_with_covariance"
+    position_topic="camera/position"
+    transform_topic="camera/transform"
+    odometry_topic="camera/odometry"
+    parent_frame_id="world"
+    mass_odometry_sensor="1e-5"
+    measurement_divisor="5"
+    measurement_delay="0"
+    unknown_delay="0.0"
+    noise_normal_position="0.0 0.0 0.0"
+    noise_normal_quaternion="0.0 0.0 0.0"
+    noise_normal_linear_velocity="0.0 0.0 0.0"
+    noise_normal_angular_velocity="0.0 0.0 0.0"
+    noise_uniform_position="0.0 0.0 0.0"
+    noise_uniform_quaternion="0.0 0.0 0.0"
+    noise_uniform_linear_velocity="0.0 0.0 0.0"
+    noise_uniform_angular_velocity="0.0 0.0 0.0"
+    enable_odometry_map="false"
+    odometry_map=""
+    image_scale="">
+    <inertia ixx="1e-6" ixy="0.0" ixz="0.0" iyy="1e-6" iyz="0.0" izz="1e-6" /> <!-- [kg m^2] [kg m^2] [kg m^2] [kg m^2] [kg m^2] [kg m^2] -->
+    <!-- This rotation is correction for blender. -->
+    <origin xyz="0.0 0.0 0" rpy="1.57 0.0 -1.57" />
+  </xacro:odometry_plugin_macro>
+  </xacro:if>
   <!-- mount gimbal -->
   <!--<xacro:gimbal_macro parent="base_link">

Commit message: Change wp manipulator 3rx transform.

File: mmuav_description/urdf/uav.base.urdf.xacro (robot description, xacro)
@@ -330,5 +330,6 @@
     <xacro:include filename="$(find aerial_manipulators_description)/urdf/manipulator_base.urdf.xacro" />
     <xacro:wp_manipulator_3rx parent="base_link">
-      <origin xyz="0 0 0.2" rpy="${pi/2} 0 0"/>
+      <!--origin xyz="0 0 0.2" rpy="${pi/2} 0 0"/-->
+      <origin xyz="0 0 0.2" rpy="0 0 0"/>
     </xacro:wp_manipulator_3rx>
     <xacro:transmisija

Commit message: added asap_manipulator to UAV

File: mmuav_description/urdf/uav.base.urdf.xacro (robot description, xacro)
@@ -447,4 +447,120 @@
     </xacro:if>
   </xacro:if>
+  <xacro:if value="${'asap_manipulator' == manipulator_type}">
+    <!-- Try to include manipulator -->
+    <xacro:include filename="$(find aerial_manipulators_description)/urdf/manipulator_base.urdf.xacro" />
+    <xacro:asap_manipulator parent="base_link">
+      <!--origin xyz="0 0 0.2" rpy="${pi/2} 0 0"/-->
+      <origin xyz="0 0 0.2" rpy="0 0 0"/>
+    </xacro:asap_manipulator>
+    <xacro:transmisija
+      trans_number="1"
+      joint_name="joint1">
+    </xacro:transmisija>
+    <xacro:transmisija
+      trans_number="2"
+      joint_name="joint2">
+    </xacro:transmisija>
+    <xacro:transmisija
+      trans_number="3"
+      joint_name="joint3">
+    </xacro:transmisija>
+    <xacro:transmisija
+      trans_number="4"
+      joint_name="joint4">
+    </xacro:transmisija>
+    <xacro:transmisija
+      trans_number="5"
+      joint_name="joint5">
+    </xacro:transmisija>
+    <xacro:if value="${'camera' == manipulator_tool}">
+      <xacro:property name="camera_link" value="0.02" />
+      <xacro:property name="camera_inertia">
+        <inertia
+        ixx="1e-8"
+        iyy="1e-8"
+        izz="1e-8"
+        ixy="0.0" ixz="0.0" iyz="0.0" />
+      </xacro:property>
+      <xacro:property name="camera_mass" value="1e-5"/>
+      <xacro:cam
+        camera_link="${camera_link}"
+        camera_mass="${camera_mass}"
+        parent="end_effector_base">
+        <origin xyz="0 0 0" rpy="${PI} 0 0"/>
+        <xacro:insert_block name="camera_inertia"/>
+      </xacro:cam>
+    </xacro:if>
+    <!-- Enable the Joint Feedback -->
+    <gazebo reference="joint5">
+      <stopCfm>0.08</stopCfm>
+      <stopErp>0.2</stopErp>
+      <implicitSpringDamper>true</implicitSpringDamper>
+      <provideFeedback>true</provideFeedback>
+    </gazebo>
+    <!-- The ft_sensor plugin  -->
+    <gazebo>
+      <plugin name="ft_sensor" filename="libgazebo_ros_ft_sensor.so">
+        <updateRate>1000.0</updateRate>
+        <robotNamespace>$(arg name)/asap_manipulator</robotNamespace>
+        <topicName>force_sensor/ft_sensor</topicName>
+        <jointName>joint5</jointName>
+        <noise>
+          <type>gaussian</type>
+          <mean>0.0</mean>
+          <stddev>0.0001</stddev> <!-- change this to simulate noise -->
+        </noise>
+      </plugin>
+    </gazebo>
+    <xacro:if value="${'rod' == manipulator_tool}">
+      <gazebo reference="rod">
+        <collision>
+          <surface>
+            <contact>
+              <collide_bitmask>${collision_bitmask}</collide_bitmask>
+            </contact>
+          </surface>
+        </collision>
+      </gazebo>
+      <!-- Rod link -->
+      <link name="rod">
+        <!--collision>
+          <origin xyz="0 0 0" rpy="0 0 0"/>
+          <geometry>
+            <box size="${camera_link} ${camera_link} ${camera_link}"/>
+          </geometry>
+        </collision-->
+        <visual>
+          <origin xyz="0.15 0 0" rpy="0 0 0"/>
+          <geometry>
+            <box size="0.3 0.01 0.01"/>
+          </geometry>
+          <material name="red"/>
+        </visual>
+        <xacro:unless value="${turn_off_all_collisions}">
+          <collision>
+            <origin xyz="0.15 0 0" rpy="0 0 0"/>
+            <geometry>
+                <box size="0.3 0.01 0.01"/>
+            </geometry>
+          </collision>
+        </xacro:unless>
+        <inertial>
+          <mass value="0.00001" />
+          <origin xyz="0.15 0 0" rpy="0 0 0"/>
+          <inertia
+            ixx="0" ixy="0" ixz="0"
+            iyx="0" iyy="0" iyz="0"
+            izx="0" izy="0" izz="0"/>
+        </inertial>
+      </link>
+      <!-- Rod joint with reference to the parent link -->
+      <joint name="rod_joint" type="fixed">
+        <origin xyz="0 0 0" rpy="0 0 0" />
+        <parent link="end_effector_base"/>
+        <child link="rod"/>
+      </joint>
+    </xacro:if>
+  </xacro:if>
   <!-- <xacro:camera_macro robot_namespace="${namespace}">
   </xacro:camera_macro> -->

Commit message: added python3 syntax

File: mmuav_description/urdf/uav.base.urdf.xacro (robot description, xacro)
@@ -452,5 +452,5 @@
     <xacro:asap_manipulator parent="base_link">
       <!--origin xyz="0 0 0.2" rpy="${pi/2} 0 0"/-->
-      <origin xyz="0 0 0.2" rpy="0 0 0"/>
+      <origin xyz="0 0 0.1" rpy="${pi/2} 0 0"/>
     </xacro:asap_manipulator>
     <xacro:transmisija

Commit message: [Description,Gazebo] Add asap_manipulator_4r as option.

File: mmuav_description/urdf/uav.base.urdf.xacro (robot description, xacro)
@@ -447,4 +447,116 @@
     </xacro:if>
   </xacro:if>
+  <xacro:if value="${'asap_manipulator_4r' == manipulator_type}">
+    <!-- Try to include manipulator -->
+    <xacro:include filename="$(find aerial_manipulators_description)/urdf/manipulator_base.urdf.xacro" />
+    <xacro:asap_manipulator_4r parent="base_link">
+      <!--origin xyz="0 0 0.2" rpy="${pi/2} 0 0"/-->
+      <origin xyz="0 0 -0.2" rpy="0 0 0"/>
+    </xacro:asap_manipulator_4r>
+    <xacro:transmisija
+      trans_number="1"
+      joint_name="joint1">
+    </xacro:transmisija>
+    <xacro:transmisija
+      trans_number="2"
+      joint_name="joint2">
+    </xacro:transmisija>
+    <xacro:transmisija
+      trans_number="3"
+      joint_name="joint3">
+    </xacro:transmisija>
+    <xacro:transmisija
+      trans_number="4"
+      joint_name="joint4">
+    </xacro:transmisija>
+    <xacro:if value="${'camera' == manipulator_tool}">
+      <xacro:property name="camera_link" value="0.02" />
+      <xacro:property name="camera_inertia">
+        <inertia
+        ixx="1e-8"
+        iyy="1e-8"
+        izz="1e-8"
+        ixy="0.0" ixz="0.0" iyz="0.0" />
+      </xacro:property>
+      <xacro:property name="camera_mass" value="1e-5"/>
+      <xacro:cam
+        camera_link="${camera_link}"
+        camera_mass="${camera_mass}"
+        parent="end_effector_base">
+        <origin xyz="0 0 0" rpy="${PI} 0 0"/>
+        <xacro:insert_block name="camera_inertia"/>
+      </xacro:cam>
+    </xacro:if>
+    <!-- Enable the Joint Feedback -->
+    <!--gazebo reference="joint3">
+      <stopCfm>0.08</stopCfm>
+      <stopErp>0.2</stopErp>
+      <implicitSpringDamper>true</implicitSpringDamper>
+      <provideFeedback>true</provideFeedback>
+    </gazebo-->
+    <!-- The ft_sensor plugin  -->
+    <gazebo>
+      <plugin name="ft_sensor" filename="libgazebo_ros_ft_sensor.so">
+        <updateRate>1000.0</updateRate>
+        <robotNamespace>$(arg name)/asap_manipulator_4r</robotNamespace>
+        <topicName>force_sensor/ft_sensor</topicName>
+        <jointName>joint4</jointName>
+        <noise>
+          <type>gaussian</type>
+          <mean>0.0</mean>
+          <stddev>0.0001</stddev> <!-- change this to simulate noise -->
+        </noise>
+      </plugin>
+    </gazebo>
+    <xacro:if value="${'rod' == manipulator_tool}">
+      <gazebo reference="rod">
+        <collision>
+          <surface>
+            <contact>
+              <collide_bitmask>${collision_bitmask}</collide_bitmask>
+            </contact>
+          </surface>
+        </collision>
+      </gazebo>
+      <!-- Rod link -->
+      <link name="rod">
+        <!--collision>
+          <origin xyz="0 0 0" rpy="0 0 0"/>
+          <geometry>
+            <box size="${camera_link} ${camera_link} ${camera_link}"/>
+          </geometry>
+        </collision-->
+        <visual>
+          <origin xyz="0.15 0 0" rpy="0 0 0"/>
+          <geometry>
+            <box size="0.3 0.01 0.01"/>
+          </geometry>
+          <material name="red"/>
+        </visual>
+        <xacro:unless value="${turn_off_all_collisions}">
+          <collision>
+            <origin xyz="0.15 0 0" rpy="0 0 0"/>
+            <geometry>
+                <box size="0.3 0.01 0.01"/>
+            </geometry>
+          </collision>
+        </xacro:unless>
+        <inertial>
+          <mass value="0.00001" />
+          <origin xyz="0.15 0 0" rpy="0 0 0"/>
+          <inertia
+            ixx="0" ixy="0" ixz="0"
+            iyx="0" iyy="0" iyz="0"
+            izx="0" izy="0" izz="0"/>
+        </inertial>
+      </link>
+      <!-- Rod joint with reference to the parent link -->
+      <joint name="rod_joint" type="fixed">
+        <origin xyz="0 0 0" rpy="0 0 0" />
+        <parent link="end_effector_base"/>
+        <child link="rod"/>
+      </joint>
+    </xacro:if>
+  </xacro:if>
   <!-- <xacro:camera_macro robot_namespace="${namespace}">
   </xacro:camera_macro> -->
