Commit message: First aerial manipulator wth ctl

File: mmuav_description/urdf/uav_wp_manipulator.gazebo.xacro (robot description, xacro)
@@ -2,24 +2,42 @@
 <robot name="uav_wp_manipulator" xmlns:xacro="http://ros.org/wiki/xacro">
     <xacro:include filename="$(find mmuav_description)/urdf/uav.gazebo.xacro" />
-    <!--xacro:include filename="$(find aerial_manipulators_description)/urdf/wp_manipulator.gazebo.xacro" /-->
+    <xacro:include filename="$(find aerial_manipulators_description)/urdf/manipulator_base.urdf.xacro" />
     <!-- aditional arm properties -->
-    <!--xacro:property name="arm_offset_z" value="0.1" /-->
-    <!-- [m] 0.0457-->
-    <!--link name="world">
+    <xacro:property name="arm_offset_z" value="0.0457" /> <!-- [m] -->
+    <link name="world">
     </link>
     <joint name="world_base_joint" type="floating">
         <parent link="world"/>
         <child link="base_link"/>
-    </joint-->
-    <!-- uav -->
-    <xacro:uav
-        mount_velodyne="${arg mount_velodyne}"
-        mount_stereo_cam="${arg mount_stereo_cam}"
-        turn_off_all_collisions="${arg turn_off_all_collisions}"
-        collision_bitmask="${arg collision_bitmask}" >
-    </xacro:uav>
+    </joint>
     <!-- wp_manipulator -->
-    <!--xacro:wp_manipulator parent="base_link">
-        <origin xyz="0 0 ${arm_offset_z}" rpy="0 0 0" />
-    </xacro:wp_manipulator-->
+    <xacro:wp_manipulator parent="base_link" >
+        <origin xyz="0 0 ${arm_offset_z}" rpy="${pi/2} 0 0"/>
+    </xacro:wp_manipulator>
+    <xacro:joint_transmission
+      trans_number="1"
+      joint_name="joint1">
+    </xacro:joint_transmission>
+    <xacro:joint_transmission
+      trans_number="2"
+      joint_name="joint2">
+    </xacro:joint_transmission>
+    <xacro:joint_transmission
+      trans_number="3"
+      joint_name="joint3">
+    </xacro:joint_transmission>
+    <xacro:joint_transmission
+      trans_number="4"
+      joint_name="joint4">
+    </xacro:joint_transmission>
+    <xacro:joint_transmission
+      trans_number="5"
+      joint_name="joint5">
+    </xacro:joint_transmission>
+    <!-- ROS control for aerial manipulator joints -->
+    <gazebo>
+      <plugin name="gazebo_ros_control" filename="libgazebo_ros_control.so">
+        <robotNamespace>uav</robotNamespace>
+      </plugin>
+    </gazebo>
 </robot>

Commit message: [model] repositioned arm

File: mmuav_description/urdf/uav_wp_manipulator.gazebo.xacro (robot description, xacro)
@@ -3,6 +3,9 @@
     <xacro:include filename="$(find mmuav_description)/urdf/uav.gazebo.xacro" />
     <xacro:include filename="$(find aerial_manipulators_description)/urdf/wp_manipulator.base.urdf.xacro" />
+    <!-- positive direction -->
+    <!-- z val = "0.0457" -->
+    <!-- r = ${pi/2} -->
     <!-- aditional arm properties -->
-    <xacro:property name="arm_offset_z" value="0.0457" /> <!-- [m] -->
+    <xacro:property name="arm_offset_z" value="-0.0457" /> <!-- [m] -->
     <link name="world">
     </link>
@@ -16,5 +19,5 @@
         gazebo="true"
         parent="base_link">
-        <origin xyz="0 0 ${arm_offset_z}" rpy="${pi/2} 0 0"/>
+        <origin xyz="0 0 ${arm_offset_z}" rpy="-${pi/2} 0 0"/>
     </xacro:aerial_manipulator>
 </robot>
